Commit message: add axes config files

File: indy_description/urdf_files/icon3.urdf (robot description, URDF)
Before this commit: robot indy, 9 links, 8 joints
Joints:
- joint joint1: axis 0 0 1 -> 0 0 -1
- joint joint2: axis 0 0 1 -> 0 0 -1; limit lower=-1.8849555921538759 upper=2.652900463031381 effort=197.23 velocity=9.16297857297023 -> lower=-3.4557519189487724 upper=1.0821041362364843 effort=197.23 velocity=9.16297857297023; origin xyz=0.0                          0.26                          0.0 rpy=0.0                         0.0                         0.0 -> xyz=0.0                          0.26                          0.0 rpy=0.0                         0.0                         1.570796327
- joint joint4: axis 0 0 1 -> 0 0 -1

File: indy_description/urdf_files/icon7l.urdf (robot description, URDF)
Before this commit: robot indy, 9 links, 8 joints
Joints:
- joint joint2: limit lower=-2.0943951023931953 upper=2.722713633111154 effort=197.23 velocity=6.806784082777885 -> lower=-3.6651914291880923 upper=1.1519173063162575 effort=197.23 velocity=6.806784082777885; origin xyz=0.0                          -0.463                          0.0 rpy=0.0                         0.0                         0.0 -> xyz=0.0                          -0.463                          0.0 rpy=0.0                         0.0                         1.570796327

File: indy_description/urdf_files/indy12_v2.urdf (robot description, URDF)
Before this commit: robot indy, 9 links, 8 joints
Joints:
- joint joint5: axis 0 0 1 -> 0 0 -1

File: indy_description/urdf_files/indy7_v2.urdf (robot description, URDF)
Before this commit: robot indy, 9 links, 8 joints
Joints:
- joint tcp: origin xyz=0.0                          0.0                          0.06 rpy=0.0                         0.0                         0.0 -> xyz=0.0                          0.0                          0.057 rpy=0.0                         0.0                         0.0

File: indy_description/urdf_files/indyrp2_v2.urdf (robot description, URDF)
Before this commit: robot indy, 10 links, 9 joints
Joints:
- joint tcp: origin xyz=0.0                          0.0                          0.06 rpy=0.0                         0.0                         0.0 -> xyz=0.0                          0.0                          0.057 rpy=0.0                         0.0                         0.0

File: indy_description/urdf_files/nuri20c.urdf (robot description, URDF)
Before this commit: robot indy, 9 links, 8 joints
Joints:
- joint joint1: axis 0 0 1 -> 0 0 -1

File: indy_description/urdf_files/nuri3s.urdf (robot description, URDF)
Before this commit: robot indy, 9 links, 8 joints
Joints:
- joint joint1: axis 0 0 1 -> 0 0 -1

File: indy_description/urdf_files/nuri4s.urdf (robot description, URDF)
Before this commit: robot indy, 9 links, 8 joints
Joints:
- joint joint1: axis 0 0 1 -> 0 0 -1
- joint joint2: axis 0 0 1 -> 0 0 -1
- joint joint4: axis 0 0 1 -> 0 0 -1

File: indy_description/urdf_files/nuri7c.urdf (robot description, URDF)
Before this commit: robot indy, 9 links, 8 joints
Joints:
- joint joint1: axis 0 0 1 -> 0 0 -1

Commit message: update for ros jazzy, add basic config for octomap

File: indy_description/urdf/indy.urdf.xacro (robot description, xacro)
@@ -14,4 +14,5 @@
     <xacro:arg name="physical_params" default="$(find indy_description)/urdf/config/$(arg indy_type)/physical_parameters.yaml"/>
     <xacro:arg name="visual_params" default="$(find indy_description)/urdf/config/$(arg indy_type)/visual_parameters.yaml"/>
+    <xacro:arg name="joint_axes_params" default="$(find indy_description)/urdf/config/$(arg indy_type)/joint_axes.yaml"/>
     <xacro:arg name="initial_positions" default="$(find indy_description)/urdf/config/initial_positions.yaml"/>
     <xacro:arg name="transmission_hw_interface" default=""/>
@@ -31,4 +32,5 @@
         physical_parameters_file="$(arg physical_params)"
         visual_parameters_file="$(arg visual_params)"
+        joint_axes_parameters_file="$(arg joint_axes_params)"
         transmission_hw_interface="$(arg transmission_hw_interface)"
         initial_positions_file="$(arg initial_positions)"
