Commit message: update urdf for indy7_v2, icon7l, opti5, add indy7_v3

File: indy_description/urdf/indy.urdf.xacro (robot description, xacro)
@@ -8,11 +8,13 @@
     <xacro:arg name="indy_type" default="indy7"/>
     <xacro:arg name="indy_eye" default="false"/>
+    <xacro:property name="arg_indy_type" value="$(arg indy_type)"/>
+    <xacro:property name="config_indy_type" value="${'indy7_v2' if arg_indy_type == 'indy7_v3' else arg_indy_type}"/>
     <!-- parameters -->
     <xacro:arg name="prefix" default="" />
-    <xacro:arg name="joint_limit_params" default="$(find indy_description)/urdf/config/$(arg indy_type)/joint_limits.yaml"/>
-    <xacro:arg name="kinematics_params" default="$(find indy_description)/urdf/config/$(arg indy_type)/kinematics.yaml"/>
-    <xacro:arg name="physical_params" default="$(find indy_description)/urdf/config/$(arg indy_type)/physical_parameters.yaml"/>
-    <xacro:arg name="visual_params" default="$(find indy_description)/urdf/config/$(arg indy_type)/visual_parameters.yaml"/>
-    <xacro:arg name="joint_axes_params" default="$(find indy_description)/urdf/config/$(arg indy_type)/joint_axes.yaml"/>
+    <xacro:arg name="joint_limit_params" default="$(find indy_description)/urdf/config/${config_indy_type}/joint_limits.yaml"/>
+    <xacro:arg name="kinematics_params" default="$(find indy_description)/urdf/config/${config_indy_type}/kinematics.yaml"/>
+    <xacro:arg name="physical_params" default="$(find indy_description)/urdf/config/${config_indy_type}/physical_parameters.yaml"/>
+    <xacro:arg name="visual_params" default="$(find indy_description)/urdf/config/${config_indy_type}/visual_parameters.yaml"/>
+    <xacro:arg name="joint_axes_params" default="$(find indy_description)/urdf/config/${config_indy_type}/joint_axes.yaml"/>
     <xacro:arg name="initial_positions" default="$(find indy_description)/urdf/config/initial_positions.yaml"/>
     <xacro:arg name="transmission_hw_interface" default=""/>

File: indy_description/urdf/indy_macro.xacro (robot description, xacro)
@@ -24,5 +24,5 @@
         <xacro:define_initialize initial_positions_file="${initial_positions_file}"
             visual_parameters_file="${visual_parameters_file}" indy_type="${indy_type}"/>
-        <xacro:if value="${ indy_type == 'indy7' or indy_type == 'indy7_v2' or indy_type == 'indyrp2' or
+        <xacro:if value="${ indy_type == 'indy7' or indy_type == 'indy7_v2' or indy_type == 'indy7_v3' or indy_type == 'indyrp2' or
                             indy_type == 'indyrp2_v2' or indy_type == 'indy12' or indy_type == 'indy12_v2' or
                             indy_type == 'nuri3s' or indy_type == 'nuri4s' or indy_type == 'nuri7c' or

Commit message: update urdf for indy7_v2, icon7l, opti5, add indy7_v3

File: indy_description/urdf/indy.urdf.xacro (robot description, xacro)
@@ -8,11 +8,13 @@
     <xacro:arg name="indy_type" default="indy7"/>
     <xacro:arg name="indy_eye" default="false"/>
+    <xacro:property name="arg_indy_type" value="$(arg indy_type)"/>
+    <xacro:property name="config_indy_type" value="${'indy7_v2' if arg_indy_type == 'indy7_v3' else arg_indy_type}"/>
     <!-- parameters -->
     <xacro:arg name="prefix" default="" />
-    <xacro:arg name="joint_limit_params" default="$(find indy_description)/urdf/config/$(arg indy_type)/joint_limits.yaml"/>
-    <xacro:arg name="kinematics_params" default="$(find indy_description)/urdf/config/$(arg indy_type)/kinematics.yaml"/>
-    <xacro:arg name="physical_params" default="$(find indy_description)/urdf/config/$(arg indy_type)/physical_parameters.yaml"/>
-    <xacro:arg name="visual_params" default="$(find indy_description)/urdf/config/$(arg indy_type)/visual_parameters.yaml"/>
-    <xacro:arg name="joint_axes_params" default="$(find indy_description)/urdf/config/$(arg indy_type)/joint_axes.yaml"/>
+    <xacro:arg name="joint_limit_params" default="$(find indy_description)/urdf/config/${config_indy_type}/joint_limits.yaml"/>
+    <xacro:arg name="kinematics_params" default="$(find indy_description)/urdf/config/${config_indy_type}/kinematics.yaml"/>
+    <xacro:arg name="physical_params" default="$(find indy_description)/urdf/config/${config_indy_type}/physical_parameters.yaml"/>
+    <xacro:arg name="visual_params" default="$(find indy_description)/urdf/config/${config_indy_type}/visual_parameters.yaml"/>
+    <xacro:arg name="joint_axes_params" default="$(find indy_description)/urdf/config/${config_indy_type}/joint_axes.yaml"/>
     <xacro:arg name="initial_positions" default="$(find indy_description)/urdf/config/initial_positions.yaml"/>
     <xacro:arg name="transmission_hw_interface" default=""/>

File: indy_description/urdf/indy_macro.xacro (robot description, xacro)
@@ -24,8 +24,8 @@
         <xacro:define_initialize initial_positions_file="${initial_positions_file}"
             visual_parameters_file="${visual_parameters_file}" indy_type="${indy_type}"/>
-        <xacro:if value="${ indy_type == 'indy7' or indy_type == 'indy7_v2' or indy_type == 'indyrp2' or
+        <xacro:if value="${ indy_type == 'indy7' or indy_type == 'indy7_v2' or indy_type == 'indy7_v3' or indy_type == 'indyrp2' or
                             indy_type == 'indyrp2_v2' or indy_type == 'indy12' or indy_type == 'indy12_v2' or
                             indy_type == 'nuri3s' or indy_type == 'nuri4s' or indy_type == 'nuri7c' or
-                            indy_type == 'nuri20c' or indy_type == 'opti5'}">
+                            indy_type == 'nuri20c' or indy_type == 'nuri30s' or indy_type == 'opti5'}">
             <xacro:property name="material_0" value="indy_white"/>
             <xacro:property name="material_1" value="indy_white"/>
