Commit message: update indy7_v3, indyrp2_v2, indy12

File: indy_description/urdf/indy.urdf.xacro (robot description, xacro)
@@ -9,5 +9,5 @@
     <xacro:arg name="indy_eye" default="false"/>
     <xacro:property name="arg_indy_type" value="$(arg indy_type)"/>
-    <xacro:property name="config_indy_type" value="${'indy7_v2' if arg_indy_type == 'indy7_v3' else arg_indy_type}"/>
+    <xacro:property name="config_indy_type" value="${arg_indy_type}"/>
     <!-- parameters -->
     <xacro:arg name="prefix" default="" />

File: indy_description/urdf/indy_macro.xacro (robot description, xacro)
@@ -121,5 +121,5 @@
         </xacro:unless>
         <!-- joints -->
-        <xacro:macro name="define_joint" params="joint_type joint_index parent_link child_link">
+        <xacro:macro name="define_joint" params="joint_type joint_name origin_key parent_link child_link">
             <xacro:property name="config_joint_limit_parameters" value="${xacro.load_yaml(joint_limits_parameters_file)}"/>
             <xacro:property name="config_kinematics_parameters" value="${xacro.load_yaml(kinematics_parameters_file)}"/>
@@ -128,20 +128,20 @@
             <xacro:property name="sec_limits" value="${config_joint_limit_parameters['joint_limits']}"/>
             <xacro:property name="sec_joint_axes" value="${config_joint_axes_parameters['joint_axes']}" />
-            <joint name="${prefix}${joint_index}" type="${joint_type}">
+            <joint name="${prefix}${joint_name}" type="${joint_type}">
                 <parent link="${prefix}${parent_link}"/>
                 <child link="${prefix}${child_link}"/>
                 <origin
-                    xyz="${sec_kinematics[joint_index]['x']}
-                        ${sec_kinematics[joint_index]['y']}
-                        ${sec_kinematics[joint_index]['z']}"
-                    rpy="${sec_kinematics[joint_index]['roll']}
-                        ${sec_kinematics[joint_index]['pitch']}
-                        ${sec_kinematics[joint_index]['yaw']}"/>
+                    xyz="${sec_kinematics[origin_key]['x']}
+                        ${sec_kinematics[origin_key]['y']}
+                        ${sec_kinematics[origin_key]['z']}"
+                    rpy="${sec_kinematics[origin_key]['roll']}
+                        ${sec_kinematics[origin_key]['pitch']}
+                        ${sec_kinematics[origin_key]['yaw']}"/>
                 <xacro:if value="${joint_type == 'revolute' or joint_type == 'continuous'}">
                     <!-- Use configurable axis if available, fallback to default [0,0,1] -->
-                    <xacro:if value="${joint_index in sec_joint_axes}">
-                        <axis xyz="${sec_joint_axes[joint_index][0]} ${sec_joint_axes[joint_index][1]} ${sec_joint_axes[joint_index][2]}"/>
+                    <xacro:if value="${origin_key in sec_joint_axes}">
+                        <axis xyz="${sec_joint_axes[origin_key][0]} ${sec_joint_axes[origin_key][1]} ${sec_joint_axes[origin_key][2]}"/>
                     </xacro:if>
-                    <xacro:unless value="${joint_index in sec_joint_axes}">
+                    <xacro:unless value="${origin_key in sec_joint_axes}">
                         <axis xyz="0 0 1"/>
                     </xacro:unless>
@@ -150,8 +150,8 @@
                 <xacro:if value="${joint_type == 'revolute'}">
                     <limit
-                        lower="${sec_limits[joint_index]['min_position']}"
-                        upper="${sec_limits[joint_index]['max_position']}"
-                        effort="${sec_limits[joint_index]['max_effort']}"
-                        velocity="${sec_limits[joint_index]['max_velocity']}"/>
+                        lower="${sec_limits[origin_key]['min_position']}"
+                        upper="${sec_limits[origin_key]['max_position']}"
+                        effort="${sec_limits[origin_key]['max_effort']}"
+                        velocity="${sec_limits[origin_key]['max_velocity']}"/>
                 </xacro:if>
             </joint>
@@ -163,22 +163,22 @@
                 <child link="$(arg prefix)body_base"/>
             </joint>
-            <xacro:define_joint joint_type="revolute" joint_index="base_frame" parent_link="body_base" child_link="body_frame"/>
-            <xacro:define_joint joint_type="fixed" joint_index="frame_cover" parent_link="body_frame" child_link="body_cover"/>
-            <xacro:define_joint joint_type="fixed" joint_index="left_arm_connect" parent_link="body_frame" child_link="left_arm_link0"/>
-            <xacro:define_joint joint_type="fixed" joint_index="right_arm_connect" parent_link="body_frame" child_link="right_arm_link0"/>
-            <xacro:define_joint joint_type="revolute" joint_index="left_arm_joint0" parent_link="left_arm_link0" child_link="left_arm_link1"/>
-            <xacro:define_joint joint_type="revolute" joint_index="left_arm_joint1" parent_link="left_arm_link1" child_link="left_arm_link2"/>
-            <xacro:define_joint joint_type="revolute" joint_index="left_arm_joint2" parent_link="left_arm_link2" child_link="left_arm_link3"/>
-            <xacro:define_joint joint_type="revolute" joint_index="left_arm_joint3" parent_link="left_arm_link3" child_link="left_arm_link4"/>
-            <xacro:define_joint joint_type="revolute" joint_index="left_arm_joint4" parent_link="left_arm_link4" child_link="left_arm_link5"/>
-            <xacro:define_joint joint_type="revolute" joint_index="left_arm_joint5" parent_link="left_arm_link5" child_link="left_arm_link6"/>
-            <xacro:define_joint joint_type="fixed"    joint_index="left_arm_tcp" parent_link="left_arm_link6" child_link="left_arm_tcp"/>
-            <xacro:define_joint joint_type="revolute" joint_index="right_arm_joint0" parent_link="right_arm_link0" child_link="right_arm_link1"/>
-            <xacro:define_joint joint_type="revolute" joint_index="right_arm_joint1" parent_link="right_arm_link1" child_link="right_arm_link2"/>
-            <xacro:define_joint joint_type="revolute" joint_index="right_arm_joint2" parent_link="right_arm_link2" child_link="right_arm_link3"/>
-            <xacro:define_joint joint_type="revolute" joint_index="right_arm_joint3" parent_link="right_arm_link3" child_link="right_arm_link4"/>
-            <xacro:define_joint joint_type="revolute" joint_index="right_arm_joint4" parent_link="right_arm_link4" child_link="right_arm_link5"/>
-            <xacro:define_joint joint_type="revolute" joint_index="right_arm_joint5" parent_link="right_arm_link5" child_link="right_arm_link6"/>
-            <xacro:define_joint joint_type="fixed"    joint_index="right_arm_tcp" parent_link="right_arm_link6" child_link="right_arm_tcp"/>
+            <xacro:define_joint joint_type="revolute" joint_name="base_frame" origin_key="base_frame" parent_link="body_base" child_link="body_frame"/>
+            <xacro:define_joint joint_type="fixed" joint_name="frame_cover" origin_key="frame_cover" parent_link="body_frame" child_link="body_cover"/>
+            <xacro:define_joint joint_type="fixed" joint_name="left_arm_connect" origin_key="left_arm_connect" parent_link="body_frame" child_link="left_arm_link0"/>
+            <xacro:define_joint joint_type="fixed" joint_name="right_arm_connect" origin_key="right_arm_connect" parent_link="body_frame" child_link="right_arm_link0"/>
+            <xacro:define_joint joint_type="revolute" joint_name="left_arm_joint0" origin_key="left_arm_joint0" parent_link="left_arm_link0" child_link="left_arm_link1"/>
+            <xacro:define_joint joint_type="revolute" joint_name="left_arm_joint1" origin_key="left_arm_joint1" parent_link="left_arm_link1" child_link="left_arm_link2"/>
+            <xacro:define_joint joint_type="revolute" joint_name="left_arm_joint2" origin_key="left_arm_joint2" parent_link="left_arm_link2" child_link="left_arm_link3"/>
+            <xacro:define_joint joint_type="revolute" joint_name="left_arm_joint3" origin_key="left_arm_joint3" parent_link="left_arm_link3" child_link="left_arm_link4"/>
+            <xacro:define_joint joint_type="revolute" joint_name="left_arm_joint4" origin_key="left_arm_joint4" parent_link="left_arm_link4" child_link="left_arm_link5"/>
+            <xacro:define_joint joint_type="revolute" joint_name="left_arm_joint5" origin_key="left_arm_joint5" parent_link="left_arm_link5" child_link="left_arm_link6"/>
+            <xacro:define_joint joint_type="fixed" joint_name="left_arm_tcp_fixed" origin_key="left_arm_tcp" parent_link="left_arm_link6" child_link="left_arm_tcp"/>
+            <xacro:define_joint joint_type="revolute" joint_name="right_arm_joint0" origin_key="right_arm_joint0" parent_link="right_arm_link0" child_link="right_arm_link1"/>
+            <xacro:define_joint joint_type="revolute" joint_name="right_arm_joint1" origin_key="right_arm_joint1" parent_link="right_arm_link1" child_link="right_arm_link2"/>
+            <xacro:define_joint joint_type="revolute" joint_name="right_arm_joint2" origin_key="right_arm_joint2" parent_link="right_arm_link2" child_link="right_arm_link3"/>
+            <xacro:define_joint joint_type="revolute" joint_name="right_arm_joint3" origin_key="right_arm_joint3" parent_link="right_arm_link3" child_link="right_arm_link4"/>
+            <xacro:define_joint joint_type="revolute" joint_name="right_arm_joint4" origin_key="right_arm_joint4" parent_link="right_arm_link4" child_link="right_arm_link5"/>
+            <xacro:define_joint joint_type="revolute" joint_name="right_arm_joint5" origin_key="right_arm_joint5" parent_link="right_arm_link5" child_link="right_arm_link6"/>
+            <xacro:define_joint joint_type="fixed" joint_name="right_arm_tcp_fixed" origin_key="right_arm_tcp" parent_link="right_arm_link6" child_link="right_arm_tcp"/>
         </xacro:if>
         <xacro:unless value="${indy_type == 'dual_icon3'}">
@@ -188,16 +188,16 @@
                 <child link="$(arg prefix)link0"/>
             </joint>
-            <xacro:define_joint joint_type="revolute" joint_index="joint0" parent_link="link0" child_link="link1"/>
-            <xacro:define_joint joint_type="revolute" joint_index="joint1" parent_link="link1" child_link="link2"/>
-            <xacro:define_joint joint_type="revolute" joint_index="joint2" parent_link="link2" child_link="link3"/>
-            <xacro:define_joint joint_type="revolute" joint_index="joint3" parent_link="link3" child_link="link4"/>
-            <xacro:define_joint joint_type="revolute" joint_index="joint4" parent_link="link4" child_link="link5"/>
-            <xacro:define_joint joint_type="revolute" joint_index="joint5" parent_link="link5" child_link="link6"/>
+            <xacro:define_joint joint_type="revolute" joint_name="joint0" origin_key="joint0" parent_link="link0" child_link="link1"/>
+            <xacro:define_joint joint_type="revolute" joint_name="joint1" origin_key="joint1" parent_link="link1" child_link="link2"/>
+            <xacro:define_joint joint_type="revolute" joint_name="joint2" origin_key="joint2" parent_link="link2" child_link="link3"/>
+            <xacro:define_joint joint_type="revolute" joint_name="joint3" origin_key="joint3" parent_link="link3" child_link="link4"/>
+            <xacro:define_joint joint_type="revolute" joint_name="joint4" origin_key="joint4" parent_link="link4" child_link="link5"/>
+            <xacro:define_joint joint_type="revolute" joint_name="joint5" origin_key="joint5" parent_link="link5" child_link="link6"/>
             <xacro:if value="${indy_type == 'indyrp2' or indy_type == 'indyrp2_v2'}">
-                <xacro:define_joint joint_type="revolute" joint_index="joint6" parent_link="link6" child_link="link7"/>
-                <xacro:define_joint joint_type="fixed" joint_index="tcp" parent_link="link7" child_link="tcp"/>
+                <xacro:define_joint joint_type="revolute" joint_name="joint6" origin_key="joint6" parent_link="link6" child_link="link7"/>
+                <xacro:define_joint joint_type="fixed" joint_name="tcp_fixed" origin_key="tcp" parent_link="link7" child_link="tcp"/>
             </xacro:if>
             <xacro:unless value="${indy_type == 'indyrp2' or indy_type == 'indyrp2_v2'}">
-                <xacro:define_joint joint_type="fixed" joint_index="tcp" parent_link="link6" child_link="tcp"/>
+                <xacro:define_joint joint_type="fixed" joint_name="tcp_fixed" origin_key="tcp" parent_link="link6" child_link="tcp"/>
             </xacro:unless>
         </xacro:unless>

File: indy_description/urdf_files/dual_icon3.urdf (robot description, URDF)
Before this commit: robot indy, 20 links, 19 joints
Joints:
- removed joint left_arm_tcp
- removed joint right_arm_tcp
- added joint left_arm_tcp_fixed: type fixed, parent left_arm_link6, child left_arm_tcp, origin xyz=0.0                          0.0                          0.0 rpy=0.0                         0.0                         0.0
- added joint right_arm_tcp_fixed: type fixed, parent right_arm_link6, child right_arm_tcp, origin xyz=0.0                          0.0                          0.0 rpy=0.0                         0.0                         0.0

File: indy_description/urdf_files/icon3.urdf (robot description, URDF)
Before this commit: robot indy, 9 links, 8 joints
Joints:
- removed joint tcp
- added joint tcp_fixed: type fixed, parent link6, child tcp, origin xyz=0.0                          0.0                          0.0 rpy=0.0                         0.0                         0.0

File: indy_description/urdf_files/icon7l.urdf (robot description, URDF)
Before this commit: robot indy, 9 links, 8 joints
Joints:
- removed joint tcp
- added joint tcp_fixed: type fixed, parent link6, child tcp, origin xyz=0.0                          0.0                          0.0 rpy=0.0                         0.0                         0.0
- joint joint1: axis 0 0 1 -> 0 0 -1
- joint joint2: axis 0 0 1 -> 0 0 -1
- joint joint4: axis 0 0 1 -> 0 0 -1
- joint joint5: origin xyz=0.0                          0.089                          0.0 rpy=1.570796327                         0.0                         3.14159265 -> xyz=0.0                          0.089                          0.0 rpy=1.570796327                         1.570796327                         3.14159265

File: indy_description/urdf_files/indy12.urdf (robot description, URDF)
Before this commit: robot indy, 9 links, 8 joints
Joints:
- removed joint tcp
- added joint tcp_fixed: type fixed, parent link6, child tcp, origin xyz=0.0                          0.0                          0.056 rpy=0.0                         0.0                         0.0
- joint joint0: origin xyz=0                          0                          0.13 rpy=0                         0                         0 -> xyz=0                          0                          0.1305 rpy=0                         0                         0
- joint joint1: origin xyz=0                          -0.1275                          0.22 rpy=1.570796327                         -1.570796327                         0 -> xyz=0                          -0.128                          0.2195 rpy=1.570796327                         -1.570796327                         0

File: indy_description/urdf_files/indy12_v2.urdf (robot description, URDF)
Before this commit: robot indy, 9 links, 8 joints
Joints:
- removed joint tcp
- added joint tcp_fixed: type fixed, parent link6, child tcp, origin xyz=0.0                          0.0                          0.085 rpy=0.0                         0.0                         0.0

File: indy_description/urdf_files/indy7.urdf (robot description, URDF)
Before this commit: robot indy, 9 links, 8 joints
Joints:
- removed joint tcp
- added joint tcp_fixed: type fixed, parent link6, child tcp, origin xyz=0.0                          0.0                          0.06 rpy=0.0                         0.0                         0.0

File: indy_description/urdf_files/indy7_eye.urdf (robot description, URDF)
Before this commit: robot indy, 9 links, 8 joints
Joints:
- removed joint tcp
- added joint tcp_fixed: type fixed, parent link6, child tcp, origin xyz=0.0                          0.0                          0.06 rpy=0.0                         0.0                         0.0

File: indy_description/urdf_files/indy7_v2.urdf (robot description, URDF)
Before this commit: robot indy, 9 links, 8 joints
Joints:
- removed joint tcp
- added joint tcp_fixed: type fixed, parent link6, child tcp, origin xyz=0.0                          0.0                          0.0505 rpy=0.0                         0.0                         0.0

File: indy_description/urdf_files/indy7_v3.urdf (robot description, URDF)
Before this commit: robot indy, 10 links, 9 joints
Links:
- removed link link7
- link link0: mass 1.6703078 -> 1.66957888
- link link1: mass 11.44444535 -> 11.43955917
- link link2: mass 4.43308185 -> 6.11383823
- link link3: mass 2.87045928 -> 2.68211719
- link link4: mass 2.68206064 -> 2.12830848
- link link5: mass 2.12987371 -> 2.32413397
- link link6: mass 2.22412271 -> 0.39652271
Joints:
- removed joint joint6
- joint joint0: origin xyz=0                          0                          0.0772 rpy=0                         0                         0 -> xyz=0                          0                          0.0785 rpy=0                         0                         0
- joint joint1: origin xyz=0                          -0.1093                          0.2228 rpy=1.570796327                         1.570796327                         0 -> xyz=0                          -0.1105                          0.2215 rpy=3.1415926536                         1.570796327                         1.570796327
- joint joint2: origin xyz=-0.384                          0                          0.0847 rpy=-1.570796327                         0                         1.570796327 -> xyz=-0.45                          0                          -0.0335 rpy=0                         0                         0
- joint joint3: limit lower=-3.0543261909900767 upper=3.0543261909900767 effort=197.23 velocity=2.6179938779914944 -> lower=-3.0543261909900767 upper=3.0543261909900767 effort=79.79 velocity=3.141592653589793; origin xyz=0                          0.1153                          0.0655 rpy=1.570796327                         1.570796327                         0 -> xyz=-0.2845                          0                          -0.0735 rpy=1.570796327                         0                         -1.570796327
- joint joint4: origin xyz=-0.2665                          0                          -0.0747 rpy=-1.570796327                         0                         1.570796327 -> xyz=0                          0.1405                          0.065486 rpy=-1.570796327                         0                         0
- joint joint5: limit lower=-3.0543261909900767 upper=3.0543261909900767 effort=79.79 velocity=3.141592653589793 -> lower=-3.7524578917878086 upper=3.7524578917878086 effort=79.79 velocity=3.141592653589793; origin xyz=0                          -0.1143                          0.0835 rpy=1.570796327                         1.570796327                         0 -> xyz=0                          -0.050495                          0.058505 rpy=1.570796327                         3.1415926536                         0
- joint tcp_fixed: origin xyz=0.0                          0.0                          0.06 rpy=0.0                         0.0                         0.0 -> xyz=0.0                          0.0                          0.0557 rpy=0.0                         0.0                         0.0; parent link7 -> link6

File: indy_description/urdf_files/indyrp2_eye.urdf (robot description, URDF)
Before this commit: robot indy, 10 links, 9 joints
Joints:
- removed joint tcp
- added joint tcp_fixed: type fixed, parent link7, child tcp, origin xyz=0.0                          0.0                          0.06 rpy=0.0                         0.0                         0.0

File: indy_description/urdf_files/indyrp2_v2.urdf (robot description, URDF)
Before this commit: robot indy, 10 links, 9 joints
Joints:
- removed joint tcp
- added joint tcp_fixed: type fixed, parent link7, child tcp, origin xyz=0.0                          0.0                          0.0515 rpy=0.0                         0.0                         0.0
- joint joint0: origin xyz=0                          0                          0.0775 rpy=0                         0                         0 -> xyz=0                          0                          0.0785 rpy=0                         0                         0
- joint joint1: origin xyz=0                          -0.109                          0.222 rpy=1.570796327                         0                         0 -> xyz=0                          -0.1103                          0.2215 rpy=1.570796327                         0                         0
- joint joint2: origin xyz=0                          0.361                          0.0845 rpy=-1.570796327                         0                         0 -> xyz=0                          0.3605                          0.0832 rpy=-1.570796327                         0                         0
- joint joint3: origin xyz=0                          0.1153                          0.0885 rpy=-1.570796327                         0                         3.1415926536 -> xyz=0                          0.1163                          0.0895 rpy=-1.570796327                         0                         3.1415926536
- joint joint4: origin xyz=0                          -0.267                          -0.075 rpy=-1.570796327                         0                         3.1415926536 -> xyz=0                          -0.2655                          -0.0737 rpy=-1.570796327                         0                         3.1415926536
- joint joint5: origin xyz=0                          -0.114                          0.0835 rpy=1.570796327                         0                         0 -> xyz=0                          -0.1153                          0.0845 rpy=1.570796327                         0                         0
- joint joint6: origin xyz=0                          0.052                          0.085 rpy=-1.570796327                         0                         0 -> xyz=0                          0.052                          0.0837 rpy=-1.570796327                         0                         0

File: indy_description/urdf_files/nuri20c.urdf (robot description, URDF)
Before this commit: robot indy, 9 links, 8 joints
Joints:
- removed joint tcp
- added joint tcp_fixed: type fixed, parent link6, child tcp, origin xyz=0.0                          0.0                          0.04 rpy=0.0                         0.0                         0.0
