Commit message: update indy7_v3, indyrp2_v2, indy12

File: indy_description/urdf_files/nuri30s.urdf (robot description, URDF)
Before this commit: robot indy, 10 links, 9 joints
Links:
- removed link link7
- link link0: mass 1.6703078 -> 12.0
- link link1: mass 11.44444535 -> 30.0
- link link2: mass 4.43308185 -> 20.0
- link link3: mass 2.87045928 -> 9.0
- link link4: mass 2.68206064 -> 8.0
- link link5: mass 2.12987371 -> 8.0
- link link6: mass 2.22412271 -> 1.0
Joints:
- removed joint joint6
- joint joint0: limit lower=-3.0543261909900767 upper=3.0543261909900767 effort=431.97 velocity=2.6179938779914944 -> lower=-6.283185307179586 upper=6.283185307179586 effort=431.97 velocity=3.141592653589793; origin xyz=0                          0                          0.0772 rpy=0                         0                         0 -> xyz=0.0                          0.0                          0.0727 rpy=0.0                         0.0                         0.0
- joint joint1: limit lower=-3.0543261909900767 upper=3.0543261909900767 effort=431.97 velocity=2.6179938779914944 -> lower=-2.705260340591211 upper=2.443460952792061 effort=431.97 velocity=3.141592653589793; origin xyz=0                          -0.1093                          0.2228 rpy=1.570796327                         1.570796327                         0 -> xyz=0.0                          0.151                          0.113 rpy=1.570796327                         0.0                         0.0
- joint joint2: limit lower=-3.0543261909900767 upper=3.0543261909900767 effort=197.23 velocity=2.6179938779914944 -> lower=-3.0543261909900767 upper=2.356194490192345 effort=197.23 velocity=3.141592653589793; origin xyz=-0.384                          0                          0.0847 rpy=-1.570796327                         0                         1.570796327 -> xyz=0.0                          0.850063                          0.0095 rpy=0.0                         0.0                         0.0
- joint joint3: limit lower=-3.0543261909900767 upper=3.0543261909900767 effort=197.23 velocity=2.6179938779914944 -> lower=-6.283185307179586 upper=6.283185307179586 effort=79.79 velocity=3.141592653589793; origin xyz=0                          0.1153                          0.0655 rpy=1.570796327                         1.570796327                         0 -> xyz=0.0                          0.7915                          -0.0025 rpy=0.0                         0.0                         0.0
- joint joint4: limit lower=-3.0543261909900767 upper=3.0543261909900767 effort=79.79 velocity=3.141592653589793 -> lower=-6.283185307179586 upper=6.283185307179586 effort=79.79 velocity=3.141592653589793; origin xyz=-0.2665                          0                          -0.0747 rpy=-1.570796327                         0                         1.570796327 -> xyz=0.0                          0.0865                          -0.072 rpy=-1.570796327                         0.0                         0.0
- joint joint5: limit lower=-3.0543261909900767 upper=3.0543261909900767 effort=79.79 velocity=3.141592653589793 -> lower=-6.283185307179586 upper=6.283185307179586 effort=79.79 velocity=3.141592653589793; origin xyz=0                          -0.1143                          0.0835 rpy=1.570796327                         1.570796327                         0 -> xyz=0.0                          0.0865                          0.072 rpy=-1.570796327                         0.0                         0.0
- joint tcp_fixed: origin xyz=0.0                          0.0                          0.06 rpy=0.0                         0.0                         0.0 -> xyz=0.0                          0.0                          0.048 rpy=0.0                         0.0                         0.0; parent link7 -> link6

File: indy_description/urdf_files/nuri3s.urdf (robot description, URDF)
Before this commit: robot indy, 9 links, 8 joints
Joints:
- removed joint tcp
- added joint tcp_fixed: type fixed, parent link6, child tcp, origin xyz=0.0                          0.0                          0.0285 rpy=0.0                         0.0                         0.0

File: indy_description/urdf_files/nuri4s.urdf (robot description, URDF)
Before this commit: robot indy, 9 links, 8 joints
Joints:
- removed joint tcp
- added joint tcp_fixed: type fixed, parent link6, child tcp, origin xyz=0.0                          0.0                          0.0285 rpy=0.0                         0.0                         0.0

File: indy_description/urdf_files/nuri7c.urdf (robot description, URDF)
Before this commit: robot indy, 9 links, 8 joints
Joints:
- removed joint tcp
- added joint tcp_fixed: type fixed, parent link6, child tcp, origin xyz=0.0                          0.0                          0.054 rpy=0.0                         0.0                         0.0

File: indy_description/urdf_files/opti5.urdf (robot description, URDF)
Before this commit: robot indy, 9 links, 8 joints
Joints:
- removed joint tcp
- added joint tcp_fixed: type fixed, parent link6, child tcp, origin xyz=0.0                          0.0                          0.054 rpy=0.0                         0.0                         0.0

Commit message: update indy7_v3, indyrp2_v2, indy12

File: indy_description/urdf/indy.urdf.xacro (robot description, xacro)
@@ -9,5 +9,5 @@
     <xacro:arg name="indy_eye" default="false"/>
     <xacro:property name="arg_indy_type" value="$(arg indy_type)"/>
-    <xacro:property name="config_indy_type" value="${'indy7_v2' if arg_indy_type == 'indy7_v3' else arg_indy_type}"/>
+    <xacro:property name="config_indy_type" value="${arg_indy_type}"/>
     <!-- parameters -->
     <xacro:arg name="prefix" default="" />

File: indy_description/urdf_files/icon7l.urdf (robot description, URDF)
Before this commit: robot indy, 9 links, 8 joints
Joints:
- joint joint1: axis 0 0 1 -> 0 0 -1
- joint joint2: axis 0 0 1 -> 0 0 -1
- joint joint4: axis 0 0 1 -> 0 0 -1
- joint joint5: origin xyz=0.0                          0.089                          0.0 rpy=1.570796327                         0.0                         3.14159265 -> xyz=0.0                          0.089                          0.0 rpy=1.570796327                         1.570796327                         3.14159265

File: indy_description/urdf_files/indy12.urdf (robot description, URDF)
Before this commit: robot indy, 9 links, 8 joints
Joints:
- joint joint0: origin xyz=0                          0                          0.13 rpy=0                         0                         0 -> xyz=0                          0                          0.1305 rpy=0                         0                         0
- joint joint1: origin xyz=0                          -0.1275                          0.22 rpy=1.570796327                         -1.570796327                         0 -> xyz=0                          -0.128                          0.2195 rpy=1.570796327                         -1.570796327                         0
- joint tcp: origin xyz=0.0                          0.0                          0.06 rpy=0.0                         0.0                         0.0 -> xyz=0.0                          0.0                          0.056 rpy=0.0                         0.0                         0.0

File: indy_description/urdf_files/indy12_v2.urdf (robot description, URDF)
Before this commit: robot indy, 9 links, 8 joints
Joints:
- joint joint0: origin xyz=0                          0                          0.083 rpy=0                         0                         0 -> xyz=0                          0                          0.0815 rpy=0                         0                         0
- joint joint1: origin xyz=0                          -0.137                          0.2675 rpy=1.570796327                         -1.570796327                         0 -> xyz=0                          -0.1355                          0.2685 rpy=1.570796327                         -1.570796327                         0
- joint joint2: origin xyz=0.652                          0                          -0.0205 rpy=0                         0                         1.570796327 -> xyz=0.65                          0                          -0.0185 rpy=0                         0                         1.570796327
- joint joint3: origin xyz=0                          -0.21                          -0.10595 rpy=-1.570796327                         0                         3.14159265 -> xyz=0                          -0.187                          -0.1065 rpy=-1.570796327                         0                         3.14159265
- joint joint4: origin xyz=0                          -0.1305                          0.3628 rpy=-1.570796327                         0                         3.14159265 -> xyz=0                          -0.129                          0.363 rpy=-1.570796327                         0                         3.14159265
- joint joint5: axis 0 0 -1 -> 0 0 1; origin xyz=0                          -0.075                          0.08 rpy=-1.570796327                         0                         3.14159265 -> xyz=0                          -0.074                          0.0795 rpy=-1.570796327                         0                         3.14159265
- joint tcp: origin xyz=0.0                          0.0                          0.09 rpy=0.0                         0.0                         0.0 -> xyz=0.0                          0.0                          0.085 rpy=0.0                         0.0                         0.0

File: indy_description/urdf_files/indy7_v3.urdf (robot description, URDF)
Before this commit: robot indy, 9 links, 8 joints
Joints:
- joint joint0: origin xyz=0                          0                          0.0775 rpy=0                         0                         0 -> xyz=0                          0                          0.0785 rpy=0                         0                         0
- joint joint1: origin xyz=0                          -0.109                          0.222 rpy=1.570796327                         0                         0 -> xyz=0                          -0.1105                          0.2215 rpy=3.1415926536                         1.570796327                         1.570796327
- joint joint2: origin xyz=0                          0.45                          -0.0305 rpy=0                         0                         3.1415926536 -> xyz=-0.45                          0                          -0.0335 rpy=0                         0                         0
- joint joint3: origin xyz=0                          -0.267                          -0.075 rpy=-1.570796327                         0                         3.1415926536 -> xyz=-0.2845                          0                          -0.0735 rpy=1.570796327                         0                         -1.570796327
- joint joint4: origin xyz=0                          -0.114                          0.0835 rpy=1.570796327                         0                         0 -> xyz=0                          0.1405                          0.065486 rpy=-1.570796327                         0                         0
- joint joint5: origin xyz=0                          0.052                          0.085 rpy=-1.570796327                         0                         0 -> xyz=0                          -0.050495                          0.058505 rpy=1.570796327                         3.1415926536                         0
- joint tcp: origin xyz=0.0                          0.0                          0.0505 rpy=0.0                         0.0                         0.0 -> xyz=0.0                          0.0                          0.0557 rpy=0.0                         0.0                         0.0

File: indy_description/urdf_files/indyrp2_v2.urdf (robot description, URDF)
Before this commit: robot indy, 10 links, 9 joints
Joints:
- joint joint0: origin xyz=0                          0                          0.0775 rpy=0                         0                         0 -> xyz=0                          0                          0.0785 rpy=0                         0                         0
- joint joint1: origin xyz=0                          -0.109                          0.222 rpy=1.570796327                         0                         0 -> xyz=0                          -0.1103                          0.2215 rpy=1.570796327                         0                         0
- joint joint2: origin xyz=0                          0.361                          0.0845 rpy=-1.570796327                         0                         0 -> xyz=0                          0.3605                          0.0832 rpy=-1.570796327                         0                         0
- joint joint3: origin xyz=0                          0.1153                          0.0885 rpy=-1.570796327                         0                         3.1415926536 -> xyz=0                          0.1163                          0.0895 rpy=-1.570796327                         0                         3.1415926536
- joint joint4: origin xyz=0                          -0.267                          -0.075 rpy=-1.570796327                         0                         3.1415926536 -> xyz=0                          -0.2655                          -0.0737 rpy=-1.570796327                         0                         3.1415926536
- joint joint5: origin xyz=0                          -0.114                          0.0835 rpy=1.570796327                         0                         0 -> xyz=0                          -0.1153                          0.0845 rpy=1.570796327                         0                         0
- joint joint6: origin xyz=0                          0.052                          0.085 rpy=-1.570796327                         0                         0 -> xyz=0                          0.052                          0.0837 rpy=-1.570796327                         0                         0
- joint tcp: origin xyz=0.0                          0.0                          0.057 rpy=0.0                         0.0                         0.0 -> xyz=0.0                          0.0                          0.0515 rpy=0.0                         0.0                         0.0

File: indy_description/urdf_files/nuri30s.urdf (robot description, URDF)
Before this commit: robot indy, 9 links, 8 joints
Links:
- link link0: mass 1.66957888 -> 12.0
- link link1: mass 11.43955917 -> 30.0
- link link2: mass 6.11383823 -> 20.0
- link link3: mass 2.68211719 -> 9.0
- link link4: mass 2.12830848 -> 8.0
- link link5: mass 2.32413397 -> 8.0
- link link6: mass 0.39652271 -> 1.0
Joints:
- joint joint0: limit lower=-3.0543261909900767 upper=3.0543261909900767 effort=431.97 velocity=2.6179938779914944 -> lower=-6.283185307179586 upper=6.283185307179586 effort=431.97 velocity=3.141592653589793; origin xyz=0                          0                          0.0775 rpy=0                         0                         0 -> xyz=0.0                          0.0                          0.0727 rpy=0.0                         0.0                         0.0
- joint joint1: limit lower=-3.0543261909900767 upper=3.0543261909900767 effort=431.97 velocity=2.6179938779914944 -> lower=-2.705260340591211 upper=2.443460952792061 effort=431.97 velocity=3.141592653589793; origin xyz=0                          -0.109                          0.222 rpy=1.570796327                         0                         0 -> xyz=0.0                          0.151                          0.113 rpy=1.570796327                         0.0                         0.0
- joint joint2: limit lower=-3.0543261909900767 upper=3.0543261909900767 effort=197.23 velocity=2.6179938779914944 -> lower=-3.0543261909900767 upper=2.356194490192345 effort=197.23 velocity=3.141592653589793; origin xyz=0                          0.45                          -0.0305 rpy=0                         0                         3.1415926536 -> xyz=0.0                          0.850063                          0.0095 rpy=0.0                         0.0                         0.0
- joint joint3: limit lower=-3.0543261909900767 upper=3.0543261909900767 effort=79.79 velocity=3.141592653589793 -> lower=-6.283185307179586 upper=6.283185307179586 effort=79.79 velocity=3.141592653589793; origin xyz=0                          -0.267                          -0.075 rpy=-1.570796327                         0                         3.1415926536 -> xyz=0.0                          0.7915                          -0.0025 rpy=0.0                         0.0                         0.0
- joint joint4: limit lower=-3.0543261909900767 upper=3.0543261909900767 effort=79.79 velocity=3.141592653589793 -> lower=-6.283185307179586 upper=6.283185307179586 effort=79.79 velocity=3.141592653589793; origin xyz=0                          -0.114                          0.0835 rpy=1.570796327                         0                         0 -> xyz=0.0                          0.0865                          -0.072 rpy=-1.570796327                         0.0                         0.0
- joint joint5: limit lower=-3.7524578917878086 upper=3.7524578917878086 effort=79.79 velocity=3.141592653589793 -> lower=-6.283185307179586 upper=6.283185307179586 effort=79.79 velocity=3.141592653589793; origin xyz=0                          0.052                          0.085 rpy=-1.570796327                         0                         0 -> xyz=0.0                          0.0865                          0.072 rpy=-1.570796327                         0.0                         0.0
- joint tcp: origin xyz=0.0                          0.0                          0.0505 rpy=0.0                         0.0                         0.0 -> xyz=0.0                          0.0                          0.048 rpy=0.0                         0.0                         0.0

File: indy_description/urdf_files/opti5.urdf (robot description, URDF)
Before this commit: robot indy, 9 links, 8 joints
Joints:
- joint tcp: origin xyz=0.0                          0.0                          0.0605 rpy=0.0                         0.0                         0.0 -> xyz=0.0                          0.0                          0.054 rpy=0.0                         0.0                         0.0
