Commit message: update for Nuri5s

File: indy_description/urdf/indy.urdf.xacro (robot description, xacro)
@@ -11,5 +11,6 @@
     <xacro:arg name="gripper_dh_ag95" default="false"/>
     <xacro:property name="arg_indy_type" value="$(arg indy_type)"/>
-    <xacro:property name="config_indy_type" value="${arg_indy_type}"/>
+    <!-- NURI5s is a compatibility alias for the existing NURI4s model. -->
+    <xacro:property name="config_indy_type" value="${'nuri4s' if arg_indy_type == 'nuri5s' else arg_indy_type}"/>
     <!-- parameters -->
     <xacro:arg name="prefix" default="" />

File: indy_description/urdf_files/nuri5s.urdf (robot description, URDF)
Before this commit: robot indy, 9 links, 8 joints
Links:
- link link0: mass 4.986732 -> 2.861045494
- link link1: mass 20.116164 -> 3.167175036
- link link2: mass 26.414028 -> 4.29096783
- link link3: mass 15.498706 -> 2.018198648
- link link4: mass 13.487443 -> 1.882223023
- link link5: mass 9.0432 -> 1.507185922
- link link6: mass 1.320725 -> 0.634034296

File: indy_description/urdf_files/nuri5sdual.urdf (robot description, URDF)
Before this commit: robot indy, 18 links, 17 joints
Links:
- link left_arm_link0: mass 4.986732 -> 2.861045494
- link left_arm_link1: mass 20.116164 -> 3.167175036
- link left_arm_link2: mass 26.414028 -> 4.29096783
- link left_arm_link3: mass 15.498706 -> 2.018198648
- link left_arm_link4: mass 13.487443 -> 1.882223023
- link left_arm_link5: mass 9.0432 -> 1.507185922
- link left_arm_link6: mass 1.320725 -> 0.634034296
- link right_arm_link0: mass 4.986732 -> 2.861045494
- link right_arm_link1: mass 20.116164 -> 3.167175036
- link right_arm_link2: mass 26.414028 -> 4.29096783
- link right_arm_link3: mass 15.498706 -> 2.018198648
- link right_arm_link4: mass 13.487443 -> 1.882223023
- link right_arm_link5: mass 9.0432 -> 1.507185922
- link right_arm_link6: mass 1.320725 -> 0.634034296

Commit message: update for Nuri5s

File: indy_description/urdf/indy.urdf.xacro (robot description, xacro)
@@ -11,5 +11,6 @@
     <xacro:arg name="gripper_dh_ag95" default="false"/>
     <xacro:property name="arg_indy_type" value="$(arg indy_type)"/>
-    <xacro:property name="config_indy_type" value="${arg_indy_type}"/>
+    <!-- NURI5s is the compatibility name for the NURI4s model. -->
+    <xacro:property name="config_indy_type" value="${'nuri4s' if arg_indy_type == 'nuri5s' else arg_indy_type}"/>
     <!-- parameters -->
     <xacro:arg name="prefix" default="" />
