Commit message: update urdf files

File: indy_description/urdf/indy_macro.xacro (robot description, xacro)
@@ -27,5 +27,5 @@
                             indy_type == 'indyrp2_v2' or indy_type == 'indy12' or indy_type == 'indy12_v2' or
                             indy_type == 'nuri3s' or indy_type == 'nuri4s' or indy_type == 'nuri7c' or
-                            indy_type == 'nuri20c' or indy_type == 'opti5'}">
+                            indy_type == 'nuri20c' or indy_type == 'nuri30s' or indy_type == 'opti5'}">
             <xacro:property name="material_0" value="indy_white"/>
             <xacro:property name="material_1" value="indy_white"/>

File: indy_description/urdf_files/dual_icon3.urdf (robot description, URDF)
Before this commit: robot indy, 9 links, 8 joints
Links:
- removed link link0
- removed link link1
- removed link link2
- removed link link3
- removed link link4
- removed link link5
- removed link link6
- removed link tcp
- added link body_base, mass 5.726; collision mesh filename=file:///home/user/indy-ros2/install/indy_description/share/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; visual mesh filename=file:///home/user/indy-ros2/install/indy_description/share/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
- added link body_cover, mass 61.443; collision mesh filename=file:///home/user/indy-ros2/install/indy_description/share/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; visual mesh filename=file:///home/user/indy-ros2/install/indy_description/share/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
- added link body_frame, mass 23.464; collision mesh filename=file:///home/user/indy-ros2/install/indy_description/share/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; visual mesh filename=file:///home/user/indy-ros2/install/indy_description/share/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
- added link left_arm_link0, mass 6.568; collision mesh filename=file:///home/user/indy-ros2/install/indy_description/share/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; visual mesh filename=file:///home/user/indy-ros2/install/indy_description/share/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
- added link left_arm_link1, mass 2.983; collision mesh filename=file:///home/user/indy-ros2/install/indy_description/share/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; visual mesh filename=file:///home/user/indy-ros2/install/indy_description/share/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
- added link left_arm_link2, mass 5.667; collision mesh filename=file:///home/user/indy-ros2/install/indy_description/share/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; visual mesh filename=file:///home/user/indy-ros2/install/indy_description/share/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
- added link left_arm_link3, mass 2.922; collision mesh filename=file:///home/user/indy-ros2/install/indy_description/share/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; visual mesh filename=file:///home/user/indy-ros2/install/indy_description/share/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
- added link left_arm_link4, mass 3.269; collision mesh filename=file:///home/user/indy-ros2/install/indy_description/share/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; visual mesh filename=file:///home/user/indy-ros2/install/indy_description/share/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
- added link left_arm_link5, mass 1.67; collision mesh filename=file:///home/user/indy-ros2/install/indy_description/share/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; visual mesh filename=file:///home/user/indy-ros2/install/indy_description/share/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
- added link left_arm_link6, mass 0.272; collision mesh filename=file:///home/user/indy-ros2/install/indy_description/share/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; visual mesh filename=file:///home/user/indy-ros2/install/indy_description/share/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
- added link left_arm_tcp
- added link right_arm_link0, mass 6.568; collision mesh filename=file:///home/user/indy-ros2/install/indy_description/share/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; visual mesh filename=file:///home/user/indy-ros2/install/indy_description/share/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
- added link right_arm_link1, mass 2.983; collision mesh filename=file:///home/user/indy-ros2/install/indy_description/share/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; visual mesh filename=file:///home/user/indy-ros2/install/indy_description/share/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
- added link right_arm_link2, mass 5.667; collision mesh filename=file:///home/user/indy-ros2/install/indy_description/share/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; visual mesh filename=file:///home/user/indy-ros2/install/indy_description/share/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
- added link right_arm_link3, mass 2.922; collision mesh filename=file:///home/user/indy-ros2/install/indy_description/share/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; visual mesh filename=file:///home/user/indy-ros2/install/indy_description/share/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
- added link right_arm_link4, mass 3.269; collision mesh filename=file:///home/user/indy-ros2/install/indy_description/share/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; visual mesh filename=file:///home/user/indy-ros2/install/indy_description/share/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
- added link right_arm_link5, mass 1.67; collision mesh filename=file:///home/user/indy-ros2/install/indy_description/share/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; visual mesh filename=file:///home/user/indy-ros2/install/indy_description/share/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
- added link right_arm_link6, mass 0.272; collision mesh filename=file:///home/user/indy-ros2/install/indy_description/share/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; visual mesh filename=file:///home/user/indy-ros2/install/indy_description/share/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
- added link right_arm_tcp
Joints:
- removed joint joint0
- removed joint joint1
- removed joint joint2
- removed joint joint3
- removed joint joint4
- removed joint joint5
- removed joint tcp
- added joint base_frame: type revolute, parent body_base, child body_frame, origin xyz=0.0                          0.0                          0.0285 rpy=0.0                         0.0                         0.0, axis 0 0 1, limit lower=-3.141592653589793 upper=3.141592653589793 effort=1000.0 velocity=10.0
- added joint frame_cover: type fixed, parent body_frame, child body_cover, origin xyz=0.0                          0.0                          0.0116 rpy=0.0                         0.0                         0.0
- added joint left_arm_connect: type fixed, parent body_frame, child left_arm_link0, origin xyz=0.011367                          0.042157                          0.541659 rpy=-1.570796327                         0.0                         -0.261799388
- added joint left_arm_joint0: type revolute, parent left_arm_link0, child left_arm_link1, origin xyz=0.0                          0.0                          0.156 rpy=0.0                         0.0                         0.0, axis 0 0 1, limit lower=-2.9670597283903604 upper=2.9670597283903604 effort=431.97 velocity=7.853981633974483
- added joint left_arm_joint1: type revolute, parent left_arm_link1, child left_arm_link2, origin xyz=0.0                          0.0                          0.174 rpy=1.570796327                         0.0                         3.14159265, axis 0 0 1, limit lower=-1.9198621771937625 upper=2.0943951023931953 effort=431.97 velocity=7.853981633974483
- added joint left_arm_joint2: type revolute, parent left_arm_link2, child left_arm_link3, origin xyz=0.0                          0.26                          0.0 rpy=0.0                         0.0                         1.570796327, axis 0 0 1, limit lower=-3.4557519189487724 upper=1.0821041362364843 effort=197.23 velocity=9.16297857297023
- added joint left_arm_joint3: type revolute, parent left_arm_link3, child left_arm_link4, origin xyz=0.021                          0.0625                          0.0 rpy=-1.570796327                         1.570796327                         0.0, axis 0 0 1, limit lower=-3.490658503988659 upper=3.490658503988659 effort=79.79 velocity=10.471975511965978
- added joint left_arm_joint4: type revolute, parent left_arm_link4, child left_arm_link5, origin xyz=0.0                          0.0                          0.237 rpy=1.570796327                         -1.570796327                         -1.570796327, axis 0 0 1, limit lower=-2.059488517353309 upper=2.059488517353309 effort=79.79 velocity=10.471975511965978
- added joint left_arm_joint5: type revolute, parent left_arm_link5, child left_arm_link6, origin xyz=0.0685                          0.0                          0.0 rpy=1.570796327                         0.0                         1.570796327, axis 0 0 1, limit lower=-6.1086523819801535 upper=6.1086523819801535 effort=79.79 velocity=13.962634015954636
- added joint left_arm_tcp: type fixed, parent left_arm_link6, child left_arm_tcp, origin xyz=0.0                          0.0                          0.0 rpy=0.0                         0.0                         0.0
- added joint right_arm_connect: type fixed, parent body_frame, child right_arm_link0, origin xyz=0.011367                          -0.042157                          0.541659 rpy=1.570796327                         0.0                         0.261799388
- added joint right_arm_joint0: type revolute, parent right_arm_link0, child right_arm_link1, origin xyz=0.0                          0.0                          0.156 rpy=0.0                         0.0                         0.0, axis 0 0 1, limit lower=-2.9670597283903604 upper=2.9670597283903604 effort=431.97 velocity=7.853981633974483
- added joint right_arm_joint1: type revolute, parent right_arm_link1, child right_arm_link2, origin xyz=0.0                          0.0                          0.174 rpy=1.570796327                         0.0                         3.14159265, axis 0 0 1, limit lower=-1.9198621771937625 upper=2.0943951023931953 effort=431.97 velocity=7.853981633974483
- added joint right_arm_joint2: type revolute, parent right_arm_link2, child right_arm_link3, origin xyz=0.0                          0.26                          0.0 rpy=0.0                         0.0                         1.570796327, axis 0 0 1, limit lower=-3.4557519189487724 upper=1.0821041362364843 effort=197.23 velocity=9.16297857297023
- added joint right_arm_joint3: type revolute, parent right_arm_link3, child right_arm_link4, origin xyz=0.021                          0.0625                          0.0 rpy=-1.570796327                         1.570796327                         0.0, axis 0 0 1, limit lower=-3.490658503988659 upper=3.490658503988659 effort=79.79 velocity=10.471975511965978
- added joint right_arm_joint4: type revolute, parent right_arm_link4, child right_arm_link5, origin xyz=0.0                          0.0                          0.237 rpy=1.570796327                         -1.570796327                         -1.570796327, axis 0 0 1, limit lower=-2.059488517353309 upper=2.059488517353309 effort=79.79 velocity=10.471975511965978
- added joint right_arm_joint5: type revolute, parent right_arm_link5, child right_arm_link6, origin xyz=0.0685                          0.0                          0.0 rpy=1.570796327                         0.0                         1.570796327, axis 0 0 1, limit lower=-6.1086523819801535 upper=6.1086523819801535 effort=79.79 velocity=13.962634015954636
- added joint right_arm_tcp: type fixed, parent right_arm_link6, child right_arm_tcp, origin xyz=0.0                          0.0                          0.0 rpy=0.0                         0.0                         0.0
- joint global: child link0 -> body_base

File: indy_description/urdf_files/icon7l.urdf (robot description, URDF)
Before this commit: robot indy, 9 links, 8 joints
Joints:
- joint joint2: limit lower=-2.0943951023931953 upper=2.722713633111154 effort=197.23 velocity=6.806784082777885 -> lower=-3.6651914291880923 upper=1.1519173063162575 effort=197.23 velocity=6.806784082777885; origin xyz=0.0                          -0.463                          0.0 rpy=0.0                         0.0                         0.0 -> xyz=0.0                          -0.463                          0.0 rpy=0.0                         0.0                         1.570796327

File: indy_description/urdf_files/indy12_v2.urdf (robot description, URDF)
Before this commit: robot indy, 9 links, 8 joints
Joints:
- joint joint0: origin xyz=0                          0                          0.083 rpy=0                         0                         0 -> xyz=0                          0                          0.0815 rpy=0                         0                         0
- joint joint1: origin xyz=0                          -0.137                          0.2675 rpy=1.570796327                         -1.570796327                         0 -> xyz=0                          -0.1355                          0.2685 rpy=1.570796327                         -1.570796327                         0
- joint joint2: origin xyz=0.652                          0                          -0.0205 rpy=0                         0                         1.570796327 -> xyz=0.65                          0                          -0.0185 rpy=0                         0                         1.570796327
- joint joint3: origin xyz=0                          -0.21                          -0.10595 rpy=-1.570796327                         0                         3.14159265 -> xyz=0                          -0.187                          -0.1065 rpy=-1.570796327                         0                         3.14159265
- joint joint4: origin xyz=0                          -0.1305                          0.3628 rpy=-1.570796327                         0                         3.14159265 -> xyz=0                          -0.129                          0.363 rpy=-1.570796327                         0                         3.14159265
- joint joint5: origin xyz=0                          -0.075                          0.08 rpy=-1.570796327                         0                         3.14159265 -> xyz=0                          -0.074                          0.0795 rpy=-1.570796327                         0                         3.14159265
- joint tcp: origin xyz=0.0                          0.0                          0.09 rpy=0.0                         0.0                         0.0 -> xyz=0.0                          0.0                          0.085 rpy=0.0                         0.0                         0.0

File: indy_description/urdf_files/indy7_v2.urdf (robot description, URDF)
Before this commit: robot indy, 9 links, 8 joints
Joints:
- joint tcp: origin xyz=0.0                          0.0                          0.06 rpy=0.0                         0.0                         0.0 -> xyz=0.0                          0.0                          0.057 rpy=0.0                         0.0                         0.0

File: indy_description/urdf_files/indyrp2_v2.urdf (robot description, URDF)
Before this commit: robot indy, 10 links, 9 joints
Joints:
- joint tcp: origin xyz=0.0                          0.0                          0.06 rpy=0.0                         0.0                         0.0 -> xyz=0.0                          0.0                          0.057 rpy=0.0                         0.0                         0.0

File: indy_description/urdf_files/nuri20c.urdf (robot description, URDF)
Before this commit: robot indy, 9 links, 8 joints
Joints:
- joint joint1: axis 0 0 1 -> 0 0 -1

File: indy_description/urdf_files/nuri3s.urdf (robot description, URDF)
Before this commit: robot indy, 9 links, 8 joints
Joints:
- joint joint1: axis 0 0 1 -> 0 0 -1

File: indy_description/urdf_files/nuri4s.urdf (robot description, URDF)
Before this commit: robot indy, 9 links, 8 joints
Joints:
- joint joint1: axis 0 0 1 -> 0 0 -1
- joint joint2: axis 0 0 1 -> 0 0 -1
- joint joint4: axis 0 0 1 -> 0 0 -1

File: indy_description/urdf_files/nuri7c.urdf (robot description, URDF)
Before this commit: robot indy, 9 links, 8 joints
Joints:
- joint joint1: axis 0 0 1 -> 0 0 -1
