Commit message: Feat: Update Indy7 simulation files for Jazzy.

File: indy_description/urdf/indy_macro.xacro (robot description, xacro)
@@ -20,9 +20,8 @@
         transmission_hw_interface:=hardware_interface/PositionJointInterface
         sim_gazebo:=false">
-        <!-- initial_positions:=${dict(joint0=0.0,joint1=0.0,joint2=-1.57,joint3=0.0,joint4=-1.57,joint5=0.0)} -->
-        <!-- Load configuration data from the provided .yaml files -->
         <xacro:define_initialize initial_positions_file="${initial_positions_file}"
             visual_parameters_file="${visual_parameters_file}" indy_type="${indy_type}"/>
-        <xacro:if value="${ indy_type == 'indy7' or indy_type == 'indy7_v2' or indy_type == 'indyrp2' or
+        <xacro:if value="${ indy_type == 'indy7' or indy_type == 'indy7_v2' or indy_type
+                            == 'indyrp2' or
                             indy_type == 'indyrp2_v2' or indy_type == 'indy12' or indy_type == 'indy12_v2' or
                             indy_type == 'nuri3s' or indy_type == 'nuri4s' or indy_type == 'nuri7c' or
@@ -36,5 +35,4 @@
             <xacro:property name="material_2" value="indy_white"/>
         </xacro:if>
-        <!-- links -  main serial chain -->
         <xacro:macro name="define_link" params="link_name physic_name visual_name material gazebo_material">
             <link name="${prefix}${link_name}">
@@ -73,52 +71,4 @@
             </link>
         </xacro:macro>
-        <xacro:if value="${indy_type == 'dual_icon3'}">
-            <!--body-->
-            <xacro:define_link link_name="body_base" physic_name="body_base" visual_name="body_base" material="${material_0}" gazebo_material=""/>
-            <xacro:define_link link_name="body_frame" physic_name="body_frame" visual_name="body_frame" material="${material_0}" gazebo_material=""/>
-            <xacro:define_link link_name="body_cover" physic_name="body_cover" visual_name="body_cover" material="${material_2}" gazebo_material=""/>
-            <!-- icon3 - left -->
-            <xacro:define_link link_name="left_arm_link0" physic_name="left_arm_link0" visual_name="left_arm_link0" material="${material_0}" gazebo_material=""/>
-            <xacro:define_link link_name="left_arm_link1" physic_name="left_arm_link1" visual_name="left_arm_link1" material="${material_1}" gazebo_material=""/>
-            <xacro:define_link link_name="left_arm_link2" physic_name="left_arm_link2" visual_name="left_arm_link2" material="${material_1}" gazebo_material=""/>
-            <xacro:define_link link_name="left_arm_link3" physic_name="left_arm_link3" visual_name="left_arm_link3" material="${material_1}" gazebo_material=""/>
-            <xacro:define_link link_name="left_arm_link4" physic_name="left_arm_link4" visual_name="left_arm_link4" material="${material_1}" gazebo_material=""/>
-            <xacro:define_link link_name="left_arm_link5" physic_name="left_arm_link5" visual_name="left_arm_link5" material="${material_0}" gazebo_material=""/>
-            <xacro:define_link link_name="left_arm_link6" physic_name="left_arm_link6" visual_name="left_arm_link6" material="${material_0}" gazebo_material=""/>
-            <!-- icon3 - right -->
-            <xacro:define_link link_name="right_arm_link0" physic_name="right_arm_link0" visual_name="right_arm_link0" material="${material_0}" gazebo_material=""/>
-            <xacro:define_link link_name="right_arm_link1" physic_name="right_arm_link1" visual_name="right_arm_link1" material="${material_1}" gazebo_material=""/>
-            <xacro:define_link link_name="right_arm_link2" physic_name="right_arm_link2" visual_name="right_arm_link2" material="${material_1}" gazebo_material=""/>
-            <xacro:define_link link_name="right_arm_link3" physic_name="right_arm_link3" visual_name="right_arm_link3" material="${material_1}" gazebo_material=""/>
-            <xacro:define_link link_name="right_arm_link4" physic_name="right_arm_link4" visual_name="right_arm_link4" material="${material_1}" gazebo_material=""/>
-            <xacro:define_link link_name="right_arm_link5" physic_name="right_arm_link5" visual_name="right_arm_link5" material="${material_0}" gazebo_material=""/>
-            <xacro:define_link link_name="right_arm_link6" physic_name="right_arm_link6" visual_name="right_arm_link6" material="${material_0}" gazebo_material=""/>
-            <link name="${prefix}left_arm_tcp"/>
-            <link name="${prefix}right_arm_tcp"/>
-        </xacro:if>
-        <xacro:unless value="${indy_type == 'dual_icon3'}">
-            <xacro:define_link link_name="link0" physic_name="link0" visual_name="link0" material="${material_0}" gazebo_material=""/>
-            <xacro:define_link link_name="link1" physic_name="link1" visual_name="link1" material="${material_1}" gazebo_material=""/>
-            <xacro:define_link link_name="link2" physic_name="link2" visual_name="link2" material="${material_1}" gazebo_material=""/>
-            <xacro:define_link link_name="link3" physic_name="link3" visual_name="link3" material="${material_1}" gazebo_material=""/>
-            <xacro:define_link link_name="link4" physic_name="link4" visual_name="link4" material="${material_1}" gazebo_material=""/>
-            <xacro:define_link link_name="link5" physic_name="link5" visual_name="link5" material="${material_0}" gazebo_material=""/>
-            <xacro:if value="${indy_eye and not (indy_type == 'indyrp2' or indy_type == 'indyrp2_v2')}">
-                <xacro:define_link link_name="link6" physic_name="link6" visual_name="link6_eye" material="${material_0}" gazebo_material=""/>
-            </xacro:if>
-            <xacro:unless value="${indy_eye and not (indy_type == 'indyrp2' or indy_type == 'indyrp2_v2')}">
-                <xacro:define_link link_name="link6" physic_name="link6" visual_name="link6" material="${material_0}" gazebo_material=""/>
-            </xacro:unless>
-            <xacro:if value="${indy_type == 'indyrp2' or indy_type == 'indyrp2_v2'}">
-                <xacro:if value="${indy_eye}">
-                    <xacro:define_link link_name="link7" physic_name="link7" visual_name="link7_eye" material="${material_0}" gazebo_material=""/>
-                </xacro:if>
-                <xacro:unless value="${indy_eye}">
-                    <xacro:define_link link_name="link7" physic_name="link7" visual_name="link7" material="${material_0}" gazebo_material=""/>
-                </xacro:unless>
-            </xacro:if>
-            <link name="${prefix}tcp"/>
-        </xacro:unless>
-        <!-- joints -->
         <xacro:macro name="define_joint" params="joint_type joint_index parent_link child_link">
             <xacro:property name="config_joint_limit_parameters" value="${xacro.load_yaml(joint_limits_parameters_file)}"/>
@@ -128,5 +78,11 @@
             <xacro:property name="sec_limits" value="${config_joint_limit_parameters['joint_limits']}"/>
             <xacro:property name="sec_joint_axes" value="${config_joint_axes_parameters['joint_axes']}" />
-            <joint name="${prefix}${joint_index}" type="${joint_type}">
+            <xacro:if value="${joint_index == 'tcp'}">
+                <xacro:property name="j_name" value="${prefix}${joint_index}_joint"/>
+            </xacro:if>
+            <xacro:unless value="${joint_index == 'tcp'}">
+                <xacro:property name="j_name" value="${prefix}${joint_index}"/>
+            </xacro:unless>
+            <joint name="${j_name}" type="${joint_type}">
                 <parent link="${prefix}${parent_link}"/>
                 <child link="${prefix}${child_link}"/>
@@ -139,5 +95,4 @@
                         ${sec_kinematics[joint_index]['yaw']}"/>
                 <xacro:if value="${joint_type == 'revolute' or joint_type == 'continuous'}">
-                    <!-- Use configurable axis if available, fallback to default [0,0,1] -->
                     <xacro:if value="${joint_index in sec_joint_axes}">
                         <axis xyz="${sec_joint_axes[joint_index][0]} ${sec_joint_axes[joint_index][1]} ${sec_joint_axes[joint_index][2]}"/>
@@ -157,7 +112,46 @@
             </joint>
         </xacro:macro>
-       <xacro:if value="${indy_type == 'dual_icon3'}">
+        <xacro:if value="${indy_type == 'dual_icon3'}">
+            <xacro:define_link link_name="body_base" physic_name="body_base" visual_name="body_base" material="${material_0}" gazebo_material=""/>
+            <xacro:define_link link_name="body_frame" physic_name="body_frame" visual_name="body_frame" material="${material_0}" gazebo_material=""/>
+            <xacro:define_link link_name="body_cover" physic_name="body_cover" visual_name="body_cover" material="${material_2}" gazebo_material=""/>
+            <xacro:define_link link_name="left_arm_link0" physic_name="left_arm_link0" visual_name="left_arm_link0" material="${material_0}" gazebo_material=""/>
+            <xacro:define_link link_name="left_arm_link1" physic_name="left_arm_link1" visual_name="left_arm_link1" material="${material_1}" gazebo_material=""/>
+            <xacro:define_link link_name="left_arm_link2" physic_name="left_arm_link2" visual_name="left_arm_link2" material="${material_1}" gazebo_material=""/>
+            <xacro:define_link link_name="left_arm_link3" physic_name="left_arm_link3" visual_name="left_arm_link3" material="${material_1}" gazebo_material=""/>
+            <xacro:define_link link_name="left_arm_link4" physic_name="left_arm_link4" visual_name="left_arm_link4" material="${material_1}" gazebo_material=""/>
+            <xacro:define_link link_name="left_arm_link5" physic_name="left_arm_link5" visual_name="left_arm_link5" material="${material_0}" gazebo_material=""/>
+            <xacro:define_link link_name="left_arm_link6" physic_name="left_arm_link6" visual_name="left_arm_link6" material="${material_0}" gazebo_material=""/>
+            <xacro:define_link link_name="right_arm_link0" physic_name="right_arm_link0" visual_name="right_arm_link0" material="${material_0}" gazebo_material=""/>
+            <xacro:define_link link_name="right_arm_link1" physic_name="right_arm_link1" visual_name="right_arm_link1" material="${material_1}" gazebo_material=""/>
+            <xacro:define_link link_name="right_arm_link2" physic_name="right_arm_link2" visual_name="right_arm_link2" material="${material_1}" gazebo_material=""/>
+            <xacro:define_link link_name="right_arm_link3" physic_name="right_arm_link3" visual_name="right_arm_link3" material="${material_1}" gazebo_material=""/>
+            <xacro:define_link link_name="right_arm_link4" physic_name="right_arm_link4" visual_name="right_arm_link4" material="${material_1}" gazebo_material=""/>
+            <xacro:define_link link_name="right_arm_link5" physic_name="right_arm_link5" visual_name="right_arm_link5" material="${material_0}" gazebo_material=""/>
+            <xacro:define_link link_name="right_arm_link6" physic_name="right_arm_link6" visual_name="right_arm_link6" material="${material_0}" gazebo_material=""/>
+            <link name="${prefix}left_arm_tcp"/>
+            <link name="${prefix}right_arm_tcp"/>
+        </xacro:if>
+        <xacro:unless value="${indy_type == 'dual_icon3'}">
+            <xacro:define_link link_name="link0" physic_name="link0" visual_name="link0" material="${material_0}" gazebo_material=""/>
+            <xacro:define_link link_name="link1" physic_name="link1" visual_name="link1" material="${material_1}" gazebo_material=""/>
+            <xacro:define_link link_name="link2" physic_name="link2" visual_name="link2" material="${material_1}" gazebo_material=""/>
+            <xacro:define_link link_name="link3" physic_name="link3" visual_name="link3" material="${material_1}" gazebo_material=""/>
+            <xacro:define_link link_name="link4" physic_name="link4" visual_name="link4" material="${material_1}" gazebo_material=""/>
+            <xacro:define_link link_name="link5" physic_name="link5" visual_name="link5" material="${material_0}" gazebo_material=""/>
+            <xacro:if value="${indy_eye and not (indy_type == 'indyrp2' or indy_type == 'indyrp2_v2')}">
+                <xacro:define_link link_name="link6" physic_name="link6" visual_name="link6_eye" material="${material_0}" gazebo_material=""/>
+            </xacro:if>
+            <xacro:unless value="${indy_eye and not (indy_type == 'indyrp2' or indy_type == 'indyrp2_v2')}">
+                <xacro:define_link link_name="link6" physic_name="link6" visual_name="link6" material="${material_0}" gazebo_material=""/>
+            </xacro:unless>
+            <xacro:if value="${indy_type == 'indyrp2' or indy_type == 'indyrp2_v2'}">
+                <xacro:define_link link_name="link7" physic_name="link7" visual_name="link7" material="${material_0}" gazebo_material=""/>
+            </xacro:if>
+            <link name="${prefix}tcp"/>
+        </xacro:unless>
+        <xacro:if value="${indy_type == 'dual_icon3'}">
             <joint name="global" type="fixed">
-                <origin xyz="0 0 0" rpy="0 0 0"/>
+                <origin xyz="0.08 0 0" rpy="0 0 0"/>
                 <parent link="${parent}"/>
                 <child link="$(arg prefix)body_base"/>
@@ -201,6 +195,70 @@
                 <xacro:define_joint joint_type="fixed" joint_index="tcp" parent_link="link6" child_link="tcp"/>
             </xacro:unless>
-        </xacro:unless>
-        <!-- ros2 control -->
+            <link name="${prefix}zed2i_camera_link">
+                <visual>
+                    <origin xyz="0 0 0" rpy="0 0 0"/>
+                    <geometry>
+                        <box size="0.162 0.042 0.030"/>
+                    </geometry>
+                    <material name="${material_0}"/>
+                </visual>
+                <collision>
+                    <origin xyz="0 0 0" rpy="0 0 0"/>
+                    <geometry>
+                        <box size="0.162 0.042 0.030"/>
+                    </geometry>
+                </collision>
+                <inertial>
+                    <mass value="0.30"/>
+                    <origin xyz="0 0 0"/>
+                    <inertia ixx="0.0001" ixy="0" ixz="0" iyy="0.0001" iyz="0" izz="0.0001"/>
+                </inertial>
+            </link>
+            <joint name="${prefix}link6_to_zed2i_joint" type="fixed">
+                <parent link="${prefix}link6"/>
+                <child link="${prefix}zed2i_camera_link"/>
+                <origin xyz="0.08 0 0" rpy="0 0 -1.5708"/>
+            </joint>
+            <link name="${prefix}zed2i_camera_frame"/>
+            <joint name="${prefix}zed2i_camera_joint" type="fixed">
+                <parent link="${prefix}zed2i_camera_link"/>
+                <child link="${prefix}zed2i_camera_frame"/>
+                <origin xyz="0 0 0" rpy="0 -1.5708 -1.5708"/>
+            </joint>
+            <gazebo reference="${prefix}zed2i_camera_frame">
+                <sensor name="${prefix}zed2i_camera" type="camera">
+                    <update_rate>30</update_rate>
+                    <topic>${name}/zed2i/rgb</topic>
+                    <frame_id>${prefix}zed2i_camera_frame</frame_id>
+                    <camera>
+                        <horizontal_fov>1.5708</horizontal_fov>
+                        <image>
+                            <width>1280</width>
+                            <height>720</height>
+                        </image>
+                        <clip>
+                            <near>0.1</near>
+                            <far>10.0</far>
+                        </clip>
+                    </camera>
+                </sensor>
+                <sensor name="${prefix}zed2i_depth" type="depth_camera">
+                    <update_rate>30</update_rate>
+                    <topic>${name}/zed2i/depth</topic>
+                    <frame_id>${prefix}zed2i_camera_frame</frame_id>
+                    <camera>
+                        <horizontal_fov>1.5708</horizontal_fov>
+                        <image>
+                            <width>1280</width>
+                            <height>720</height>
+                        </image>
+                        <clip>
+                            <near>0.1</near>
+                            <far>10.0</far>
+                        </clip>
+                    </camera>
+                </sensor>
+            </gazebo>
+            </xacro:unless>
         <xacro:indy_ros2_control
             name="${name}"
@@ -209,6 +267,4 @@
             initial_positions="${initial_positions}"
             sim_gazebo="${sim_gazebo}"/>
-        <!-- Add URDF transmission elements (for ros_control) -->
-        <!-- <xacro:indy_transmission prefix="${prefix}" hw_interface="${transmission_hw_interface}" indy_type="${indy_type}"/> -->
-    </xacro:macro>
+        </xacro:macro>
 </robot>

File: indy_description/urdf_files/indy7.urdf (robot description, URDF)
Before this commit: robot indy, 9 links, 8 joints
Joints:
- removed joint tcp
- added joint tcp_joint: type fixed, parent link6, child tcp, origin xyz=0.0                          0.0                          0.06 rpy=0.0                         0.0                         0.0

Commit message: add indy12v3, nuri12c, update parameters

File: indy_description/urdf/indy_macro.xacro (robot description, xacro)
@@ -25,7 +25,7 @@
             visual_parameters_file="${visual_parameters_file}" indy_type="${indy_type}"/>
         <xacro:if value="${ indy_type == 'indy7' or indy_type == 'indy7_v2' or indy_type == 'indy7_v3' or indy_type == 'indyrp2' or
-                            indy_type == 'indyrp2_v2' or indy_type == 'indy12' or indy_type == 'indy12_v2' or
-                            indy_type == 'nuri3s' or indy_type == 'nuri4s' or indy_type == 'nuri7c' or
-                            indy_type == 'nuri20c' or indy_type == 'nuri30s' or indy_type == 'opti5'}">
+                            indy_type == 'indyrp2_v2' or indy_type == 'indy12' or indy_type == 'indy12_v2' or indy_type == 'indy12_v3' or
+                            indy_type == 'nuri3s' or indy_type == 'nuri4s' or indy_type == 'nuri7c' or indy_type == 'nuri12c' or
+                            indy_type == 'nuri20c' or indy_type == 'nuri30' or indy_type == 'opti5'}">
             <xacro:property name="material_0" value="indy_white"/>
             <xacro:property name="material_1" value="indy_white"/>
@@ -42,6 +42,9 @@
                 <xacro:property name="sec_inertia_parameters" value="${config_physical_parameters['inertia_parameters']}" />
                 <xacro:if value="${visual_name != ''}">
+                    <xacro:property name="visual_link_entry" value="${sec_mesh_files[visual_name]}"/>
+                    <xacro:property name="visual_origin_xyz" value="${visual_link_entry['visual_origin']['xyz'] if 'visual_origin' in visual_link_entry else '0 0 0'}"/>
+                    <xacro:property name="visual_origin_rpy" value="${visual_link_entry['visual_origin']['rpy'] if 'visual_origin' in visual_link_entry else '0 0 0'}"/>
                     <visual>
-                        <origin xyz="0 0 0" rpy="0 0 0"/>
+                        <origin xyz="${visual_origin_xyz}" rpy="${visual_origin_rpy}"/>
                         <geometry>
                             <xacro:get_mesh name="${visual_name}" type="visual"/>
@@ -50,5 +53,5 @@
                     </visual>
                     <collision>
-                        <origin xyz="0 0 0" rpy="0 0 0"/>
+                        <origin xyz="${visual_origin_xyz}" rpy="${visual_origin_rpy}"/>
                         <geometry>
                             <xacro:get_mesh name="${visual_name}" type="collision"/>

File: indy_description/urdf_files/indy12_v2.urdf (robot description, URDF)
Before this commit: robot indy, 9 links, 8 joints
Links:
- link link2: mass 13.86898329 -> 14.27904794
