Commit message: add indy12v3, nuri12c, update parameters

File: indy_description/urdf/indy_macro.xacro (robot description, xacro)
@@ -25,7 +25,7 @@
             visual_parameters_file="${visual_parameters_file}" indy_type="${indy_type}"/>
         <xacro:if value="${ indy_type == 'indy7' or indy_type == 'indy7_v2' or indy_type == 'indy7_v3' or indy_type == 'indyrp2' or
-                            indy_type == 'indyrp2_v2' or indy_type == 'indy12' or indy_type == 'indy12_v2' or
-                            indy_type == 'nuri3s' or indy_type == 'nuri4s' or indy_type == 'nuri7c' or
-                            indy_type == 'nuri20c' or indy_type == 'nuri30s' or indy_type == 'opti5'}">
+                            indy_type == 'indyrp2_v2' or indy_type == 'indy12' or indy_type == 'indy12_v2' or indy_type == 'indy12_v3' or
+                            indy_type == 'nuri3s' or indy_type == 'nuri4s' or indy_type == 'nuri7c' or indy_type == 'nuri12c' or
+                            indy_type == 'nuri20c' or indy_type == 'nuri30' or indy_type == 'opti5'}">
             <xacro:property name="material_0" value="indy_white"/>
             <xacro:property name="material_1" value="indy_white"/>
@@ -42,6 +42,9 @@
                 <xacro:property name="sec_inertia_parameters" value="${config_physical_parameters['inertia_parameters']}" />
                 <xacro:if value="${visual_name != ''}">
+                    <xacro:property name="visual_link_entry" value="${sec_mesh_files[visual_name]}"/>
+                    <xacro:property name="visual_origin_xyz" value="${visual_link_entry['visual_origin']['xyz'] if 'visual_origin' in visual_link_entry else '0 0 0'}"/>
+                    <xacro:property name="visual_origin_rpy" value="${visual_link_entry['visual_origin']['rpy'] if 'visual_origin' in visual_link_entry else '0 0 0'}"/>
                     <visual>
-                        <origin xyz="0 0 0" rpy="0 0 0"/>
+                        <origin xyz="${visual_origin_xyz}" rpy="${visual_origin_rpy}"/>
                         <geometry>
                             <xacro:get_mesh name="${visual_name}" type="visual"/>
@@ -50,5 +53,5 @@
                     </visual>
                     <collision>
-                        <origin xyz="0 0 0" rpy="0 0 0"/>
+                        <origin xyz="${visual_origin_xyz}" rpy="${visual_origin_rpy}"/>
                         <geometry>
                             <xacro:get_mesh name="${visual_name}" type="collision"/>

File: indy_description/urdf_files/dual_icon3.urdf (robot description, URDF)
Before this commit: robot indy, 20 links, 19 joints
Joints:
- removed joint left_arm_tcp
- removed joint right_arm_tcp
- added joint left_arm_tcp_fixed: type fixed, parent left_arm_link6, child left_arm_tcp, origin xyz=0.0                          0.0                          0.0 rpy=0.0                         0.0                         0.0
- added joint right_arm_tcp_fixed: type fixed, parent right_arm_link6, child right_arm_tcp, origin xyz=0.0                          0.0                          0.0 rpy=0.0                         0.0                         0.0

File: indy_description/urdf_files/icon3.urdf (robot description, URDF)
Before this commit: robot indy, 9 links, 8 joints
Joints:
- removed joint tcp
- added joint tcp_fixed: type fixed, parent link6, child tcp, origin xyz=0.0                          0.0                          0.0 rpy=0.0                         0.0                         0.0

File: indy_description/urdf_files/icon7l.urdf (robot description, URDF)
Before this commit: robot indy, 9 links, 8 joints
Joints:
- removed joint tcp
- added joint tcp_fixed: type fixed, parent link6, child tcp, origin xyz=0.0                          0.0                          0.0 rpy=0.0                         0.0                         0.0

File: indy_description/urdf_files/indy12.urdf (robot description, URDF)
Before this commit: robot indy, 9 links, 8 joints
Joints:
- removed joint tcp
- added joint tcp_fixed: type fixed, parent link6, child tcp, origin xyz=0.0                          0.0                          0.056 rpy=0.0                         0.0                         0.0

File: indy_description/urdf_files/indy12_v2.urdf (robot description, URDF)
Before this commit: robot indy, 9 links, 8 joints
Links:
- link link2: mass 13.86898329 -> 14.27904794
Joints:
- removed joint tcp
- added joint tcp_fixed: type fixed, parent link6, child tcp, origin xyz=0.0                          0.0                          0.085 rpy=0.0                         0.0                         0.0

File: indy_description/urdf_files/indy7.urdf (robot description, URDF)
Before this commit: robot indy, 9 links, 8 joints
Joints:
- removed joint tcp
- added joint tcp_fixed: type fixed, parent link6, child tcp, origin xyz=0.0                          0.0                          0.06 rpy=0.0                         0.0                         0.0

File: indy_description/urdf_files/indy7_eye.urdf (robot description, URDF)
Before this commit: robot indy, 9 links, 8 joints
Joints:
- removed joint tcp
- added joint tcp_fixed: type fixed, parent link6, child tcp, origin xyz=0.0                          0.0                          0.06 rpy=0.0                         0.0                         0.0

File: indy_description/urdf_files/indy7_v2.urdf (robot description, URDF)
Before this commit: robot indy, 9 links, 8 joints
Joints:
- removed joint tcp
- added joint tcp_fixed: type fixed, parent link6, child tcp, origin xyz=0.0                          0.0                          0.0505 rpy=0.0                         0.0                         0.0

File: indy_description/urdf_files/indy7_v3.urdf (robot description, URDF)
Before this commit: robot indy, 9 links, 8 joints
Joints:
- removed joint tcp
- added joint tcp_fixed: type fixed, parent link6, child tcp, origin xyz=0.0                          0.0                          0.0557 rpy=0.0                         0.0                         0.0

File: indy_description/urdf_files/indyrp2.urdf (robot description, URDF)
Before this commit: robot indy, 10 links, 9 joints
Joints:
- removed joint tcp
- added joint tcp_fixed: type fixed, parent link7, child tcp, origin xyz=0.0                          0.0                          0.06 rpy=0.0                         0.0                         0.0

File: indy_description/urdf_files/indyrp2_eye.urdf (robot description, URDF)
Before this commit: robot indy, 10 links, 9 joints
Joints:
- removed joint tcp
- added joint tcp_fixed: type fixed, parent link7, child tcp, origin xyz=0.0                          0.0                          0.06 rpy=0.0                         0.0                         0.0

File: indy_description/urdf_files/indyrp2_v2.urdf (robot description, URDF)
Before this commit: robot indy, 10 links, 9 joints
Joints:
- removed joint tcp
- added joint tcp_fixed: type fixed, parent link7, child tcp, origin xyz=0.0                          0.0                          0.0515 rpy=0.0                         0.0                         0.0

File: indy_description/urdf_files/nuri20c.urdf (robot description, URDF)
Before this commit: robot indy, 9 links, 8 joints
Joints:
- removed joint tcp
- added joint tcp_fixed: type fixed, parent link6, child tcp, origin xyz=0.0                          0.0                          0.04 rpy=0.0                         0.0                         0.0

File: indy_description/urdf_files/nuri30s.urdf (robot description, URDF)
Before this commit: robot indy, 9 links, 8 joints
Joints:
- removed joint tcp
- added joint tcp_fixed: type fixed, parent link6, child tcp, origin xyz=0.0                          0.0                          0.048 rpy=0.0                         0.0                         0.0

File: indy_description/urdf_files/nuri3s.urdf (robot description, URDF)
Before this commit: robot indy, 9 links, 8 joints
Joints:
- removed joint tcp
- added joint tcp_fixed: type fixed, parent link6, child tcp, origin xyz=0.0                          0.0                          0.0285 rpy=0.0                         0.0                         0.0

File: indy_description/urdf_files/nuri4s.urdf (robot description, URDF)
Before this commit: robot indy, 9 links, 8 joints
Joints:
- removed joint tcp
- added joint tcp_fixed: type fixed, parent link6, child tcp, origin xyz=0.0                          0.0                          0.0285 rpy=0.0                         0.0                         0.0

File: indy_description/urdf_files/nuri7c.urdf (robot description, URDF)
Before this commit: robot indy, 9 links, 8 joints
Joints:
- removed joint tcp
- added joint tcp_fixed: type fixed, parent link6, child tcp, origin xyz=0.0                          0.0                          0.054 rpy=0.0                         0.0                         0.0

File: indy_description/urdf_files/opti5.urdf (robot description, URDF)
Before this commit: robot indy, 9 links, 8 joints
Joints:
- removed joint tcp
- added joint tcp_fixed: type fixed, parent link6, child tcp, origin xyz=0.0                          0.0                          0.054 rpy=0.0                         0.0                         0.0

Commit message: update physical_param for indy eye

File: indy_description/urdf/indy_macro.xacro (robot description, xacro)
@@ -36,4 +36,6 @@
             <xacro:property name="material_2" value="indy_white"/>
         </xacro:if>
+        <xacro:property name="supports_link6_eye" value="${indy_type == 'indy7' or indy_type == 'indy7_v2' or indy_type == 'indy7_v3' or indy_type == 'indy12_v3'}"/>
+        <xacro:property name="supports_link7_eye" value="${indy_type == 'indyrp2' or indy_type == 'indyrp2_v2'}"/>
         <!-- links -  main serial chain -->
         <xacro:macro name="define_link" params="link_name physic_name visual_name material gazebo_material">
@@ -107,13 +109,16 @@
             <xacro:define_link link_name="link4" physic_name="link4" visual_name="link4" material="${material_1}" gazebo_material=""/>
             <xacro:define_link link_name="link5" physic_name="link5" visual_name="link5" material="${material_0}" gazebo_material=""/>
-            <xacro:if value="${indy_eye and (indy_type == 'indy7' or indy_type == 'indy7_v2' or indy_type == 'indy7_v3' or indy_type == 'indy12_v3')}">
-                <xacro:define_link link_name="link6" physic_name="link6" visual_name="link6_eye" material="${material_0}" gazebo_material=""/>
-            </xacro:if>
-            <xacro:unless value="${indy_eye and (indy_type == 'indy7' or indy_type == 'indy7_v2' or indy_type == 'indy7_v3' or indy_type == 'indy12_v3')}">
+            <xacro:if value="${indy_eye and supports_link6_eye}">
+                <xacro:define_link link_name="link6" physic_name="link6_eye" visual_name="link6_eye" material="${material_0}" gazebo_material=""/>
+            </xacro:if>
+            <xacro:unless value="${indy_eye}">
                 <xacro:define_link link_name="link6" physic_name="link6" visual_name="link6" material="${material_0}" gazebo_material=""/>
             </xacro:unless>
+            <xacro:if value="${indy_eye and supports_link7_eye}">
+                <xacro:define_link link_name="link6" physic_name="link6" visual_name="link6" material="${material_0}" gazebo_material=""/>
+            </xacro:if>
             <xacro:if value="${indy_type == 'indyrp2' or indy_type == 'indyrp2_v2'}">
                 <xacro:if value="${indy_eye}">
-                    <xacro:define_link link_name="link7" physic_name="link7" visual_name="link7_eye" material="${material_0}" gazebo_material=""/>
+                    <xacro:define_link link_name="link7" physic_name="link7_eye" visual_name="link7_eye" material="${material_0}" gazebo_material=""/>
                 </xacro:if>
                 <xacro:unless value="${indy_eye}">
