Commit message: add nuri50

File: indy_description/urdf/indy_macro.xacro (robot description, xacro)
@@ -27,5 +27,5 @@
                             indy_type == 'indyrp2_v2' or indy_type == 'indy12' or indy_type == 'indy12_v2' or indy_type == 'indy12_v3' or
                             indy_type == 'nuri3s' or indy_type == 'nuri4s' or indy_type == 'nuri5s' or indy_type == 'nuri7c' or indy_type == 'nuri12c' or
-                            indy_type == 'nuri20c' or indy_type == 'nuri30' or indy_type == 'nuri5sdual' or
+                            indy_type == 'nuri20c' or indy_type == 'nuri30' or indy_type == 'nuri50' or indy_type == 'nuri5sdual' or
                             indy_type == 'opti5' or indy_type == 'opti3'}">
             <xacro:property name="material_0" value="indy_white"/>
@@ -160,5 +160,5 @@
                         <axis xyz="0 0 1"/>
                     </xacro:unless>
-                    <dynamics damping="0.1" friction="10.0"/>
+                    <dynamics damping="${sec_limits[joint_index]['damping']}" friction="${sec_limits[joint_index]['friction']}"/>
                 </xacro:if>
                 <xacro:if value="${joint_type == 'revolute'}">
