Commit message: humble

File: indy_description/urdf/indy.ros2_control.xacro (robot description, xacro)
@@ -5,4 +5,5 @@
         indy_type
         prefix
+        initial_positions
         sim_gazebo:=false">
         <ros2_control name="${name}" type="system">
@@ -26,6 +27,12 @@
                     <param name="max">3.15</param>
                 </command_interface>
-                <state_interface name="position"/>
-                <state_interface name="velocity"/>
+                <!-- <state_interface name="position"/> -->
+                <state_interface name="position">
+                    <param name="initial_value">${initial_positions['joint0']}</param>
+                </state_interface>
+                <!-- <state_interface name="velocity"/> -->
+                <state_interface name="velocity">
+                    <param name="initial_value">0.0</param>
+                </state_interface>
                 <state_interface name="effort"/>
             </joint>
@@ -39,12 +46,17 @@
                     <param name="max">3.15</param>
                 </command_interface>
-                <state_interface name="position"/>
-                <state_interface name="velocity"/>
+                <!-- <state_interface name="position"/> -->
+                <state_interface name="position">
+                    <param name="initial_value">${initial_positions['joint1']}</param>
+                </state_interface>
+                <state_interface name="velocity">
+                    <param name="initial_value">0.0</param>
+                </state_interface>
                 <state_interface name="effort"/>
             </joint>
             <joint name="${prefix}joint2">
                 <command_interface name="position">
-                    <param name="min">{-pi}</param>
-                    <param name="max">{pi}</param>
+                    <param name="min">{-2*pi}</param>
+                    <param name="max">{2*pi}</param>
                 </command_interface>
                 <command_interface name="velocity">
@@ -52,6 +64,11 @@
                     <param name="max">3.15</param>
                 </command_interface>
-                <state_interface name="position"/>
-                <state_interface name="velocity"/>
+                <!-- <state_interface name="position"/> -->
+                <state_interface name="position">
+                    <param name="initial_value">${initial_positions['joint2']}</param>
+                </state_interface>
+                <state_interface name="velocity">
+                    <param name="initial_value">0.0</param>
+                </state_interface>
                 <state_interface name="effort"/>
             </joint>
@@ -65,6 +82,11 @@
                     <param name="max">3.15</param>
                 </command_interface>
-                <state_interface name="position"/>
-                <state_interface name="velocity"/>
+                <!-- <state_interface name="position"/> -->
+                <state_interface name="position">
+                    <param name="initial_value">${initial_positions['joint3']}</param>
+                </state_interface>
+                <state_interface name="velocity">
+                    <param name="initial_value">0.0</param>
+                </state_interface>
                 <state_interface name="effort"/>
             </joint>
@@ -78,6 +100,11 @@
                     <param name="max">3.15</param>
                 </command_interface>
-                <state_interface name="position"/>
-                <state_interface name="velocity"/>
+                <!-- <state_interface name="position"/> -->
+                <state_interface name="position">
+                    <param name="initial_value">${initial_positions['joint4']}</param>
+                </state_interface>
+                <state_interface name="velocity">
+                    <param name="initial_value">0.0</param>
+                </state_interface>
                 <state_interface name="effort"/>
             </joint>
@@ -91,6 +118,11 @@
                     <param name="max">3.15</param>
                 </command_interface>
-                <state_interface name="position"/>
-                <state_interface name="velocity"/>
+                <!-- <state_interface name="position"/> -->
+                <state_interface name="position">
+                    <param name="initial_value">${initial_positions['joint5']}</param>
+                </state_interface>
+                <state_interface name="velocity">
+                    <param name="initial_value">0.0</param>
+                </state_interface>
                 <state_interface name="effort"/>
             </joint>
@@ -105,10 +137,11 @@
                         <param name="max">3.15</param>
                     </command_interface>
-                    <!-- <state_interface name="position">
-                        <param name="initial_value">${initial_positions['joint0']}</param>
-                    </state_interface> -->
-                    <!-- <param name="initial_position">0</param> -->
-                    <state_interface name="position"/>
-                    <state_interface name="velocity"/>
+                    <!-- <state_interface name="position"/> -->
+                    <state_interface name="position">
+                        <param name="initial_value">${initial_positions['joint6']}</param>
+                    </state_interface>
+                    <state_interface name="velocity">
+                        <param name="initial_value">0.0</param>
+                    </state_interface>
                     <state_interface name="effort"/>
                 </joint>

File: indy_description/urdf/indy.urdf.xacro (robot description, xacro)
@@ -14,4 +14,5 @@
     <xacro:arg name="physical_params" default="$(find indy_description)/urdf/config/$(arg indy_type)/physical_parameters.yaml"/>
     <xacro:arg name="visual_params" default="$(find indy_description)/urdf/config/$(arg indy_type)/visual_parameters.yaml"/>
+    <xacro:arg name="initial_positions" default="$(find indy_description)/urdf/config/initial_positions.yaml"/>
     <xacro:arg name="transmission_hw_interface" default=""/>
     <xacro:arg name="sim_gazebo" default="false" />
@@ -31,4 +32,5 @@
         visual_parameters_file="$(arg visual_params)"
         transmission_hw_interface="$(arg transmission_hw_interface)"
+        initial_positions_file="$(arg initial_positions)"
         sim_gazebo="$(arg sim_gazebo)"
         >

File: indy_description/urdf/indy_common.xacro (robot description, xacro)
@@ -8,9 +8,9 @@
         </inertial>
     </xacro:macro>
-    <xacro:macro name="get_visual_params" params="name:=^ type:=^">
+    <xacro:macro name="get_visual_params" params="name:=^ type:=^" >
         <xacro:property name="visual_params" value="${sec_mesh_files[name][type]}" scope="parent"/>
     </xacro:macro>
     <!-- Get mesh files -->
-    <xacro:macro name="get_mesh_path" params="name:=^ type:=^">
+    <xacro:macro name="get_mesh_path" params="name:=^ type:=^" >
         <xacro:get_visual_params />
         <!--RVIZ2-->
@@ -21,14 +21,20 @@
         <xacro:property name="mesh" value="file://$(find ${visual_params['mesh']['package']})/${visual_params['mesh']['path']}" scope="parent"/>
     </xacro:macro>
-    <xacro:macro name="get_mesh" params="name type">
+    <xacro:macro name="get_mesh" params="name type" >
         <xacro:get_mesh_path/>
         <mesh filename="${mesh}"/>
     </xacro:macro>
-    <xacro:macro name="read_model_data" params="joint_limits_parameters_file kinematics_parameters_file physical_parameters_file visual_parameters_file indy_type">
+    <xacro:macro name="read_model_data" params="joint_limits_parameters_file
+        kinematics_parameters_file
+        physical_parameters_file
+        visual_parameters_file
+        initial_positions_file
+        indy_type">
         <!-- Read .yaml files from disk, load content into properties -->
-        <xacro:property name="config_joint_limit_parameters" value="${load_yaml(joint_limits_parameters_file)}"/>
-        <xacro:property name="config_kinematics_parameters" value="${load_yaml(kinematics_parameters_file)}"/>
-        <xacro:property name="config_physical_parameters" value="${load_yaml(physical_parameters_file)}"/>
-        <xacro:property name="config_visual_parameters" value="${load_yaml(visual_parameters_file)}"/>
+        <xacro:property name="config_joint_limit_parameters" value="${xacro.load_yaml(joint_limits_parameters_file)}"/>
+        <xacro:property name="config_kinematics_parameters" value="${xacro.load_yaml(kinematics_parameters_file)}"/>
+        <xacro:property name="config_physical_parameters" value="${xacro.load_yaml(physical_parameters_file)}"/>
+        <xacro:property name="config_visual_parameters" value="${xacro.load_yaml(visual_parameters_file)}"/>
+        <xacro:property name="initial_positions_parameters" value="${xacro.load_yaml(initial_positions_file)}"/>
         <!-- Extract subsections from yaml dictionaries -->
         <xacro:property name="sec_limits" value="${config_joint_limit_parameters['joint_limits']}"/>
@@ -157,5 +163,4 @@
         <xacro:property name="inertia_link6_ixz" value="${sec_inertia_parameters['link6']['ixz']}" scope="parent"/>
         <!--indyrp2 with 7 DOF-->
-        <!-- <xacro:if value="${indy_type == 'indyrp2'}"> -->
         <xacro:if value="${indy_type == 'indyrp2' or indy_type == 'indyrp2_v2'}">
             <xacro:property name="joint6_lower_limit" value="${sec_limits['joint6']['min_position']}" scope="parent"/>
@@ -176,5 +181,9 @@
             <xacro:property name="inertia_link7_iyz" value="${sec_inertia_parameters['link7']['iyz']}" scope="parent"/>
             <xacro:property name="inertia_link7_ixz" value="${sec_inertia_parameters['link7']['ixz']}" scope="parent"/>
+            <xacro:property name="initial_positions" value="${initial_positions_parameters['7dof']}" scope="parent"/>
         </xacro:if>
+        <xacro:unless value="${indy_type == 'indyrp2' or indy_type == 'indyrp2_v2'}">
+            <xacro:property name="initial_positions" value="${initial_positions_parameters['6dof']}" scope="parent"/>
+        </xacro:unless>
     </xacro:macro>
 </robot>

File: indy_description/urdf/indy_macro.xacro (robot description, xacro)
@@ -16,6 +16,8 @@
         physical_parameters_file
         visual_parameters_file
+        initial_positions_file
         transmission_hw_interface:=hardware_interface/PositionJointInterface
         sim_gazebo:=false">
+        <!-- initial_positions:=${dict(joint0=0.0,joint1=0.0,joint2=-1.57,joint3=0.0,joint4=-1.57,joint5=0.0)} -->
         <!-- Load configuration data from the provided .yaml files -->
         <xacro:read_model_data
@@ -24,4 +26,5 @@
             physical_parameters_file="${physical_parameters_file}"
             visual_parameters_file="${visual_parameters_file}"
+            initial_positions_file="${initial_positions_file}"
             indy_type="${indy_type}"/>
         <xacro:property name="indy_material" value="metal_white"/>
@@ -298,4 +301,5 @@
             indy_type="${indy_type}"
             prefix="${prefix}"
+            initial_positions="${initial_positions}"
             sim_gazebo="${sim_gazebo}"/>
         <!-- Add URDF transmission elements (for ros_control) -->

Commit message: foxy no roscom version release

File: indy_description/urdf/indy.ros2_control.xacro (robot description, xacro)
@@ -45,6 +45,6 @@
             <joint name="${prefix}joint2">
                 <command_interface name="position">
-                    <param name="min">{-pi}</param>
-                    <param name="max">{pi}</param>
+                    <param name="min">{-2*pi}</param>
+                    <param name="max">{2*pi}</param>
                 </command_interface>
                 <command_interface name="velocity">
@@ -105,8 +105,4 @@
                         <param name="max">3.15</param>
                     </command_interface>
-                    <!-- <state_interface name="position">
-                        <param name="initial_value">${initial_positions['joint0']}</param>
-                    </state_interface> -->
-                    <!-- <param name="initial_position">0</param> -->
                     <state_interface name="position"/>
                     <state_interface name="velocity"/>

File: indy_description/urdf/indy_common.xacro (robot description, xacro)
@@ -25,5 +25,9 @@
         <mesh filename="${mesh}"/>
     </xacro:macro>
-    <xacro:macro name="read_model_data" params="joint_limits_parameters_file kinematics_parameters_file physical_parameters_file visual_parameters_file indy_type">
+    <xacro:macro name="read_model_data" params="joint_limits_parameters_file
+	    kinematics_parameters_file
+	    physical_parameters_file
+	    visual_parameters_file
+	    indy_type">
         <!-- Read .yaml files from disk, load content into properties -->
         <xacro:property name="config_joint_limit_parameters" value="${load_yaml(joint_limits_parameters_file)}"/>
@@ -157,5 +161,4 @@
         <xacro:property name="inertia_link6_ixz" value="${sec_inertia_parameters['link6']['ixz']}" scope="parent"/>
         <!--indyrp2 with 7 DOF-->
-        <!-- <xacro:if value="${indy_type == 'indyrp2'}"> -->
         <xacro:if value="${indy_type == 'indyrp2' or indy_type == 'indyrp2_v2'}">
             <xacro:property name="joint6_lower_limit" value="${sec_limits['joint6']['min_position']}" scope="parent"/>
