Commit message: update for foxy

File: indy_description/urdf/indy.ros2_control.xacro (robot description, xacro)
@@ -5,5 +5,4 @@
         indy_type
         prefix
-        initial_positions
         sim_gazebo:=false">
         <ros2_control name="${name}" type="system">
@@ -27,13 +26,7 @@
                     <param name="max">3.15</param>
                 </command_interface>
-                <!-- <state_interface name="position"/> -->
-                <state_interface name="position">
-                    <param name="initial_value">${initial_positions['joint0']}</param>
-                </state_interface>
-                <!-- <state_interface name="velocity"/> -->
-                <state_interface name="velocity">
-                    <param name="initial_value">0.0</param>
-                </state_interface>
-                <state_interface name="effort"/>
+                <state_interface name="position"/>
+                <state_interface name="velocity"/>
+                <!-- <state_interface name="effort"/> -->
             </joint>
             <joint name="${prefix}joint1">
@@ -46,12 +39,7 @@
                     <param name="max">3.15</param>
                 </command_interface>
-                <!-- <state_interface name="position"/> -->
-                <state_interface name="position">
-                    <param name="initial_value">${initial_positions['joint1']}</param>
-                </state_interface>
-                <state_interface name="velocity">
-                    <param name="initial_value">0.0</param>
-                </state_interface>
-                <state_interface name="effort"/>
+                <state_interface name="position"/>
+                <state_interface name="velocity"/>
+                <!-- <state_interface name="effort"/> -->
             </joint>
             <joint name="${prefix}joint2">
@@ -64,12 +52,7 @@
                     <param name="max">3.15</param>
                 </command_interface>
-                <!-- <state_interface name="position"/> -->
-                <state_interface name="position">
-                    <param name="initial_value">${initial_positions['joint2']}</param>
-                </state_interface>
-                <state_interface name="velocity">
-                    <param name="initial_value">0.0</param>
-                </state_interface>
-                <state_interface name="effort"/>
+                <state_interface name="position"/>
+                <state_interface name="velocity"/>
+                <!-- <state_interface name="effort"/> -->
             </joint>
             <joint name="${prefix}joint3">
@@ -82,12 +65,7 @@
                     <param name="max">3.15</param>
                 </command_interface>
-                <!-- <state_interface name="position"/> -->
-                <state_interface name="position">
-                    <param name="initial_value">${initial_positions['joint3']}</param>
-                </state_interface>
-                <state_interface name="velocity">
-                    <param name="initial_value">0.0</param>
-                </state_interface>
-                <state_interface name="effort"/>
+                <state_interface name="position"/>
+                <state_interface name="velocity"/>
+                <!-- <state_interface name="effort"/> -->
             </joint>
             <joint name="${prefix}joint4">
@@ -100,12 +78,7 @@
                     <param name="max">3.15</param>
                 </command_interface>
-                <!-- <state_interface name="position"/> -->
-                <state_interface name="position">
-                    <param name="initial_value">${initial_positions['joint4']}</param>
-                </state_interface>
-                <state_interface name="velocity">
-                    <param name="initial_value">0.0</param>
-                </state_interface>
-                <state_interface name="effort"/>
+                <state_interface name="position"/>
+                <state_interface name="velocity"/>
+                <!-- <state_interface name="effort"/> -->
             </joint>
             <joint name="${prefix}joint5">
@@ -118,12 +91,7 @@
                     <param name="max">3.15</param>
                 </command_interface>
-                <!-- <state_interface name="position"/> -->
-                <state_interface name="position">
-                    <param name="initial_value">${initial_positions['joint5']}</param>
-                </state_interface>
-                <state_interface name="velocity">
-                    <param name="initial_value">0.0</param>
-                </state_interface>
-                <state_interface name="effort"/>
+                <state_interface name="position"/>
+                <state_interface name="velocity"/>
+                <!-- <state_interface name="effort"/> -->
             </joint>
             <xacro:if value="${indy_type == 'indyrp2' or indy_type == 'indyrp2_v2'}">
@@ -137,12 +105,7 @@
                         <param name="max">3.15</param>
                     </command_interface>
-                    <!-- <state_interface name="position"/> -->
-                    <state_interface name="position">
-                        <param name="initial_value">${initial_positions['joint6']}</param>
-                    </state_interface>
-                    <state_interface name="velocity">
-                        <param name="initial_value">0.0</param>
-                    </state_interface>
-                    <state_interface name="effort"/>
+                    <state_interface name="position"/>
+                    <state_interface name="velocity"/>
+                    <!-- <state_interface name="effort"/> -->
                 </joint>
             </xacro:if>

File: indy_description/urdf/indy.urdf.xacro (robot description, xacro)
@@ -14,5 +14,4 @@
     <xacro:arg name="physical_params" default="$(find indy_description)/urdf/config/$(arg indy_type)/physical_parameters.yaml"/>
     <xacro:arg name="visual_params" default="$(find indy_description)/urdf/config/$(arg indy_type)/visual_parameters.yaml"/>
-    <xacro:arg name="initial_positions" default="$(find indy_description)/urdf/config/initial_positions.yaml"/>
     <xacro:arg name="transmission_hw_interface" default=""/>
     <xacro:arg name="sim_gazebo" default="false" />
@@ -32,5 +31,4 @@
         visual_parameters_file="$(arg visual_params)"
         transmission_hw_interface="$(arg transmission_hw_interface)"
-        initial_positions_file="$(arg initial_positions)"
         sim_gazebo="$(arg sim_gazebo)"
         >
@@ -44,7 +42,7 @@
             </plugin>
         </gazebo>
-            <!-- <robot_param>robot_description</robot_param> -->
-            <!-- <robot_param_node>robot_state_publisher</robot_param_node> -->
-            <!-- <parameters>$(find indy_gazebo)/controller/indy_controllers_7dof.yaml</parameters> -->
+        <!-- <robot_param>robot_description</robot_param> -->
+        <!-- <robot_param_node>robot_state_publisher</robot_param_node> -->
+        <!-- <parameters>$(find indy_gazebo)/controller/indy_controllers_7dof.yaml</parameters> -->
     </xacro:if>
 </robot>

File: indy_description/urdf/indy_common.xacro (robot description, xacro)
@@ -8,9 +8,9 @@
         </inertial>
     </xacro:macro>
-    <xacro:macro name="get_visual_params" params="name:=^ type:=^" >
+    <xacro:macro name="get_visual_params" params="name:=^ type:=^">
         <xacro:property name="visual_params" value="${sec_mesh_files[name][type]}" scope="parent"/>
     </xacro:macro>
     <!-- Get mesh files -->
-    <xacro:macro name="get_mesh_path" params="name:=^ type:=^" >
+    <xacro:macro name="get_mesh_path" params="name:=^ type:=^">
         <xacro:get_visual_params />
         <!--RVIZ2-->
@@ -21,20 +21,18 @@
         <xacro:property name="mesh" value="file://$(find ${visual_params['mesh']['package']})/${visual_params['mesh']['path']}" scope="parent"/>
     </xacro:macro>
-    <xacro:macro name="get_mesh" params="name type" >
+    <xacro:macro name="get_mesh" params="name type">
         <xacro:get_mesh_path/>
         <mesh filename="${mesh}"/>
     </xacro:macro>
     <xacro:macro name="read_model_data" params="joint_limits_parameters_file
-        kinematics_parameters_file
-        physical_parameters_file
-        visual_parameters_file
-        initial_positions_file
-        indy_type">
+	    kinematics_parameters_file
+	    physical_parameters_file
+	    visual_parameters_file
+	    indy_type">
         <!-- Read .yaml files from disk, load content into properties -->
-        <xacro:property name="config_joint_limit_parameters" value="${xacro.load_yaml(joint_limits_parameters_file)}"/>
-        <xacro:property name="config_kinematics_parameters" value="${xacro.load_yaml(kinematics_parameters_file)}"/>
-        <xacro:property name="config_physical_parameters" value="${xacro.load_yaml(physical_parameters_file)}"/>
-        <xacro:property name="config_visual_parameters" value="${xacro.load_yaml(visual_parameters_file)}"/>
-        <xacro:property name="initial_positions_parameters" value="${xacro.load_yaml(initial_positions_file)}"/>
+        <xacro:property name="config_joint_limit_parameters" value="${load_yaml(joint_limits_parameters_file)}"/>
+        <xacro:property name="config_kinematics_parameters" value="${load_yaml(kinematics_parameters_file)}"/>
+        <xacro:property name="config_physical_parameters" value="${load_yaml(physical_parameters_file)}"/>
+        <xacro:property name="config_visual_parameters" value="${load_yaml(visual_parameters_file)}"/>
         <!-- Extract subsections from yaml dictionaries -->
         <xacro:property name="sec_limits" value="${config_joint_limit_parameters['joint_limits']}"/>
@@ -47,30 +45,24 @@
         <xacro:property name="joint0_velocity_limit" value="${sec_limits['joint0']['max_velocity']}" scope="parent"/>
         <xacro:property name="joint0_effort_limit" value="${sec_limits['joint0']['max_effort']}" scope="parent"/>
-        <!-- <xacro:property name="joint0_acceleration_limit" value="${sec_limits['joint0']['max_acceleration']}" scope="parent"/> -->
         <xacro:property name="joint1_lower_limit" value="${sec_limits['joint1']['min_position']}" scope="parent"/>
         <xacro:property name="joint1_upper_limit" value="${sec_limits['joint1']['max_position']}" scope="parent"/>
         <xacro:property name="joint1_velocity_limit" value="${sec_limits['joint1']['max_velocity']}" scope="parent"/>
         <xacro:property name="joint1_effort_limit" value="${sec_limits['joint1']['max_effort']}" scope="parent"/>
-        <!-- <xacro:property name="joint1_acceleration_limit" value="${sec_limits['joint1']['max_acceleration']}" scope="parent"/> -->
         <xacro:property name="joint2_lower_limit" value="${sec_limits['joint2']['min_position']}" scope="parent"/>
         <xacro:property name="joint2_upper_limit" value="${sec_limits['joint2']['max_position']}" scope="parent"/>
         <xacro:property name="joint2_velocity_limit" value="${sec_limits['joint2']['max_velocity']}" scope="parent"/>
         <xacro:property name="joint2_effort_limit" value="${sec_limits['joint2']['max_effort']}" scope="parent"/>
-        <!-- <xacro:property name="joint2_acceleration_limit" value="${sec_limits['joint2']['max_acceleration']}" scope="parent"/> -->
         <xacro:property name="joint3_lower_limit" value="${sec_limits['joint3']['min_position']}" scope="parent"/>
         <xacro:property name="joint3_upper_limit" value="${sec_limits['joint3']['max_position']}" scope="parent"/>
         <xacro:property name="joint3_velocity_limit" value="${sec_limits['joint3']['max_velocity']}" scope="parent"/>
         <xacro:property name="joint3_effort_limit" value="${sec_limits['joint3']['max_effort']}" scope="parent"/>
-        <!-- <xacro:property name="joint3_acceleration_limit" value="${sec_limits['joint3']['max_acceleration']}" scope="parent"/> -->
         <xacro:property name="joint4_lower_limit" value="${sec_limits['joint4']['min_position']}" scope="parent"/>
         <xacro:property name="joint4_upper_limit" value="${sec_limits['joint4']['max_position']}" scope="parent"/>
         <xacro:property name="joint4_velocity_limit" value="${sec_limits['joint4']['max_velocity']}" scope="parent"/>
         <xacro:property name="joint4_effort_limit" value="${sec_limits['joint4']['max_effort']}" scope="parent"/>
-        <!-- <xacro:property name="joint4_acceleration_limit" value="${sec_limits['joint4']['max_acceleration']}" scope="parent"/> -->
         <xacro:property name="joint5_lower_limit" value="${sec_limits['joint5']['min_position']}" scope="parent"/>
         <xacro:property name="joint5_upper_limit" value="${sec_limits['joint5']['max_position']}" scope="parent"/>
         <xacro:property name="joint5_velocity_limit" value="${sec_limits['joint5']['max_velocity']}" scope="parent"/>
         <xacro:property name="joint5_effort_limit" value="${sec_limits['joint5']['max_effort']}" scope="parent"/>
-        <!-- <xacro:property name="joint5_acceleration_limit" value="${sec_limits['joint5']['max_acceleration']}" scope="parent"/> -->
         <!-- kinematics -->
         <xacro:property name="joint0_x" value="${sec_kinematics['joint0']['x']}" scope="parent"/>
@@ -181,9 +173,5 @@
             <xacro:property name="inertia_link7_iyz" value="${sec_inertia_parameters['link7']['iyz']}" scope="parent"/>
             <xacro:property name="inertia_link7_ixz" value="${sec_inertia_parameters['link7']['ixz']}" scope="parent"/>
-            <xacro:property name="initial_positions" value="${initial_positions_parameters['7dof']}" scope="parent"/>
         </xacro:if>
-        <xacro:unless value="${indy_type == 'indyrp2' or indy_type == 'indyrp2_v2'}">
-            <xacro:property name="initial_positions" value="${initial_positions_parameters['6dof']}" scope="parent"/>
-        </xacro:unless>
     </xacro:macro>
 </robot>

File: indy_description/urdf/indy_macro.xacro (robot description, xacro)
@@ -16,8 +16,6 @@
         physical_parameters_file
         visual_parameters_file
-        initial_positions_file
         transmission_hw_interface:=hardware_interface/PositionJointInterface
         sim_gazebo:=false">
-        <!-- initial_positions:=${dict(joint0=0.0,joint1=0.0,joint2=-1.57,joint3=0.0,joint4=-1.57,joint5=0.0)} -->
         <!-- Load configuration data from the provided .yaml files -->
         <xacro:read_model_data
@@ -26,5 +24,4 @@
             physical_parameters_file="${physical_parameters_file}"
             visual_parameters_file="${visual_parameters_file}"
-            initial_positions_file="${initial_positions_file}"
             indy_type="${indy_type}"/>
         <xacro:property name="indy_material" value="metal_white"/>
@@ -301,5 +298,4 @@
             indy_type="${indy_type}"
             prefix="${prefix}"
-            initial_positions="${initial_positions}"
             sim_gazebo="${sim_gazebo}"/>
         <!-- Add URDF transmission elements (for ros_control) -->
