Commit message: feature KEPCO project. Sigma7 + Indy Teleoperation function

File: indy_description/urdf/indy.ros2_control.xacro (robot description, xacro)
@@ -2,21 +2,13 @@
 <robot xmlns:xacro="http://wiki.ros.org/xacro">
     <xacro:macro name="indy_ros2_control" params="
-        name
-        indy_type
-        prefix
-        sim_gazebo:=false">
-        <ros2_control name="${name}" type="system">
+        robot_name
+        indy_type">
+        <ros2_control name="indy" type="system">
             <hardware>
-                <xacro:if value="${sim_gazebo}">
-                    <plugin>gazebo_ros2_control/GazeboSystem</plugin>
-                </xacro:if>
-                <xacro:unless value="${sim_gazebo}">
-                    <plugin>fake_components/GenericSystem</plugin>
-                    <!-- <param name="fake_sensor_commands">${fake_sensor_commands}</param> -->
-                    <param name="state_following_offset">0.0</param>
-                </xacro:unless>
+                <plugin>fake_components/GenericSystem</plugin>
+                <param name="state_following_offset">0.0</param>
             </hardware>
             <xacro:macro name="define_control_joint" params="joint_index">
-                <joint name="${prefix}${joint_index}">
+                <joint name="${robot_name}${joint_index}">
                     <command_interface name="position">
                         <param name="min">{-2*pi}</param>

File: indy_description/urdf/indy_macro.xacro (robot description, xacro)
@@ -2,12 +2,10 @@
 <robot xmlns:xacro="http://wiki.ros.org/xacro">
     <xacro:include filename="$(find indy_description)/urdf/indy.ros2_control.xacro" />
-    <xacro:include filename="$(find indy_description)/urdf/indy_transmissions.xacro"/>
     <xacro:include filename="$(find indy_description)/urdf/indy_common.xacro"/>
     <xacro:include filename="$(find indy_description)/urdf/materials.xacro"/>
     <xacro:macro name="indy_robot" params="
-        name
+        robot_name
         indy_type
         indy_eye
-        prefix
         parent
         *origin
@@ -15,14 +13,10 @@
         kinematics_parameters_file
         physical_parameters_file
-        visual_parameters_file
-        transmission_hw_interface:=hardware_interface/PositionJointInterface
-        sim_gazebo:=false">
-        <!-- initial_positions:=${dict(joint0=0.0,joint1=0.0,joint2=-1.57,joint3=0.0,joint4=-1.57,joint5=0.0)} -->
-        <!-- Load configuration data from the provided .yaml files -->
+        visual_parameters_file">
         <xacro:define_initialize visual_parameters_file="${visual_parameters_file}"/>
         <xacro:property name="indy_material" value="metal_white"/>
-        <!-- links -  main serial chain -->
+        <!-- links - main serial chain -->
         <xacro:macro name="define_link" params="link_index link_mesh">
-            <link name="${prefix}${link_index}">
+            <link name="${robot_name}${link_index}">
                 <xacro:property name="config_physical_parameters" value="${load_yaml(physical_parameters_file)}"/>
                 <xacro:property name="sec_inertia_parameters" value="${config_physical_parameters['inertia_parameters']}" />
@@ -77,10 +71,9 @@
             </xacro:unless>
         </xacro:if>
-        <link name="${prefix}tcp"/>
-        <!-- joints -->
-        <joint name="global" type="fixed">
-            <origin xyz="0 0 0" rpy="0 0 0"/>
-            <parent link="${parent}"/> <!--world-->
-            <child link="$(arg prefix)link0"/>
+        <link name="${robot_name}tcp"/>
+        <joint name="${robot_name}global" type="fixed">
+            <xacro:insert_block name="origin" />
+            <parent link="${parent}"/>
+            <child link="${robot_name}link0"/>
         </joint>
         <xacro:macro name="define_joint" params="joint_index link_1_index link_2_index" >
@@ -89,7 +82,7 @@
             <xacro:property name="sec_kinematics" value="${config_kinematics_parameters['kinematics']}" />
             <xacro:property name="sec_limits" value="${config_joint_limit_parameters['joint_limits']}"/>
-            <joint name="${prefix}${joint_index}" type="revolute">
-                <parent link="${prefix}${link_1_index}"/>
-                <child link="${prefix}${link_2_index}"/>
+            <joint name="${robot_name}${joint_index}" type="revolute">
+                <parent link="${robot_name}${link_1_index}"/>
+                <child link="${robot_name}${link_2_index}"/>
                 <origin
                     xyz="${sec_kinematics[joint_index]['x']}
@@ -115,14 +108,14 @@
         <xacro:if value="${indy_type == 'indyrp2' or indy_type == 'indyrp2_v2'}">
             <xacro:define_joint joint_index="joint6" link_1_index="link6" link_2_index="link7"/>
-            <joint name="${prefix}tcp" type="fixed">
-                <parent link="${prefix}link7"/>
-                <child link="${prefix}tcp"/>
+            <joint name="${robot_name}tcp" type="fixed">
+                <parent link="${robot_name}link7"/>
+                <child link="${robot_name}tcp"/>
                 <origin xyz="0 0 0.06" rpy="0 0 0"/>
             </joint>
         </xacro:if>
         <xacro:unless value="${indy_type == 'indyrp2' or indy_type == 'indyrp2_v2'}">
-            <joint name="${prefix}tcp" type="fixed">
-                <parent link="${prefix}link6"/>
-                <child link="${prefix}tcp"/>
+            <joint name="${robot_name}tcp" type="fixed">
+                <parent link="${robot_name}link6"/>
+                <child link="${robot_name}tcp"/>
                 <origin xyz="0 0 0.06" rpy="0 0 0"/>
             </joint>
@@ -130,10 +123,6 @@
         <!-- ros2 control -->
         <xacro:indy_ros2_control
-            name="${name}"
             indy_type="${indy_type}"
-            prefix="${prefix}"
-            sim_gazebo="${sim_gazebo}"/>
-        <!-- Add URDF transmission elements (for ros_control) -->
-        <!-- <xacro:indy_transmission prefix="${prefix}" hw_interface="${transmission_hw_interface}" indy_type="${indy_type}"/> -->
+            robot_name="${robot_name}"/>
     </xacro:macro>
 </robot>

File: indy_moveit/srdf/indy_macro.srdf.xacro (robot description, xacro)
@@ -5,5 +5,5 @@
     A URDF file must exist for this robot as well, where the joints and the links that are referenced are defined
     -->
-    <xacro:macro name="indy_srdf" params="name prefix indy_type">
+    <xacro:macro name="indy_srdf" params="robot_name indy_type">
         <!--GROUPS - Representation of a set of joints and links. This can be useful for specifying DOF to plan for, defining arms, end effectors, etc-->
         <!--LINKS - When a link is specified, the parent joint of that link (if it exists) is automatically included-->
@@ -11,26 +11,26 @@
         <!--CHAINS - When a chain is specified, all the links along the chain (including endpoints) are included in the group. Additionally, all the joints that are parents to included links are also included. This means that joints along the chain and the parent joint of the base link are included in the group-->
         <!--SUBGROUPS - Groups can also be formed by referencing to already defined group names-->
-        <group name="${prefix}${name}_manipulator">
-            <chain base_link="${prefix}link0" tip_link="${prefix}tcp" />
+        <group name="${robot_name}manipulator">
+            <chain base_link="${robot_name}link0" tip_link="${robot_name}tcp" />
         </group>
         <xacro:if value="${indy_type == 'indyrp2' or indy_type == 'indyrp2_v2'}">
             <!--GROUP STATES - Purpose - Define a named state for a particular group, in terms of joint values. This is useful to define states like 'folded arms'-->
-            <group_state name="${prefix}HomePos" group="${prefix}${name}_manipulator">
-                <joint name="${prefix}joint0" value="0" />
-                <joint name="${prefix}joint1" value="0" />
-                <joint name="${prefix}joint2" value="0" />
-                <joint name="${prefix}joint3" value="-1.570796327" />
-                <joint name="${prefix}joint4" value="0" />
-                <joint name="${prefix}joint5" value="-1.570796327" />
-                <joint name="${prefix}joint6" value="0" />
+            <group_state name="${robot_name}HomePos" group="${robot_name}manipulator">
+                <joint name="${robot_name}joint0" value="0" />
+                <joint name="${robot_name}joint1" value="0" />
+                <joint name="${robot_name}joint2" value="0" />
+                <joint name="${robot_name}joint3" value="-1.570796327" />
+                <joint name="${robot_name}joint4" value="0" />
+                <joint name="${robot_name}joint5" value="-1.570796327" />
+                <joint name="${robot_name}joint6" value="0" />
             </group_state>
-            <group_state name="${prefix}ZeroPos" group="${prefix}${name}_manipulator">
-                <joint name="${prefix}joint0" value="0" />
-                <joint name="${prefix}joint1" value="0" />
-                <joint name="${prefix}joint2" value="0" />
-                <joint name="${prefix}joint3" value="0" />
-                <joint name="${prefix}joint4" value="0" />
-                <joint name="${prefix}joint5" value="0" />
-                <joint name="${prefix}joint6" value="0" />
+            <group_state name="${robot_name}ZeroPos" group="${robot_name}manipulator">
+                <joint name="${robot_name}joint0" value="0" />
+                <joint name="${robot_name}joint1" value="0" />
+                <joint name="${robot_name}joint2" value="0" />
+                <joint name="${robot_name}joint3" value="0" />
+                <joint name="${robot_name}joint4" value="0" />
+                <joint name="${robot_name}joint5" value="0" />
+                <joint name="${robot_name}joint6" value="0" />
             </group_state>
             <!--END EFFECTOR - Purpose - Represent information about an end effector.-->
@@ -38,29 +38,29 @@
             <virtual_joint name="FixedBase" type="fixed" parent_frame="global" child_link="world" />
             <!--DISABLE COLLISIONS - By default it is assumed that any link of the robot could potentially come into collision with any other link in the robot. This tag disables collision checking between a specified pair of links. -->
-            <disable_collisions link1="link0" link2="link1" reason="Adjacent" />
-            <disable_collisions link1="link1" link2="link2" reason="Adjacent" />
-            <disable_collisions link1="link2" link2="link3" reason="Adjacent" />
-            <disable_collisions link1="link3" link2="link4" reason="Adjacent" />
-            <disable_collisions link1="link4" link2="link5" reason="Adjacent" />
-            <disable_collisions link1="link5" link2="link6" reason="Adjacent" />
-            <disable_collisions link1="link6" link2="link7" reason="Adjacent" />
+            <disable_collisions link1="${robot_name}link0" link2="${robot_name}link1" reason="Adjacent" />
+            <disable_collisions link1="${robot_name}link1" link2="${robot_name}link2" reason="Adjacent" />
+            <disable_collisions link1="${robot_name}link2" link2="${robot_name}link3" reason="Adjacent" />
+            <disable_collisions link1="${robot_name}link3" link2="${robot_name}link4" reason="Adjacent" />
+            <disable_collisions link1="${robot_name}link4" link2="${robot_name}link5" reason="Adjacent" />
+            <disable_collisions link1="${robot_name}link5" link2="${robot_name}link6" reason="Adjacent" />
+            <disable_collisions link1="${robot_name}link6" link2="${robot_name}link7" reason="Adjacent" />
         </xacro:if>
         <xacro:unless value="${indy_type == 'indyrp2' or indy_type == 'indyrp2_v2'}">
             <!--GROUP STATES - Purpose - Define a named state for a particular group, in terms of joint values. This is useful to define states like 'folded arms'-->
-            <group_state name="${prefix}HomePos" group="${prefix}${name}_manipulator">
-                <joint name="${prefix}joint0" value="0" />
-                <joint name="${prefix}joint1" value="0" />
-                <joint name="${prefix}joint2" value="-1.570796327" />
-                <joint name="${prefix}joint3" value="0" />
-                <joint name="${prefix}joint4" value="-1.570796327" />
-                <joint name="${prefix}joint5" value="0" />
+            <group_state name="${robot_name}HomePos" group="${robot_name}manipulator">
+                <joint name="${robot_name}joint0" value="0" />
+                <joint name="${robot_name}joint1" value="0" />
+                <joint name="${robot_name}joint2" value="-1.570796327" />
+                <joint name="${robot_name}joint3" value="0" />
+                <joint name="${robot_name}joint4" value="-1.570796327" />
+                <joint name="${robot_name}joint5" value="0" />
             </group_state>
-            <group_state name="${prefix}ZeroPos" group="${prefix}${name}_manipulator">
-                <joint name="${prefix}joint0" value="0" />
-                <joint name="${prefix}joint1" value="0" />
-                <joint name="${prefix}joint2" value="0" />
-                <joint name="${prefix}joint3" value="0" />
-                <joint name="${prefix}joint4" value="0" />
-                <joint name="${prefix}joint5" value="0" />
+            <group_state name="${robot_name}ZeroPos" group="${robot_name}manipulator">
+                <joint name="${robot_name}joint0" value="0" />
+                <joint name="${robot_name}joint1" value="0" />
+                <joint name="${robot_name}joint2" value="0" />
+                <joint name="${robot_name}joint3" value="0" />
+                <joint name="${robot_name}joint4" value="0" />
+                <joint name="${robot_name}joint5" value="0" />
             </group_state>
             <!--END EFFECTOR - Purpose - Represent information about an end effector.-->
@@ -68,16 +68,16 @@
             <virtual_joint name="FixedBase" type="fixed" parent_frame="global" child_link="world" />
             <!--DISABLE COLLISIONS - By default it is assumed that any link of the robot could potentially come into collision with any other link in the robot. This tag disables collision checking between a specified pair of links. -->
-            <disable_collisions link1="link0" link2="link1" reason="Adjacent" />
-            <disable_collisions link1="link1" link2="link2" reason="Adjacent" />
-            <disable_collisions link1="link2" link2="link3" reason="Adjacent" />
-            <disable_collisions link1="link3" link2="link4" reason="Adjacent" />
-            <disable_collisions link1="link4" link2="link5" reason="Adjacent" />
-            <disable_collisions link1="link5" link2="link6" reason="Adjacent" />
-            <disable_collisions link1="link2" link2="link4" reason="Never" />
-            <disable_collisions link1="link2" link2="link5" reason="Never" />
-            <disable_collisions link1="link2" link2="link6" reason="Never" />
-            <disable_collisions link1="link3" link2="link5" reason="Never" />
-            <disable_collisions link1="link3" link2="link6" reason="Never" />
-            <disable_collisions link1="link4" link2="link6" reason="Never" />
+            <disable_collisions link1="${robot_name}link0" link2="${robot_name}link1" reason="Adjacent" />
+            <disable_collisions link1="${robot_name}link1" link2="${robot_name}link2" reason="Adjacent" />
+            <disable_collisions link1="${robot_name}link2" link2="${robot_name}link3" reason="Adjacent" />
+            <disable_collisions link1="${robot_name}link3" link2="${robot_name}link4" reason="Adjacent" />
+            <disable_collisions link1="${robot_name}link4" link2="${robot_name}link5" reason="Adjacent" />
+            <disable_collisions link1="${robot_name}link5" link2="${robot_name}link6" reason="Adjacent" />
+            <disable_collisions link1="${robot_name}link2" link2="${robot_name}link4" reason="Never" />
+            <disable_collisions link1="${robot_name}link2" link2="${robot_name}link5" reason="Never" />
+            <disable_collisions link1="${robot_name}link2" link2="${robot_name}link6" reason="Never" />
+            <disable_collisions link1="${robot_name}link3" link2="${robot_name}link5" reason="Never" />
+            <disable_collisions link1="${robot_name}link3" link2="${robot_name}link6" reason="Never" />
+            <disable_collisions link1="${robot_name}link4" link2="${robot_name}link6" reason="Never" />
         </xacro:unless>
     </xacro:macro>
