Commit message: add eir robot

File: indy_moveit/srdf/indy_macro.srdf.xacro (robot description, xacro)
@@ -5,5 +5,5 @@
     A URDF file must exist for this robot as well, where the joints and the links that are referenced are defined
     -->
-    <xacro:macro name="indy_srdf" params="name prefix indy_type">
+    <xacro:macro name="indy_srdf" params="name prefix indy_type gripper_dh_ag95:=false">
         <!--GROUPS - Representation of a set of joints and links. This can be useful for specifying DOF to plan for, defining arms, end effectors, etc-->
         <!--LINKS - When a link is specified, the parent joint of that link (if it exists) is automatically included-->
@@ -11,73 +11,146 @@
         <!--CHAINS - When a chain is specified, all the links along the chain (including endpoints) are included in the group. Additionally, all the joints that are parents to included links are also included. This means that joints along the chain and the parent joint of the base link are included in the group-->
         <!--SUBGROUPS - Groups can also be formed by referencing to already defined group names-->
-        <group name="${prefix}${name}_manipulator">
-            <chain base_link="${prefix}link0" tip_link="${prefix}tcp" />
-        </group>
-        <xacro:if value="${indy_type == 'indyrp2' or indy_type == 'indyrp2_v2'}">
-            <!--GROUP STATES - Purpose - Define a named state for a particular group, in terms of joint values. This is useful to define states like 'folded arms'-->
-            <group_state name="${prefix}HomePos" group="${prefix}${name}_manipulator">
-                <joint name="${prefix}joint0" value="0" />
-                <joint name="${prefix}joint1" value="0" />
-                <joint name="${prefix}joint2" value="0" />
-                <joint name="${prefix}joint3" value="-1.570796327" />
-                <joint name="${prefix}joint4" value="0" />
-                <joint name="${prefix}joint5" value="-1.570796327" />
-                <joint name="${prefix}joint6" value="0" />
+        <xacro:if value="${indy_type == 'eir'}">
+            <group name="${prefix}left_arm">
+                <chain base_link="${prefix}left_arm_base" tip_link="${prefix}left_arm_link_7" />
+            </group>
+            <group name="${prefix}right_arm">
+                <chain base_link="${prefix}right_arm_base" tip_link="${prefix}right_arm_link_7" />
+            </group>
+            <group name="${prefix}dual_arm">
+                <group name="${prefix}left_arm" />
+                <group name="${prefix}right_arm" />
+            </group>
+            <group_state name="${prefix}LeftZero" group="${prefix}left_arm">
+                <joint name="${prefix}Joint_L2_L" value="0" />
+                <joint name="${prefix}Joint_L3_L" value="0" />
+                <joint name="${prefix}Joint_L4_L" value="0" />
+                <joint name="${prefix}Joint_L5_L" value="0" />
+                <joint name="${prefix}Joint_L6_L" value="0" />
+                <joint name="${prefix}Joint_L7_L" value="0" />
+                <joint name="${prefix}Joint_L8_L" value="0" />
             </group_state>
-            <group_state name="${prefix}ZeroPos" group="${prefix}${name}_manipulator">
-                <joint name="${prefix}joint0" value="0" />
-                <joint name="${prefix}joint1" value="0" />
-                <joint name="${prefix}joint2" value="0" />
-                <joint name="${prefix}joint3" value="0" />
-                <joint name="${prefix}joint4" value="0" />
-                <joint name="${prefix}joint5" value="0" />
-                <joint name="${prefix}joint6" value="0" />
+            <group_state name="${prefix}RightZero" group="${prefix}right_arm">
+                <joint name="${prefix}Joint_L2_R" value="0" />
+                <joint name="${prefix}Joint_L3_R" value="0" />
+                <joint name="${prefix}Joint_L4_R" value="0" />
+                <joint name="${prefix}Joint_L5_R" value="0" />
+                <joint name="${prefix}Joint_L6_R" value="0" />
+                <joint name="${prefix}Joint_L7_R" value="0" />
+                <joint name="${prefix}Joint_L8_R" value="0" />
             </group_state>
-            <!--END EFFECTOR - Purpose - Represent information about an end effector.-->
-            <!--VIRTUAL JOINT - Purpose - this element defines a virtual joint between a robot link and an external frame of reference (considered fixed with respect to the robot)-->
             <virtual_joint name="FixedBase" type="fixed" parent_frame="global" child_link="world" />
-            <!--DISABLE COLLISIONS - By default it is assumed that any link of the robot could potentially come into collision with any other link in the robot. This tag disables collision checking between a specified pair of links. -->
-            <disable_collisions link1="link0" link2="link1" reason="Adjacent" />
-            <disable_collisions link1="link1" link2="link2" reason="Adjacent" />
-            <disable_collisions link1="link2" link2="link3" reason="Adjacent" />
-            <disable_collisions link1="link3" link2="link4" reason="Adjacent" />
-            <disable_collisions link1="link4" link2="link5" reason="Adjacent" />
-            <disable_collisions link1="link5" link2="link6" reason="Adjacent" />
-            <disable_collisions link1="link6" link2="link7" reason="Adjacent" />
+            <disable_collisions link1="${prefix}base_link" link2="${prefix}torso_yaw" reason="Adjacent" />
+            <disable_collisions link1="${prefix}torso_yaw" link2="${prefix}torso_pitch" reason="Adjacent" />
+            <disable_collisions link1="${prefix}torso_pitch" link2="${prefix}head_pitch" reason="Adjacent" />
+            <disable_collisions link1="${prefix}head_pitch" link2="${prefix}head_yaw" reason="Adjacent" />
+            <disable_collisions link1="${prefix}torso_pitch" link2="${prefix}left_arm_base" reason="Adjacent" />
+            <disable_collisions link1="${prefix}left_arm_base" link2="${prefix}left_arm_link_1" reason="Adjacent" />
+            <disable_collisions link1="${prefix}left_arm_link_1" link2="${prefix}left_arm_link_2" reason="Adjacent" />
+            <disable_collisions link1="${prefix}left_arm_link_2" link2="${prefix}left_arm_link_3" reason="Adjacent" />
+            <disable_collisions link1="${prefix}left_arm_link_3" link2="${prefix}left_arm_link_4" reason="Adjacent" />
+            <disable_collisions link1="${prefix}left_arm_link_4" link2="${prefix}left_arm_link_5" reason="Adjacent" />
+            <disable_collisions link1="${prefix}left_arm_link_5" link2="${prefix}left_arm_link_6" reason="Adjacent" />
+            <disable_collisions link1="${prefix}left_arm_link_6" link2="${prefix}left_arm_link_7" reason="Adjacent" />
+            <disable_collisions link1="${prefix}torso_pitch" link2="${prefix}right_arm_base" reason="Adjacent" />
+            <disable_collisions link1="${prefix}right_arm_base" link2="${prefix}right_arm_link_1" reason="Adjacent" />
+            <disable_collisions link1="${prefix}right_arm_link_1" link2="${prefix}right_arm_link_2" reason="Adjacent" />
+            <disable_collisions link1="${prefix}right_arm_link_2" link2="${prefix}right_arm_link_3" reason="Adjacent" />
+            <disable_collisions link1="${prefix}right_arm_link_3" link2="${prefix}right_arm_link_4" reason="Adjacent" />
+            <disable_collisions link1="${prefix}right_arm_link_4" link2="${prefix}right_arm_link_5" reason="Adjacent" />
+            <disable_collisions link1="${prefix}right_arm_link_5" link2="${prefix}right_arm_link_6" reason="Adjacent" />
+            <disable_collisions link1="${prefix}right_arm_link_6" link2="${prefix}right_arm_link_7" reason="Adjacent" />
+            <xacro:if value="${gripper_dh_ag95}">
+                <disable_collisions link1="${prefix}left_arm_link_7" link2="${prefix}left_gripper_base_link" reason="Adjacent" />
+                <disable_collisions link1="${prefix}left_gripper_base_link" link2="${prefix}left_gripper_finger1_inner_knuckle_link" reason="Adjacent" />
+                <disable_collisions link1="${prefix}left_gripper_base_link" link2="${prefix}left_gripper_finger2_inner_knuckle_link" reason="Adjacent" />
+                <disable_collisions link1="${prefix}left_gripper_finger1_finger_link" link2="${prefix}left_gripper_finger1_finger_tip_link" reason="Adjacent" />
+                <disable_collisions link1="${prefix}left_gripper_finger1_finger_tip_link" link2="${prefix}left_gripper_finger1_inner_knuckle_link" reason="Adjacent" />
+                <disable_collisions link1="${prefix}left_gripper_finger1_inner_knuckle_link" link2="${prefix}left_gripper_finger1_knuckle_link" reason="Adjacent" />
+                <disable_collisions link1="${prefix}left_gripper_finger2_finger_link" link2="${prefix}left_gripper_finger2_finger_tip_link" reason="Adjacent" />
+                <disable_collisions link1="${prefix}left_gripper_finger2_finger_tip_link" link2="${prefix}left_gripper_finger2_inner_knuckle_link" reason="Adjacent" />
+                <disable_collisions link1="${prefix}left_gripper_finger2_inner_knuckle_link" link2="${prefix}left_gripper_finger2_knuckle_link" reason="Adjacent" />
+                <disable_collisions link1="${prefix}right_arm_link_7" link2="${prefix}right_gripper_base_link" reason="Adjacent" />
+                <disable_collisions link1="${prefix}right_gripper_base_link" link2="${prefix}right_gripper_finger1_inner_knuckle_link" reason="Adjacent" />
+                <disable_collisions link1="${prefix}right_gripper_base_link" link2="${prefix}right_gripper_finger2_inner_knuckle_link" reason="Adjacent" />
+                <disable_collisions link1="${prefix}right_gripper_finger1_finger_link" link2="${prefix}right_gripper_finger1_finger_tip_link" reason="Adjacent" />
+                <disable_collisions link1="${prefix}right_gripper_finger1_finger_tip_link" link2="${prefix}right_gripper_finger1_inner_knuckle_link" reason="Adjacent" />
+                <disable_collisions link1="${prefix}right_gripper_finger1_inner_knuckle_link" link2="${prefix}right_gripper_finger1_knuckle_link" reason="Adjacent" />
+                <disable_collisions link1="${prefix}right_gripper_finger2_finger_link" link2="${prefix}right_gripper_finger2_finger_tip_link" reason="Adjacent" />
+                <disable_collisions link1="${prefix}right_gripper_finger2_finger_tip_link" link2="${prefix}right_gripper_finger2_inner_knuckle_link" reason="Adjacent" />
+                <disable_collisions link1="${prefix}right_gripper_finger2_inner_knuckle_link" link2="${prefix}right_gripper_finger2_knuckle_link" reason="Adjacent" />
+            </xacro:if>
         </xacro:if>
-        <xacro:unless value="${indy_type == 'indyrp2' or indy_type == 'indyrp2_v2'}">
-            <!--GROUP STATES - Purpose - Define a named state for a particular group, in terms of joint values. This is useful to define states like 'folded arms'-->
-            <group_state name="${prefix}HomePos" group="${prefix}${name}_manipulator">
-                <joint name="${prefix}joint0" value="0" />
-                <joint name="${prefix}joint1" value="0" />
-                <joint name="${prefix}joint2" value="-1.570796327" />
-                <joint name="${prefix}joint3" value="0" />
-                <joint name="${prefix}joint4" value="-1.570796327" />
-                <joint name="${prefix}joint5" value="0" />
-            </group_state>
-            <group_state name="${prefix}ZeroPos" group="${prefix}${name}_manipulator">
-                <joint name="${prefix}joint0" value="0" />
-                <joint name="${prefix}joint1" value="0" />
-                <joint name="${prefix}joint2" value="0" />
-                <joint name="${prefix}joint3" value="0" />
-                <joint name="${prefix}joint4" value="0" />
-                <joint name="${prefix}joint5" value="0" />
-            </group_state>
-            <!--END EFFECTOR - Purpose - Represent information about an end effector.-->
-            <!--VIRTUAL JOINT - Purpose - this element defines a virtual joint between a robot link and an external frame of reference (considered fixed with respect to the robot)-->
-            <virtual_joint name="FixedBase" type="fixed" parent_frame="global" child_link="world" />
-            <!--DISABLE COLLISIONS - By default it is assumed that any link of the robot could potentially come into collision with any other link in the robot. This tag disables collision checking between a specified pair of links. -->
-            <disable_collisions link1="link0" link2="link1" reason="Adjacent" />
-            <disable_collisions link1="link1" link2="link2" reason="Adjacent" />
-            <disable_collisions link1="link2" link2="link3" reason="Adjacent" />
-            <disable_collisions link1="link3" link2="link4" reason="Adjacent" />
-            <disable_collisions link1="link4" link2="link5" reason="Adjacent" />
-            <disable_collisions link1="link5" link2="link6" reason="Adjacent" />
-            <disable_collisions link1="link2" link2="link4" reason="Never" />
-            <disable_collisions link1="link2" link2="link5" reason="Never" />
-            <disable_collisions link1="link2" link2="link6" reason="Never" />
-            <disable_collisions link1="link3" link2="link5" reason="Never" />
-            <disable_collisions link1="link3" link2="link6" reason="Never" />
-            <disable_collisions link1="link4" link2="link6" reason="Never" />
+        <xacro:unless value="${indy_type == 'eir'}">
+            <group name="${prefix}${name}_manipulator">
+                <chain base_link="${prefix}link0" tip_link="${prefix}tcp" />
+            </group>
+            <xacro:if value="${indy_type == 'indyrp2' or indy_type == 'indyrp2_v2'}">
+                <!--GROUP STATES - Purpose - Define a named state for a particular group, in terms of joint values. This is useful to define states like 'folded arms'-->
+                <group_state name="${prefix}HomePos" group="${prefix}${name}_manipulator">
+                    <joint name="${prefix}joint0" value="0" />
+                    <joint name="${prefix}joint1" value="0" />
+                    <joint name="${prefix}joint2" value="0" />
+                    <joint name="${prefix}joint3" value="-1.570796327" />
+                    <joint name="${prefix}joint4" value="0" />
+                    <joint name="${prefix}joint5" value="-1.570796327" />
+                    <joint name="${prefix}joint6" value="0" />
+                </group_state>
+                <group_state name="${prefix}ZeroPos" group="${prefix}${name}_manipulator">
+                    <joint name="${prefix}joint0" value="0" />
+                    <joint name="${prefix}joint1" value="0" />
+                    <joint name="${prefix}joint2" value="0" />
+                    <joint name="${prefix}joint3" value="0" />
+                    <joint name="${prefix}joint4" value="0" />
+                    <joint name="${prefix}joint5" value="0" />
+                    <joint name="${prefix}joint6" value="0" />
+                </group_state>
+                <!--END EFFECTOR - Purpose - Represent information about an end effector.-->
+                <!--VIRTUAL JOINT - Purpose - this element defines a virtual joint between a robot link and an external frame of reference (considered fixed with respect to the robot)-->
+                <virtual_joint name="FixedBase" type="fixed" parent_frame="global" child_link="world" />
+                <!--DISABLE COLLISIONS - By default it is assumed that any link of the robot could potentially come into collision with any other link in the robot. This tag disables collision checking between a specified pair of links. -->
+                <disable_collisions link1="link0" link2="link1" reason="Adjacent" />
+                <disable_collisions link1="link1" link2="link2" reason="Adjacent" />
+                <disable_collisions link1="link2" link2="link3" reason="Adjacent" />
+                <disable_collisions link1="link3" link2="link4" reason="Adjacent" />
+                <disable_collisions link1="link4" link2="link5" reason="Adjacent" />
+                <disable_collisions link1="link5" link2="link6" reason="Adjacent" />
+                <disable_collisions link1="link6" link2="link7" reason="Adjacent" />
+            </xacro:if>
+            <xacro:unless value="${indy_type == 'indyrp2' or indy_type == 'indyrp2_v2'}">
+                <!--GROUP STATES - Purpose - Define a named state for a particular group, in terms of joint values. This is useful to define states like 'folded arms'-->
+                <group_state name="${prefix}HomePos" group="${prefix}${name}_manipulator">
+                    <joint name="${prefix}joint0" value="0" />
+                    <joint name="${prefix}joint1" value="0" />
+                    <joint name="${prefix}joint2" value="-1.570796327" />
+                    <joint name="${prefix}joint3" value="0" />
+                    <joint name="${prefix}joint4" value="-1.570796327" />
+                    <joint name="${prefix}joint5" value="0" />
+                </group_state>
+                <group_state name="${prefix}ZeroPos" group="${prefix}${name}_manipulator">
+                    <joint name="${prefix}joint0" value="0" />
+                    <joint name="${prefix}joint1" value="0" />
+                    <joint name="${prefix}joint2" value="0" />
+                    <joint name="${prefix}joint3" value="0" />
+                    <joint name="${prefix}joint4" value="0" />
+                    <joint name="${prefix}joint5" value="0" />
+                </group_state>
+                <!--END EFFECTOR - Purpose - Represent information about an end effector.-->
+                <!--VIRTUAL JOINT - Purpose - this element defines a virtual joint between a robot link and an external frame of reference (considered fixed with respect to the robot)-->
+                <virtual_joint name="FixedBase" type="fixed" parent_frame="global" child_link="world" />
+                <!--DISABLE COLLISIONS - By default it is assumed that any link of the robot could potentially come into collision with any other link in the robot. This tag disables collision checking between a specified pair of links. -->
+                <disable_collisions link1="link0" link2="link1" reason="Adjacent" />
+                <disable_collisions link1="link1" link2="link2" reason="Adjacent" />
+                <disable_collisions link1="link2" link2="link3" reason="Adjacent" />
+                <disable_collisions link1="link3" link2="link4" reason="Adjacent" />
+                <disable_collisions link1="link4" link2="link5" reason="Adjacent" />
+                <disable_collisions link1="link5" link2="link6" reason="Adjacent" />
+                <disable_collisions link1="link2" link2="link4" reason="Never" />
+                <disable_collisions link1="link2" link2="link5" reason="Never" />
+                <disable_collisions link1="link2" link2="link6" reason="Never" />
+                <disable_collisions link1="link3" link2="link5" reason="Never" />
+                <disable_collisions link1="link3" link2="link6" reason="Never" />
+                <disable_collisions link1="link4" link2="link6" reason="Never" />
+            </xacro:unless>
         </xacro:unless>
     </xacro:macro>
