Commit message: add eir robot

File: indy_description/urdf/indy.ros2_control.xacro (robot description, xacro)
@@ -50,3 +50,63 @@
         </ros2_control>
     </xacro:macro>
+    <xacro:macro name="eir_ros2_control" params="
+        name
+        prefix
+        gripper_dh_ag95:=false
+        sim_gazebo:=false">
+        <ros2_control name="${name}" type="system">
+            <hardware>
+                <xacro:if value="${sim_gazebo}">
+                    <plugin>gazebo_ros2_control/GazeboSystem</plugin>
+                </xacro:if>
+                <xacro:unless value="${sim_gazebo}">
+                    <plugin>fake_components/GenericSystem</plugin>
+                    <param name="state_following_offset">0.0</param>
+                </xacro:unless>
+            </hardware>
+            <xacro:macro name="define_eir_control_joint" params="joint_name">
+                <joint name="${prefix}${joint_name}">
+                    <command_interface name="position">
+                        <param name="min">-6.283185</param>
+                        <param name="max">6.283185</param>
+                    </command_interface>
+                    <command_interface name="velocity">
+                        <param name="min">-6.283185</param>
+                        <param name="max">6.283185</param>
+                    </command_interface>
+                    <state_interface name="position">
+                        <param name="initial_value">0.0</param>
+                    </state_interface>
+                    <state_interface name="velocity">
+                        <param name="initial_value">0.0</param>
+                    </state_interface>
+                    <state_interface name="effort">
+                        <param name="initial_value">0.0</param>
+                    </state_interface>
+                </joint>
+            </xacro:macro>
+            <xacro:define_eir_control_joint joint_name="Joint_L0"/>
+            <xacro:define_eir_control_joint joint_name="Joint_L1"/>
+            <xacro:define_eir_control_joint joint_name="Joint_L2_U"/>
+            <xacro:define_eir_control_joint joint_name="Joint_L3_U"/>
+            <xacro:define_eir_control_joint joint_name="Joint_L2_L"/>
+            <xacro:define_eir_control_joint joint_name="Joint_L3_L"/>
+            <xacro:define_eir_control_joint joint_name="Joint_L4_L"/>
+            <xacro:define_eir_control_joint joint_name="Joint_L5_L"/>
+            <xacro:define_eir_control_joint joint_name="Joint_L6_L"/>
+            <xacro:define_eir_control_joint joint_name="Joint_L7_L"/>
+            <xacro:define_eir_control_joint joint_name="Joint_L8_L"/>
+            <xacro:define_eir_control_joint joint_name="Joint_L2_R"/>
+            <xacro:define_eir_control_joint joint_name="Joint_L3_R"/>
+            <xacro:define_eir_control_joint joint_name="Joint_L4_R"/>
+            <xacro:define_eir_control_joint joint_name="Joint_L5_R"/>
+            <xacro:define_eir_control_joint joint_name="Joint_L6_R"/>
+            <xacro:define_eir_control_joint joint_name="Joint_L7_R"/>
+            <xacro:define_eir_control_joint joint_name="Joint_L8_R"/>
+            <xacro:if value="${gripper_dh_ag95}">
+                <xacro:define_eir_control_joint joint_name="right_gripper_finger1_joint"/>
+                <xacro:define_eir_control_joint joint_name="left_gripper_finger1_joint"/>
+            </xacro:if>
+        </ros2_control>
+    </xacro:macro>
 </robot>

File: indy_description/urdf/indy.urdf.xacro (robot description, xacro)
@@ -3,4 +3,5 @@
     <!-- import main macro -->
     <xacro:include filename="$(find indy_description)/urdf/indy_macro.xacro"/>
+    <xacro:include filename="$(find indy_description)/urdf/eir_macro.xacro"/>
     <!-- robot name parameter -->
     <xacro:arg name="name" default="indy"/>
@@ -8,4 +9,5 @@
     <xacro:arg name="indy_type" default="indy7"/>
     <xacro:arg name="indy_eye" default="false"/>
+    <xacro:arg name="gripper_dh_ag95" default="false"/>
     <xacro:property name="arg_indy_type" value="$(arg indy_type)"/>
     <xacro:property name="config_indy_type" value="${arg_indy_type}"/>
@@ -17,4 +19,5 @@
     <xacro:arg name="visual_params" default="$(find indy_description)/urdf/config/${config_indy_type}/visual_parameters.yaml"/>
     <xacro:arg name="joint_axes_params" default="$(find indy_description)/urdf/config/${config_indy_type}/joint_axes.yaml"/>
+    <xacro:arg name="joint_mimics_params" default="$(find indy_description)/urdf/config/${config_indy_type}/joint_mimics.yaml"/>
     <xacro:arg name="initial_positions" default="$(find indy_description)/urdf/config/initial_positions.yaml"/>
     <xacro:arg name="transmission_hw_interface" default=""/>
@@ -22,23 +25,47 @@
     <xacro:arg name="simulation_controllers" default="" />
     <link name="world" />
-    <!-- define robot -->
-    <!-- transmission_hw_interface use for ros1 -->
-    <xacro:indy_robot
-        name="$(arg name)"
-        indy_type="$(arg indy_type)"
-        indy_eye="$(arg indy_eye)"
-        prefix="$(arg prefix)"
-        parent="world"
-        joint_limits_parameters_file="$(arg joint_limit_params)"
-        kinematics_parameters_file="$(arg kinematics_params)"
-        physical_parameters_file="$(arg physical_params)"
-        visual_parameters_file="$(arg visual_params)"
-        joint_axes_parameters_file="$(arg joint_axes_params)"
-        transmission_hw_interface="$(arg transmission_hw_interface)"
-        initial_positions_file="$(arg initial_positions)"
-        sim_gazebo="$(arg sim_gazebo)"
-        >
-        <origin xyz="0 0 0" rpy="0 0 0" />          <!-- position robot in the world -->
-    </xacro:indy_robot>
+    <xacro:if value="${config_indy_type == 'eir'}">
+        <xacro:eir_robot
+            name="$(arg name)"
+            gripper_dh_ag95="$(arg gripper_dh_ag95)"
+            prefix="$(arg prefix)"
+            parent="world"
+            joint_limits_parameters_file="$(arg joint_limit_params)"
+            kinematics_parameters_file="$(arg kinematics_params)"
+            physical_parameters_file="$(arg physical_params)"
+            visual_parameters_file="$(arg visual_params)"
+            joint_axes_parameters_file="$(arg joint_axes_params)"
+            joint_mimics_parameters_file="$(arg joint_mimics_params)"
+            >
+            <origin xyz="0 0 0" rpy="0 0 0" />
+        </xacro:eir_robot>
+        <xacro:eir_ros2_control
+            name="$(arg name)"
+            prefix="$(arg prefix)"
+            gripper_dh_ag95="$(arg gripper_dh_ag95)"
+            sim_gazebo="$(arg sim_gazebo)"
+        />
+    </xacro:if>
+    <xacro:unless value="${config_indy_type == 'eir'}">
+        <!-- define robot -->
+        <!-- transmission_hw_interface use for ros1 -->
+        <xacro:indy_robot
+            name="$(arg name)"
+            indy_type="$(arg indy_type)"
+            indy_eye="$(arg indy_eye)"
+            prefix="$(arg prefix)"
+            parent="world"
+            joint_limits_parameters_file="$(arg joint_limit_params)"
+            kinematics_parameters_file="$(arg kinematics_params)"
+            physical_parameters_file="$(arg physical_params)"
+            visual_parameters_file="$(arg visual_params)"
+            joint_axes_parameters_file="$(arg joint_axes_params)"
+            transmission_hw_interface="$(arg transmission_hw_interface)"
+            initial_positions_file="$(arg initial_positions)"
+            sim_gazebo="$(arg sim_gazebo)"
+            >
+            <origin xyz="0 0 0" rpy="0 0 0" />          <!-- position robot in the world -->
+        </xacro:indy_robot>
+    </xacro:unless>
     <xacro:if value="$(arg sim_gazebo)">
         <gazebo reference="world"> </gazebo>

File: indy_description/urdf_files/dual_icon3.urdf (robot description, URDF)
Before this commit: robot indy, 20 links, 19 joints
Joints:
- removed joint left_arm_tcp_fixed
- removed joint right_arm_tcp_fixed
- added joint left_arm_tcp: type fixed, parent left_arm_link6, child left_arm_tcp, origin xyz=0.0                          0.0                          0.0 rpy=0.0                         0.0                         0.0
- added joint right_arm_tcp: type fixed, parent right_arm_link6, child right_arm_tcp, origin xyz=0.0                          0.0                          0.0 rpy=0.0                         0.0                         0.0

File: indy_description/urdf_files/icon3.urdf (robot description, URDF)
Before this commit: robot indy, 9 links, 8 joints
Joints:
- removed joint tcp_fixed
- added joint tcp: type fixed, parent link6, child tcp, origin xyz=0.0                          0.0                          0.0 rpy=0.0                         0.0                         0.0

File: indy_description/urdf_files/icon7l.urdf (robot description, URDF)
Before this commit: robot indy, 9 links, 8 joints
Joints:
- removed joint tcp_fixed
- added joint tcp: type fixed, parent link6, child tcp, origin xyz=0.0                          0.0                          0.0 rpy=0.0                         0.0                         0.0

File: indy_description/urdf_files/indy12.urdf (robot description, URDF)
Before this commit: robot indy, 9 links, 8 joints
Joints:
- removed joint tcp_fixed
- added joint tcp: type fixed, parent link6, child tcp, origin xyz=0.0                          0.0                          0.056 rpy=0.0                         0.0                         0.0

File: indy_description/urdf_files/indy12_v2.urdf (robot description, URDF)
Before this commit: robot indy, 9 links, 8 joints
Joints:
- removed joint tcp_fixed
- added joint tcp: type fixed, parent link6, child tcp, origin xyz=0.0                          0.0                          0.085 rpy=0.0                         0.0                         0.0

File: indy_description/urdf_files/indy12_v3.urdf (robot description, URDF)
Before this commit: robot indy, 9 links, 8 joints
Links:
- link link0: mass 2.56262283 -> 2.5639949
- link link1: mass 23.04941339 -> 23.991417
- link link2: mass 14.27904794 -> 14.931367
- link link3: mass 4.33211778 -> 5.3500368
- link link4: mass 5.29001581 -> 5.1733062
- link link5: mass 3.54429783 -> 3.9260857
- link link6: mass 3.6323592 -> 0.887075491127
Joints:
- removed joint tcp_fixed
- added joint tcp: type fixed, parent link6, child tcp, origin xyz=0.0                          0.0                          0.074 rpy=0.0                         0.0                         0.0

File: indy_description/urdf_files/indy7.urdf (robot description, URDF)
Before this commit: robot indy, 9 links, 8 joints
Joints:
- removed joint tcp_fixed
- added joint tcp: type fixed, parent link6, child tcp, origin xyz=0.0                          0.0                          0.06 rpy=0.0                         0.0                         0.0

File: indy_description/urdf_files/indy7_eye.urdf (robot description, URDF)
Before this commit: robot indy, 9 links, 8 joints
Links:
- link link6: mass 0.38254932 -> 0.974986020981
Joints:
- removed joint tcp_fixed
- added joint tcp: type fixed, parent link6, child tcp, origin xyz=0.0                          0.0                          0.06 rpy=0.0                         0.0                         0.0

File: indy_description/urdf_files/indy7_v2.urdf (robot description, URDF)
Before this commit: robot indy, 9 links, 8 joints
Joints:
- removed joint tcp_fixed
- added joint tcp: type fixed, parent link6, child tcp, origin xyz=0.0                          0.0                          0.0505 rpy=0.0                         0.0                         0.0

File: indy_description/urdf_files/indy7_v3.urdf (robot description, URDF)
Before this commit: robot indy, 9 links, 8 joints
Links:
- link link0: mass 1.66957888 -> 1.8675212
- link link1: mass 11.43955917 -> 13.799347
- link link2: mass 6.11383823 -> 7.6008233
- link link3: mass 2.68211719 -> 3.3232222
- link link4: mass 2.12830848 -> 2.6598934
- link link5: mass 2.32413397 -> 2.6363853
- link link6: mass 0.39652271 -> 0.60020684
Joints:
- removed joint tcp_fixed
- added joint tcp: type fixed, parent link6, child tcp, origin xyz=0.0                          0.0                          0.0557 rpy=0.0                         0.0                         0.0

File: indy_description/urdf_files/indyrp2.urdf (robot description, URDF)
Before this commit: robot indy, 10 links, 9 joints
Joints:
- removed joint tcp_fixed
- added joint tcp: type fixed, parent link7, child tcp, origin xyz=0.0                          0.0                          0.06 rpy=0.0                         0.0                         0.0

File: indy_description/urdf_files/indyrp2_eye.urdf (robot description, URDF)
Before this commit: robot indy, 10 links, 9 joints
Links:
- link link7: mass 0.38254932 -> 0.974986020981
Joints:
- removed joint tcp_fixed
- added joint tcp: type fixed, parent link7, child tcp, origin xyz=0.0                          0.0                          0.06 rpy=0.0                         0.0                         0.0

File: indy_description/urdf_files/indyrp2_v2.urdf (robot description, URDF)
Before this commit: robot indy, 10 links, 9 joints
Joints:
- removed joint tcp_fixed
- added joint tcp: type fixed, parent link7, child tcp, origin xyz=0.0                          0.0                          0.0515 rpy=0.0                         0.0                         0.0

File: indy_description/urdf_files/nuri12c.urdf (robot description, URDF)
Before this commit: robot indy, 9 links, 8 joints
Joints:
- removed joint tcp_fixed
- added joint tcp: type fixed, parent link6, child tcp, origin xyz=0.0                          0.0                          0.048 rpy=0.0                         0.0                         0.0

File: indy_description/urdf_files/nuri20c.urdf (robot description, URDF)
Before this commit: robot indy, 9 links, 8 joints
Joints:
- removed joint tcp_fixed
- added joint tcp: type fixed, parent link6, child tcp, origin xyz=0.0                          0.0                          0.04 rpy=0.0                         0.0                         0.0

File: indy_description/urdf_files/nuri30.urdf (robot description, URDF)
Before this commit: robot indy, 9 links, 8 joints
Joints:
- removed joint tcp_fixed
- added joint tcp: type fixed, parent link6, child tcp, origin xyz=0.0                          0.0                          0.048 rpy=0.0                         0.0                         0.0

File: indy_description/urdf_files/nuri3s.urdf (robot description, URDF)
Before this commit: robot indy, 9 links, 8 joints
Joints:
- removed joint tcp_fixed
- added joint tcp: type fixed, parent link6, child tcp, origin xyz=0.0                          0.0                          0.0285 rpy=0.0                         0.0                         0.0

File: indy_description/urdf_files/nuri4s.urdf (robot description, URDF)
Before this commit: robot indy, 9 links, 8 joints
Joints:
- removed joint tcp_fixed
- added joint tcp: type fixed, parent link6, child tcp, origin xyz=0.0                          0.0                          0.0285 rpy=0.0                         0.0                         0.0
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