Commit message: add nuri5s and nuri5sdual

File: indy_description/urdf/indy.ros2_control.xacro (robot description, xacro)
@@ -17,6 +17,6 @@
                 </xacro:unless>
             </hardware>
-            <xacro:macro name="define_control_joint" params="joint_index">
-                <joint name="${prefix}${joint_index}">
+            <xacro:macro name="define_control_joint" params="joint_name initial_value">
+                <joint name="${prefix}${joint_name}">
                     <command_interface name="position">
                         <param name="min">-6.283185</param>
@@ -28,5 +28,5 @@
                     </command_interface>
                     <state_interface name="position">
-                        <param name="initial_value">${initial_positions[joint_index]}</param>
+                        <param name="initial_value">${initial_value}</param>
                     </state_interface>
                     <state_interface name="velocity">
@@ -38,12 +38,28 @@
                 </joint>
             </xacro:macro>
-            <xacro:define_control_joint joint_index="joint0"/>
-            <xacro:define_control_joint joint_index="joint1"/>
-            <xacro:define_control_joint joint_index="joint2"/>
-            <xacro:define_control_joint joint_index="joint3"/>
-            <xacro:define_control_joint joint_index="joint4"/>
-            <xacro:define_control_joint joint_index="joint5"/>
-            <xacro:if value="${indy_type == 'indyrp2' or indy_type == 'indyrp2_v2'}">
-                <xacro:define_control_joint joint_index="joint6"/>
+            <xacro:unless value="${indy_type == 'nuri5sdual'}">
+                <xacro:define_control_joint joint_name="joint0" initial_value="${initial_positions['joint0']}"/>
+                <xacro:define_control_joint joint_name="joint1" initial_value="${initial_positions['joint1']}"/>
+                <xacro:define_control_joint joint_name="joint2" initial_value="${initial_positions['joint2']}"/>
+                <xacro:define_control_joint joint_name="joint3" initial_value="${initial_positions['joint3']}"/>
+                <xacro:define_control_joint joint_name="joint4" initial_value="${initial_positions['joint4']}"/>
+                <xacro:define_control_joint joint_name="joint5" initial_value="${initial_positions['joint5']}"/>
+                <xacro:if value="${indy_type == 'indyrp2' or indy_type == 'indyrp2_v2'}">
+                    <xacro:define_control_joint joint_name="joint6" initial_value="${initial_positions['joint6']}"/>
+                </xacro:if>
+            </xacro:unless>
+            <xacro:if value="${indy_type == 'nuri5sdual'}">
+                <xacro:define_control_joint joint_name="left_arm_joint0" initial_value="${initial_positions['joint0']}"/>
+                <xacro:define_control_joint joint_name="left_arm_joint1" initial_value="${initial_positions['joint1']}"/>
+                <xacro:define_control_joint joint_name="left_arm_joint2" initial_value="${initial_positions['joint2']}"/>
+                <xacro:define_control_joint joint_name="left_arm_joint3" initial_value="${initial_positions['joint3']}"/>
+                <xacro:define_control_joint joint_name="left_arm_joint4" initial_value="${initial_positions['joint4']}"/>
+                <xacro:define_control_joint joint_name="left_arm_joint5" initial_value="${initial_positions['joint5']}"/>
+                <xacro:define_control_joint joint_name="right_arm_joint0" initial_value="${initial_positions['joint0']}"/>
+                <xacro:define_control_joint joint_name="right_arm_joint1" initial_value="${initial_positions['joint1']}"/>
+                <xacro:define_control_joint joint_name="right_arm_joint2" initial_value="${initial_positions['joint2']}"/>
+                <xacro:define_control_joint joint_name="right_arm_joint3" initial_value="${initial_positions['joint3']}"/>
+                <xacro:define_control_joint joint_name="right_arm_joint4" initial_value="${initial_positions['joint4']}"/>
+                <xacro:define_control_joint joint_name="right_arm_joint5" initial_value="${initial_positions['joint5']}"/>
             </xacro:if>
         </ros2_control>

File: indy_description/urdf/indy_common.xacro (robot description, xacro)
@@ -20,5 +20,8 @@
             <xacro:property name="initial_positions" value="${initial_positions_parameters['7dof']}" scope="parent"/>
         </xacro:if>
-        <xacro:unless value="${indy_type == 'indyrp2' or indy_type == 'indyrp2_v2'}">
+        <xacro:if value="${indy_type == 'nuri5sdual'}">
+            <xacro:property name="initial_positions" value="${initial_positions_parameters['nuri5sdual']}" scope="parent"/>
+        </xacro:if>
+        <xacro:unless value="${indy_type == 'indyrp2' or indy_type == 'indyrp2_v2' or indy_type == 'nuri5sdual'}">
             <xacro:property name="initial_positions" value="${initial_positions_parameters['6dof']}" scope="parent"/>
         </xacro:unless>

File: indy_description/urdf/indy_macro.xacro (robot description, xacro)
@@ -26,6 +26,7 @@
         <xacro:if value="${ indy_type == 'indy7' or indy_type == 'indy7_v2' or indy_type == 'indy7_v3' or indy_type == 'indyrp2' or
                             indy_type == 'indyrp2_v2' or indy_type == 'indy12' or indy_type == 'indy12_v2' or indy_type == 'indy12_v3' or
-                            indy_type == 'nuri3s' or indy_type == 'nuri4s' or indy_type == 'nuri7c' or indy_type == 'nuri12c' or
-                            indy_type == 'nuri20c' or indy_type == 'nuri30' or indy_type == 'opti5' or indy_type == 'opti3'}">
+                            indy_type == 'nuri3s' or indy_type == 'nuri4s' or indy_type == 'nuri5s' or indy_type == 'nuri7c' or indy_type == 'nuri12c' or
+                            indy_type == 'nuri20c' or indy_type == 'nuri30' or indy_type == 'nuri5sdual' or
+                            indy_type == 'opti5' or indy_type == 'opti3'}">
             <xacro:property name="material_0" value="indy_white"/>
             <xacro:property name="material_1" value="indy_white"/>
@@ -38,4 +39,5 @@
         <xacro:property name="supports_link6_eye" value="${indy_type == 'indy7' or indy_type == 'indy7_v2' or indy_type == 'indy7_v3' or indy_type == 'indy12_v3'}"/>
         <xacro:property name="supports_link7_eye" value="${indy_type == 'indyrp2' or indy_type == 'indyrp2_v2'}"/>
+        <xacro:property name="is_dual_robot" value="${indy_type == 'dual_icon3' or indy_type == 'nuri5sdual'}"/>
         <!-- links -  main serial chain -->
         <xacro:macro name="define_link" params="link_name physic_name visual_name material gazebo_material">
@@ -78,10 +80,14 @@
             </link>
         </xacro:macro>
-        <xacro:if value="${indy_type == 'dual_icon3'}">
-            <!--body-->
-            <xacro:define_link link_name="body_base" physic_name="body_base" visual_name="body_base" material="${material_0}" gazebo_material=""/>
-            <xacro:define_link link_name="body_frame" physic_name="body_frame" visual_name="body_frame" material="${material_0}" gazebo_material=""/>
-            <xacro:define_link link_name="body_cover" physic_name="body_cover" visual_name="body_cover" material="${material_2}" gazebo_material=""/>
-            <!-- icon3 - left -->
+        <xacro:if value="${is_dual_robot}">
+            <xacro:if value="${indy_type == 'dual_icon3'}">
+                <xacro:define_link link_name="body_base" physic_name="body_base" visual_name="body_base" material="${material_0}" gazebo_material=""/>
+                <xacro:define_link link_name="body_frame" physic_name="body_frame" visual_name="body_frame" material="${material_0}" gazebo_material=""/>
+                <xacro:define_link link_name="body_cover" physic_name="body_cover" visual_name="body_cover" material="${material_2}" gazebo_material=""/>
+            </xacro:if>
+            <xacro:if value="${indy_type == 'nuri5sdual'}">
+                <xacro:define_link link_name="body_base" physic_name="body_base" visual_name="body_base" material="${material_0}" gazebo_material=""/>
+            </xacro:if>
+            <!-- left arm -->
             <xacro:define_link link_name="left_arm_link0" physic_name="left_arm_link0" visual_name="left_arm_link0" material="${material_0}" gazebo_material=""/>
             <xacro:define_link link_name="left_arm_link1" physic_name="left_arm_link1" visual_name="left_arm_link1" material="${material_1}" gazebo_material=""/>
@@ -91,5 +97,5 @@
             <xacro:define_link link_name="left_arm_link5" physic_name="left_arm_link5" visual_name="left_arm_link5" material="${material_0}" gazebo_material=""/>
             <xacro:define_link link_name="left_arm_link6" physic_name="left_arm_link6" visual_name="left_arm_link6" material="${material_0}" gazebo_material=""/>
-            <!-- icon3 - right -->
+            <!-- right arm -->
             <xacro:define_link link_name="right_arm_link0" physic_name="right_arm_link0" visual_name="right_arm_link0" material="${material_0}" gazebo_material=""/>
             <xacro:define_link link_name="right_arm_link1" physic_name="right_arm_link1" visual_name="right_arm_link1" material="${material_1}" gazebo_material=""/>
@@ -102,5 +108,5 @@
             <link name="${prefix}right_arm_tcp"/>
         </xacro:if>
-        <xacro:unless value="${indy_type == 'dual_icon3'}">
+        <xacro:unless value="${is_dual_robot}">
             <xacro:define_link link_name="link0" physic_name="link0" visual_name="link0" material="${material_0}" gazebo_material=""/>
             <xacro:define_link link_name="link1" physic_name="link1" visual_name="link1" material="${material_1}" gazebo_material=""/>
@@ -165,5 +171,5 @@
             </joint>
         </xacro:macro>
-       <xacro:if value="${indy_type == 'dual_icon3'}">
+       <xacro:if value="${is_dual_robot}">
             <joint name="global" type="fixed">
                 <origin xyz="0 0 0" rpy="0 0 0"/>
@@ -171,8 +177,14 @@
                 <child link="$(arg prefix)body_base"/>
             </joint>
-            <xacro:define_joint joint_type="revolute" joint_name="base_frame" origin_key="base_frame" parent_link="body_base" child_link="body_frame"/>
-            <xacro:define_joint joint_type="fixed" joint_name="frame_cover" origin_key="frame_cover" parent_link="body_frame" child_link="body_cover"/>
-            <xacro:define_joint joint_type="fixed" joint_name="left_arm_connect" origin_key="left_arm_connect" parent_link="body_frame" child_link="left_arm_link0"/>
-            <xacro:define_joint joint_type="fixed" joint_name="right_arm_connect" origin_key="right_arm_connect" parent_link="body_frame" child_link="right_arm_link0"/>
+            <xacro:if value="${indy_type == 'dual_icon3'}">
+                <xacro:define_joint joint_type="revolute" joint_name="base_frame" origin_key="base_frame" parent_link="body_base" child_link="body_frame"/>
+                <xacro:define_joint joint_type="fixed" joint_name="frame_cover" origin_key="frame_cover" parent_link="body_frame" child_link="body_cover"/>
+                <xacro:define_joint joint_type="fixed" joint_name="left_arm_connect" origin_key="left_arm_connect" parent_link="body_frame" child_link="left_arm_link0"/>
+                <xacro:define_joint joint_type="fixed" joint_name="right_arm_connect" origin_key="right_arm_connect" parent_link="body_frame" child_link="right_arm_link0"/>
+            </xacro:if>
+            <xacro:if value="${indy_type == 'nuri5sdual'}">
+                <xacro:define_joint joint_type="fixed" joint_name="left_arm_connect" origin_key="left_arm_connect" parent_link="body_base" child_link="left_arm_link0"/>
+                <xacro:define_joint joint_type="fixed" joint_name="right_arm_connect" origin_key="right_arm_connect" parent_link="body_base" child_link="right_arm_link0"/>
+            </xacro:if>
             <xacro:define_joint joint_type="revolute" joint_name="left_arm_joint0" origin_key="left_arm_joint0" parent_link="left_arm_link0" child_link="left_arm_link1"/>
             <xacro:define_joint joint_type="revolute" joint_name="left_arm_joint1" origin_key="left_arm_joint1" parent_link="left_arm_link1" child_link="left_arm_link2"/>
@@ -190,5 +202,5 @@
             <xacro:define_joint joint_type="fixed" joint_name="right_arm_tcp_fixed" origin_key="right_arm_tcp" parent_link="right_arm_link6" child_link="right_arm_tcp"/>
         </xacro:if>
-        <xacro:unless value="${indy_type == 'dual_icon3'}">
+        <xacro:unless value="${is_dual_robot}">
             <joint name="global" type="fixed">
                 <origin xyz="0 0 0" rpy="0 0 0"/>

File: indy_moveit/srdf/indy_macro.srdf.xacro (robot description, xacro)
@@ -82,5 +82,76 @@
             </xacro:if>
         </xacro:if>
-        <xacro:unless value="${indy_type == 'eir'}">
+        <xacro:if value="${indy_type == 'nuri5sdual'}">
+            <group name="${prefix}left_arm">
+                <chain base_link="${prefix}left_arm_link0" tip_link="${prefix}left_arm_tcp" />
+            </group>
+            <group name="${prefix}right_arm">
+                <chain base_link="${prefix}right_arm_link0" tip_link="${prefix}right_arm_tcp" />
+            </group>
+            <group name="${prefix}dual_arm">
+                <group name="${prefix}left_arm" />
+                <group name="${prefix}right_arm" />
+            </group>
+            <group_state name="${prefix}LeftHome" group="${prefix}left_arm">
+                <joint name="${prefix}left_arm_joint0" value="0" />
+                <joint name="${prefix}left_arm_joint1" value="0" />
+                <joint name="${prefix}left_arm_joint2" value="0" />
+                <joint name="${prefix}left_arm_joint3" value="0" />
+                <joint name="${prefix}left_arm_joint4" value="0" />
+                <joint name="${prefix}left_arm_joint5" value="0" />
+            </group_state>
+            <group_state name="${prefix}RightHome" group="${prefix}right_arm">
+                <joint name="${prefix}right_arm_joint0" value="0" />
+                <joint name="${prefix}right_arm_joint1" value="0" />
+                <joint name="${prefix}right_arm_joint2" value="0" />
+                <joint name="${prefix}right_arm_joint3" value="0" />
+                <joint name="${prefix}right_arm_joint4" value="0" />
+                <joint name="${prefix}right_arm_joint5" value="0" />
+            </group_state>
+            <group_state name="${prefix}LeftZero" group="${prefix}left_arm">
+                <joint name="${prefix}left_arm_joint0" value="0" />
+                <joint name="${prefix}left_arm_joint1" value="0" />
+                <joint name="${prefix}left_arm_joint2" value="0" />
+                <joint name="${prefix}left_arm_joint3" value="0" />
+                <joint name="${prefix}left_arm_joint4" value="0" />
+                <joint name="${prefix}left_arm_joint5" value="0" />
+            </group_state>
+            <group_state name="${prefix}RightZero" group="${prefix}right_arm">
+                <joint name="${prefix}right_arm_joint0" value="0" />
+                <joint name="${prefix}right_arm_joint1" value="0" />
+                <joint name="${prefix}right_arm_joint2" value="0" />
+                <joint name="${prefix}right_arm_joint3" value="0" />
+                <joint name="${prefix}right_arm_joint4" value="0" />
+                <joint name="${prefix}right_arm_joint5" value="0" />
+            </group_state>
+            <virtual_joint name="FixedBase" type="fixed" parent_frame="global" child_link="world" />
+            <disable_collisions link1="${prefix}body_base" link2="${prefix}left_arm_link0" reason="Adjacent" />
+            <disable_collisions link1="${prefix}body_base" link2="${prefix}right_arm_link0" reason="Adjacent" />
+            <disable_collisions link1="${prefix}left_arm_link0" link2="${prefix}left_arm_link1" reason="Adjacent" />
+            <disable_collisions link1="${prefix}left_arm_link1" link2="${prefix}left_arm_link2" reason="Adjacent" />
+            <disable_collisions link1="${prefix}left_arm_link2" link2="${prefix}left_arm_link3" reason="Adjacent" />
+            <disable_collisions link1="${prefix}left_arm_link3" link2="${prefix}left_arm_link4" reason="Adjacent" />
+            <disable_collisions link1="${prefix}left_arm_link4" link2="${prefix}left_arm_link5" reason="Adjacent" />
+            <disable_collisions link1="${prefix}left_arm_link5" link2="${prefix}left_arm_link6" reason="Adjacent" />
+            <disable_collisions link1="${prefix}right_arm_link0" link2="${prefix}right_arm_link1" reason="Adjacent" />
+            <disable_collisions link1="${prefix}right_arm_link1" link2="${prefix}right_arm_link2" reason="Adjacent" />
+            <disable_collisions link1="${prefix}right_arm_link2" link2="${prefix}right_arm_link3" reason="Adjacent" />
+            <disable_collisions link1="${prefix}right_arm_link3" link2="${prefix}right_arm_link4" reason="Adjacent" />
+            <disable_collisions link1="${prefix}right_arm_link4" link2="${prefix}right_arm_link5" reason="Adjacent" />
+            <disable_collisions link1="${prefix}right_arm_link5" link2="${prefix}right_arm_link6" reason="Adjacent" />
+            <disable_collisions link1="${prefix}left_arm_link2" link2="${prefix}left_arm_link4" reason="Never" />
+            <disable_collisions link1="${prefix}left_arm_link2" link2="${prefix}left_arm_link5" reason="Never" />
+            <disable_collisions link1="${prefix}left_arm_link2" link2="${prefix}left_arm_link6" reason="Never" />
+            <disable_collisions link1="${prefix}left_arm_link3" link2="${prefix}left_arm_link5" reason="Never" />
+            <disable_collisions link1="${prefix}left_arm_link3" link2="${prefix}left_arm_link6" reason="Never" />
+            <disable_collisions link1="${prefix}left_arm_link4" link2="${prefix}left_arm_link6" reason="Never" />
+            <disable_collisions link1="${prefix}right_arm_link2" link2="${prefix}right_arm_link4" reason="Never" />
+            <disable_collisions link1="${prefix}right_arm_link2" link2="${prefix}right_arm_link5" reason="Never" />
+            <disable_collisions link1="${prefix}right_arm_link2" link2="${prefix}right_arm_link6" reason="Never" />
+            <disable_collisions link1="${prefix}right_arm_link3" link2="${prefix}right_arm_link5" reason="Never" />
+            <disable_collisions link1="${prefix}right_arm_link3" link2="${prefix}right_arm_link6" reason="Never" />
+            <disable_collisions link1="${prefix}right_arm_link4" link2="${prefix}right_arm_link6" reason="Never" />
+        </xacro:if>
+        <xacro:unless value="${indy_type == 'eir' or indy_type == 'nuri5sdual'}">
             <group name="${prefix}${name}_manipulator">
                 <chain base_link="${prefix}link0" tip_link="${prefix}tcp" />
