Commit message: Use package:// for mesh paths instead of an absolute build directory
Every mesh reference in indy_description points into a developer's own build
tree:

    file:///home/user/indy-ros2/install/indy_description/share/
    indy_description/meshes/indyrp2_v2/visual/IndyRP2_v2_0.stl

That path only resolves on a machine where a user named `user` built the
package at exactly that location, so as published the descriptions do not load
anywhere else -- RViz, Gazebo, MoveIt and any non-ROS consumer alike.  Loading
indyrp2_v2.urdf fails with "Error opening file
'file:///home/user/indy-ros2/install/...'".

Replaced with the package-relative form, which is what the meshes' actual
location supports:

    package://indy_description/meshes/indyrp2_v2/visual/IndyRP2_v2_0.stl

27 files, 512 references.  Nothing but the paths changed: no geometry,
kinematics, inertias, joint limits or materials are touched, and the diff is
512 insertions against 512 deletions.

Verified by resolving all 512 new paths against indy_description/ on disk --
every referenced mesh exists.

File: indy_description/urdf_files/eir.urdf (robot description, URDF)
Before this commit: robot indy, 22 links, 21 joints
Links:
- link base_link: geometry collision mesh filename=package://indy_description/meshes/eir/collision/base_link.S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 scale=1 1 1; visual mesh filename=package://indy_description/meshes/eir/visual/base_link.glb scale=1 1 1
- link head_pitch: geometry collision mesh filename=package://indy_description/meshes/eir/collision/link_3.STL scale=1 1 1; visual mesh filename=package://indy_description/meshes/eir/visual/link_3.STL scale=1 1 1
- link head_yaw: geometry collision mesh filename=package://indy_description/meshes/eir/collision/link_4.STL scale=1 1 1; visual mesh filename=package://indy_description/meshes/eir/visual/link_4.STL scale=1 1 1
- link left_arm_base: geometry collision mesh filename=package://indy_description/meshes/eir/collision/AR5-5_07L-W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 scale=0.001 0.001 0.001; visual mesh filename=package://indy_description/meshes/eir/visual/AR5-5_07L-W4C4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 scale=0.001 0.001 0.001
- link left_arm_link_1: geometry collision mesh filename=package://indy_description/meshes/eir/collision/AR5-5_07L-W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 scale=0.001 0.001 0.001; visual mesh filename=package://indy_description/meshes/eir/visual/AR5-5_07L-W4C4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 scale=0.001 0.001 0.001
- link left_arm_link_2: geometry collision mesh filename=package://indy_description/meshes/eir/collision/AR5-5_07L-W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 scale=0.001 0.001 0.001; visual mesh filename=package://indy_description/meshes/eir/visual/AR5-5_07L-W4C4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 scale=0.001 0.001 0.001
- link left_arm_link_3: geometry collision mesh filename=package://indy_description/meshes/eir/collision/AR5-5_07L-W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 scale=0.001 0.001 0.001; visual mesh filename=package://indy_description/meshes/eir/visual/AR5-5_07L-W4C4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 scale=0.001 0.001 0.001
- link left_arm_link_4: geometry collision mesh filename=package://indy_description/meshes/eir/collision/AR5-5_07L-W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 scale=0.001 0.001 0.001; visual mesh filename=package://indy_description/meshes/eir/visual/AR5-5_07L-W4C4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 scale=0.001 0.001 0.001
- link left_arm_link_5: geometry collision mesh filename=package://indy_description/meshes/eir/collision/AR5-5_07L-W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 scale=0.001 0.001 0.001; visual mesh filename=package://indy_description/meshes/eir/visual/AR5-5_07L-W4C4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 scale=0.001 0.001 0.001
- link left_arm_link_6: geometry collision mesh filename=package://indy_description/meshes/eir/collision/AR5-5_07L-W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 scale=0.001 0.001 0.001; visual mesh filename=package://indy_description/meshes/eir/visual/AR5-5_07L-W4C4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 scale=0.001 0.001 0.001
- link left_arm_link_7: geometry collision mesh filename=package://indy_description/meshes/eir/collision/AR5-5_07L-W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 scale=0.001 0.001 0.001; visual mesh filename=package://indy_description/meshes/eir/visual/AR5-5_07L-W4C4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 scale=0.001 0.001 0.001
- link right_arm_base: geometry collision mesh filename=package://indy_description/meshes/eir/collision/AR5-5_07R-W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 scale=0.001 0.001 0.001; visual mesh filename=package://indy_description/meshes/eir/visual/AR5-5_07R-W4C4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 scale=0.001 0.001 0.001
- link right_arm_link_1: geometry collision mesh filename=package://indy_description/meshes/eir/collision/AR5-5_07R-W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 scale=0.001 0.001 0.001; visual mesh filename=package://indy_description/meshes/eir/visual/AR5-5_07R-W4C4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 scale=0.001 0.001 0.001
- link right_arm_link_2: geometry collision mesh filename=package://indy_description/meshes/eir/collision/AR5-5_07R-W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 scale=0.001 0.001 0.001; visual mesh filename=package://indy_description/meshes/eir/visual/AR5-5_07R-W4C4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 scale=0.001 0.001 0.001
- link right_arm_link_3: geometry collision mesh filename=package://indy_description/meshes/eir/collision/AR5-5_07R-W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 scale=0.001 0.001 0.001; visual mesh filename=package://indy_description/meshes/eir/visual/AR5-5_07R-W4C4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 scale=0.001 0.001 0.001
- link right_arm_link_4: geometry collision mesh filename=package://indy_description/meshes/eir/collision/AR5-5_07R-W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 scale=0.001 0.001 0.001; visual mesh filename=package://indy_description/meshes/eir/visual/AR5-5_07R-W4C4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 scale=0.001 0.001 0.001
- link right_arm_link_5: geometry collision mesh filename=package://indy_description/meshes/eir/collision/AR5-5_07R-W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 scale=0.001 0.001 0.001; visual mesh filename=package://indy_description/meshes/eir/visual/AR5-5_07R-W4C4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 scale=0.001 0.001 0.001
- link right_arm_link_6: geometry collision mesh filename=package://indy_description/meshes/eir/collision/AR5-5_07R-W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 scale=0.001 0.001 0.001; visual mesh filename=package://indy_description/meshes/eir/visual/AR5-5_07R-W4C4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 scale=0.001 0.001 0.001
- link right_arm_link_7: geometry collision mesh filename=package://indy_description/meshes/eir/collision/AR5-5_07R-W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 scale=0.001 0.001 0.001; visual mesh filename=package://indy_description/meshes/eir/visual/AR5-5_07R-W4C4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 scale=0.001 0.001 0.001
- link torso_pitch: geometry collision mesh filename=package://indy_description/meshes/eir/collision/link_2.STL scale=1 1 1; visual mesh filename=package://indy_description/meshes/eir/visual/link_2.STL scale=1 1 1
- link torso_yaw: geometry collision mesh filename=package://indy_description/meshes/eir/collision/link_1.STL scale=1 1 1; visual mesh filename=package://indy_description/meshes/eir/visual/link_1.STL scale=1 1 1

File: indy_description/urdf_files/eir_dh_ag95.urdf (robot description, URDF)
Before this commit: robot indy, 42 links, 41 joints
Links:
- link base_link: geometry collision mesh filename=package://indy_description/meshes/eir/collision/base_link.S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 scale=1 1 1; visual mesh filename=package://indy_description/meshes/eir/visual/base_link.glb scale=1 1 1
- link head_pitch: geometry collision mesh filename=package://indy_description/meshes/eir/collision/link_3.STL scale=1 1 1; visual mesh filename=package://indy_description/meshes/eir/visual/link_3.STL scale=1 1 1
- link head_yaw: geometry collision mesh filename=package://indy_description/meshes/eir/collision/link_4.STL scale=1 1 1; visual mesh filename=package://indy_description/meshes/eir/visual/link_4.STL scale=1 1 1
- link left_arm_base: geometry collision mesh filename=package://indy_description/meshes/eir/collision/AR5-5_07L-W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 scale=0.001 0.001 0.001; visual mesh filename=package://indy_description/meshes/eir/visual/AR5-5_07L-W4C4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 scale=0.001 0.001 0.001
- link left_arm_link_1: geometry collision mesh filename=package://indy_description/meshes/eir/collision/AR5-5_07L-W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 scale=0.001 0.001 0.001; visual mesh filename=package://indy_description/meshes/eir/visual/AR5-5_07L-W4C4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 scale=0.001 0.001 0.001
- link left_arm_link_2: geometry collision mesh filename=package://indy_description/meshes/eir/collision/AR5-5_07L-W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 scale=0.001 0.001 0.001; visual mesh filename=package://indy_description/meshes/eir/visual/AR5-5_07L-W4C4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 scale=0.001 0.001 0.001
- link left_arm_link_3: geometry collision mesh filename=package://indy_description/meshes/eir/collision/AR5-5_07L-W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 scale=0.001 0.001 0.001; visual mesh filename=package://indy_description/meshes/eir/visual/AR5-5_07L-W4C4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 scale=0.001 0.001 0.001
- link left_arm_link_4: geometry collision mesh filename=package://indy_description/meshes/eir/collision/AR5-5_07L-W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 scale=0.001 0.001 0.001; visual mesh filename=package://indy_description/meshes/eir/visual/AR5-5_07L-W4C4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 scale=0.001 0.001 0.001
- link left_arm_link_5: geometry collision mesh filename=package://indy_description/meshes/eir/collision/AR5-5_07L-W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 scale=0.001 0.001 0.001; visual mesh filename=package://indy_description/meshes/eir/visual/AR5-5_07L-W4C4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 scale=0.001 0.001 0.001
- link left_arm_link_6: geometry collision mesh filename=package://indy_description/meshes/eir/collision/AR5-5_07L-W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 scale=0.001 0.001 0.001; visual mesh filename=package://indy_description/meshes/eir/visual/AR5-5_07L-W4C4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 scale=0.001 0.001 0.001
- link left_arm_link_7: geometry collision mesh filename=package://indy_description/meshes/eir/collision/AR5-5_07L-W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 scale=0.001 0.001 0.001; visual mesh filename=package://indy_description/meshes/eir/visual/AR5-5_07L-W4C4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 scale=0.001 0.001 0.001
- link left_gripper_base_link: geometry collision mesh filename=package://indy_description/meshes/eir/collision/gripper_bas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 scale=0.001 0.001 0.001; visual mesh filename=package://indy_description/meshes/eir/visual/gripper_base_l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 scale=0.001 0.001 0.001
- link left_gripper_finger1_finger_link: geometry collision mesh filename=package://indy_description/meshes/eir/collision/gripper_rod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 scale=0.001 0.001 0.001; visual mesh filename=package://indy_description/meshes/eir/visual/gripper_rod_li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 scale=0.001 0.001 0.001
- link left_gripper_finger1_finger_tip_link: geometry collision mesh filename=package://indy_description/meshes/eir/collision/gripper_dis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 scale=0.001 0.001 0.001; visual mesh filename=package://indy_description/meshes/eir/visual/gripper_distal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 scale=0.001 0.001 0.001
- link left_gripper_finger1_inner_knuckle_link: geometry collision mesh filename=package://indy_description/meshes/eir/collision/gripper_pro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 scale=0.001 0.001 0.001; visual mesh filename=package://indy_description/meshes/eir/visual/gripper_proxim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 scale=0.001 0.001 0.001
- link left_gripper_finger1_knuckle_link: geometry collision mesh filename=package://indy_description/meshes/eir/collision/gripper_cra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 scale=0.001 0.001 0.001; visual mesh filename=package://indy_description/meshes/eir/visual/gripper_crank_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 scale=0.001 0.001 0.001
- link left_gripper_finger2_finger_link: geometry collision mesh filename=package://indy_description/meshes/eir/collision/gripper_rod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 scale=0.001 0.001 0.001; visual mesh filename=package://indy_description/meshes/eir/visual/gripper_rod_li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 scale=0.001 0.001 0.001
- link left_gripper_finger2_finger_tip_link: geometry collision mesh filename=package://indy_description/meshes/eir/collision/gripper_dis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 scale=0.001 0.001 0.001; visual mesh filename=package://indy_description/meshes/eir/visual/gripper_distal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 scale=0.001 0.001 0.001
- link left_gripper_finger2_inner_knuckle_link: geometry collision mesh filename=package://indy_description/meshes/eir/collision/gripper_pro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 scale=0.001 0.001 0.001; visual mesh filename=package://indy_description/meshes/eir/visual/gripper_proxim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 scale=0.001 0.001 0.001
- link left_gripper_finger2_knuckle_link: geometry collision mesh filename=package://indy_description/meshes/eir/collision/gripper_cra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 scale=0.001 0.001 0.001; visual mesh filename=package://indy_description/meshes/eir/visual/gripper_crank_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 scale=0.001 0.001 0.001
- link right_arm_base: geometry collision mesh filename=package://indy_description/meshes/eir/collision/AR5-5_07R-W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 scale=0.001 0.001 0.001; visual mesh filename=package://indy_description/meshes/eir/visual/AR5-5_07R-W4C4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 scale=0.001 0.001 0.001
- link right_arm_link_1: geometry collision mesh filename=package://indy_description/meshes/eir/collision/AR5-5_07R-W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 scale=0.001 0.001 0.001; visual mesh filename=package://indy_description/meshes/eir/visual/AR5-5_07R-W4C4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 scale=0.001 0.001 0.001
- link right_arm_link_2: geometry collision mesh filename=package://indy_description/meshes/eir/collision/AR5-5_07R-W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 scale=0.001 0.001 0.001; visual mesh filename=package://indy_description/meshes/eir/visual/AR5-5_07R-W4C4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 scale=0.001 0.001 0.001
- link right_arm_link_3: geometry collision mesh filename=package://indy_description/meshes/eir/collision/AR5-5_07R-W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 scale=0.001 0.001 0.001; visual mesh filename=package://indy_description/meshes/eir/visual/AR5-5_07R-W4C4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 scale=0.001 0.001 0.001
- link right_arm_link_4: geometry collision mesh filename=package://indy_description/meshes/eir/collision/AR5-5_07R-W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 scale=0.001 0.001 0.001; visual mesh filename=package://indy_description/meshes/eir/visual/AR5-5_07R-W4C4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 scale=0.001 0.001 0.001
- link right_arm_link_5: geometry collision mesh filename=package://indy_description/meshes/eir/collision/AR5-5_07R-W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 scale=0.001 0.001 0.001; visual mesh filename=package://indy_description/meshes/eir/visual/AR5-5_07R-W4C4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 scale=0.001 0.001 0.001
- link right_arm_link_6: geometry collision mesh filename=package://indy_description/meshes/eir/collision/AR5-5_07R-W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 scale=0.001 0.001 0.001; visual mesh filename=package://indy_description/meshes/eir/visual/AR5-5_07R-W4C4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 scale=0.001 0.001 0.001
- link right_arm_link_7: geometry collision mesh filename=package://indy_description/meshes/eir/collision/AR5-5_07R-W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 scale=0.001 0.001 0.001; visual mesh filename=package://indy_description/meshes/eir/visual/AR5-5_07R-W4C4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 scale=0.001 0.001 0.001
- link right_gripper_base_link: geometry collision mesh filename=package://indy_description/meshes/eir/collision/gripper_bas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 scale=0.001 0.001 0.001; visual mesh filename=package://indy_description/meshes/eir/visual/gripper_base_l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 scale=0.001 0.001 0.001
- link right_gripper_finger1_finger_link: geometry collision mesh filename=package://indy_description/meshes/eir/collision/gripper_rod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 scale=0.001 0.001 0.001; visual mesh filename=package://indy_description/meshes/eir/visual/gripper_rod_li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 scale=0.001 0.001 0.001
- link right_gripper_finger1_finger_tip_link: geometry collision mesh filename=package://indy_description/meshes/eir/collision/gripper_dis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 scale=0.001 0.001 0.001; visual mesh filename=package://indy_description/meshes/eir/visual/gripper_distal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 scale=0.001 0.001 0.001
- link right_gripper_finger1_inner_knuckle_link: geometry collision mesh filename=package://indy_description/meshes/eir/collision/gripper_pro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 scale=0.001 0.001 0.001; visual mesh filename=package://indy_description/meshes/eir/visual/gripper_proxim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 scale=0.001 0.001 0.001
- link right_gripper_finger1_knuckle_link: geometry collision mesh filename=package://indy_description/meshes/eir/collision/gripper_cra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 scale=0.001 0.001 0.001; visual mesh filename=package://indy_description/meshes/eir/visual/gripper_crank_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 scale=0.001 0.001 0.001
- link right_gripper_finger2_finger_link: geometry collision mesh filename=package://indy_description/meshes/eir/collision/gripper_rod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 scale=0.001 0.001 0.001; visual mesh filename=package://indy_description/meshes/eir/visual/gripper_rod_li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 scale=0.001 0.001 0.001
- link right_gripper_finger2_finger_tip_link: geometry collision mesh filename=package://indy_description/meshes/eir/collision/gripper_dis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 scale=0.001 0.001 0.001; visual mesh filename=package://indy_description/meshes/eir/visual/gripper_distal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 scale=0.001 0.001 0.001
- link right_gripper_finger2_inner_knuckle_link: geometry collision mesh filename=package://indy_description/meshes/eir/collision/gripper_pro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 scale=0.001 0.001 0.001; visual mesh filename=package://indy_description/meshes/eir/visual/gripper_proxim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 scale=0.001 0.001 0.001
- link right_gripper_finger2_knuckle_link: geometry collision mesh filename=package://indy_description/meshes/eir/collision/gripper_cra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 scale=0.001 0.001 0.001; visual mesh filename=package://indy_description/meshes/eir/visual/gripper_crank_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 scale=0.001 0.001 0.001
- link torso_pitch: geometry collision mesh filename=package://indy_description/meshes/eir/collision/link_2.STL scale=1 1 1; visual mesh filename=package://indy_description/meshes/eir/visual/link_2.STL scale=1 1 1
- link torso_yaw: geometry collision mesh filename=package://indy_description/meshes/eir/collision/link_1.STL scale=1 1 1; visual mesh filename=package://indy_description/meshes/eir/visual/link_1.STL scale=1 1 1
